Commit message: reconfirm Go1 inertial params

File: robots/aliengo_description/xacro/robot.xacro (robot description, xacro)
@@ -67,5 +67,5 @@
             <mass value="0.001"/>
             <origin rpy="0 0 0" xyz="0 0 0"/>
-            <inertia ixx="0.0001" ixy="0" ixz="0" iyy="0.000001" iyz="0" izz="0.0001"/>
+            <inertia ixx="0.0001" ixy="0" ixz="0" iyy="0.0001" iyz="0" izz="0.0001"/>
         </inertial>
         <visual>

File: robots/b1_description/xacro/robot.xacro (robot description, xacro)
@@ -67,5 +67,5 @@
             <mass value="0.001"/>
             <origin rpy="0 0 0" xyz="0 0 0"/>
-            <inertia ixx="0.0001" ixy="0" ixz="0" iyy="0.000001" iyz="0" izz="0.0001"/>
+            <inertia ixx="0.0001" ixy="0" ixz="0" iyy="0.0001" iyz="0" izz="0.0001"/>
         </inertial>
         <visual>

File: robots/go1_description/urdf/go1.urdf (robot description, URDF)
Before this commit: robot go1, 38 links, 37 joints
Links:
- removed link FL_thigh_shoulder
- removed link FR_thigh_shoulder
- removed link RL_thigh_shoulder
- removed link RR_thigh_shoulder
- added link FL_calf_rotor, mass 0.089; collision cylinder length=0.02 radius=0.035; visual cylinder length=0.02 radius=0.035
- added link FL_hip_rotor, mass 0.089; collision cylinder length=0.02 radius=0.035; visual cylinder length=0.02 radius=0.035
- added link FL_thigh_rotor, mass 0.089; collision cylinder length=0.02 radius=0.035; visual cylinder length=0.02 radius=0.035
- added link FR_calf_rotor, mass 0.089; collision cylinder length=0.02 radius=0.035; visual cylinder length=0.02 radius=0.035
- added link FR_hip_rotor, mass 0.089; collision cylinder length=0.02 radius=0.035; visual cylinder length=0.02 radius=0.035
- added link FR_thigh_rotor, mass 0.089; collision cylinder length=0.02 radius=0.035; visual cylinder length=0.02 radius=0.035
- added link RL_calf_rotor, mass 0.089; collision cylinder length=0.02 radius=0.035; visual cylinder length=0.02 radius=0.035
- added link RL_hip_rotor, mass 0.089; collision cylinder length=0.02 radius=0.035; visual cylinder length=0.02 radius=0.035
- added link RL_thigh_rotor, mass 0.089; collision cylinder length=0.02 radius=0.035; visual cylinder length=0.02 radius=0.035
- added link RR_calf_rotor, mass 0.089; collision cylinder length=0.02 radius=0.035; visual cylinder length=0.02 radius=0.035
- added link RR_hip_rotor, mass 0.089; collision cylinder length=0.02 radius=0.035; visual cylinder length=0.02 radius=0.035
- added link RR_thigh_rotor, mass 0.089; collision cylinder length=0.02 radius=0.035; visual cylinder length=0.02 radius=0.035
- link FL_calf: mass 0.131 -> 0.135862
- link FR_calf: mass 0.131 -> 0.135862
- link RL_calf: mass 0.131 -> 0.135862
- link RR_calf: mass 0.131 -> 0.135862
Joints:
- removed joint FL_hip_fixed
- removed joint FR_hip_fixed
- removed joint RL_hip_fixed
- removed joint RR_hip_fixed
- added joint FL_calf_rotor_joint: type fixed, parent FL_thigh, child FL_calf_rotor, origin xyz=0.0 -0.03235 0 rpy=0 0 0
- added joint FL_hip_rotor_joint: type fixed, parent trunk, child FL_hip_rotor, origin xyz=0.11215 0.04675 0 rpy=0 0 0
- added joint FL_thigh_rotor_joint: type fixed, parent FL_hip, child FL_thigh_rotor, origin xyz=0.0 -0.00015 0 rpy=0 0 0
- added joint FR_calf_rotor_joint: type fixed, parent FR_thigh, child FR_calf_rotor, origin xyz=0.0 0.03235 0 rpy=0 0 0
- added joint FR_hip_rotor_joint: type fixed, parent trunk, child FR_hip_rotor, origin xyz=0.11215 -0.04675 0 rpy=0 0 0
- added joint FR_thigh_rotor_joint: type fixed, parent FR_hip, child FR_thigh_rotor, origin xyz=0.0 0.00015 0 rpy=0 0 0
- added joint RL_calf_rotor_joint: type fixed, parent RL_thigh, child RL_calf_rotor, origin xyz=0.0 -0.03235 0 rpy=0 0 0
- added joint RL_hip_rotor_joint: type fixed, parent trunk, child RL_hip_rotor, origin xyz=-0.11215 0.04675 0 rpy=0 0 0
- added joint RL_thigh_rotor_joint: type fixed, parent RL_hip, child RL_thigh_rotor, origin xyz=0.0 -0.00015 0 rpy=0 0 0
- added joint RR_calf_rotor_joint: type fixed, parent RR_thigh, child RR_calf_rotor, origin xyz=0.0 0.03235 0 rpy=0 0 0
- added joint RR_hip_rotor_joint: type fixed, parent trunk, child RR_hip_rotor, origin xyz=-0.11215 -0.04675 0 rpy=0 0 0
- added joint RR_thigh_rotor_joint: type fixed, parent RR_hip, child RR_thigh_rotor, origin xyz=0.0 0.00015 0 rpy=0 0 0
- joint FL_calf_joint: limit lower=-2.72271363311 upper=-0.837758040957 effort=23.7 velocity=30.1 -> lower=-2.818 upper=-0.888 effort=35.55 velocity=20.06
- joint FL_hip_joint: limit lower=-1.0471975512 upper=1.0471975512 effort=23.7 velocity=30.1 -> lower=-0.863 upper=0.863 effort=23.7 velocity=30.1
- joint FL_thigh_joint: limit lower=-0.663225115758 upper=2.96705972839 effort=23.7 velocity=30.1 -> lower=-0.686 upper=4.501 effort=23.7 velocity=30.1
- joint FR_calf_joint: limit lower=-2.72271363311 upper=-0.837758040957 effort=23.7 velocity=30.1 -> lower=-2.818 upper=-0.888 effort=35.55 velocity=20.06
- joint FR_hip_joint: limit lower=-1.0471975512 upper=1.0471975512 effort=23.7 velocity=30.1 -> lower=-0.863 upper=0.863 effort=23.7 velocity=30.1
- joint FR_thigh_joint: limit lower=-0.663225115758 upper=2.96705972839 effort=23.7 velocity=30.1 -> lower=-0.686 upper=4.501 effort=23.7 velocity=30.1
- joint RL_calf_joint: limit lower=-2.72271363311 upper=-0.837758040957 effort=23.7 velocity=30.1 -> lower=-2.818 upper=-0.888 effort=35.55 velocity=20.06
- joint RL_hip_joint: limit lower=-1.0471975512 upper=1.0471975512 effort=23.7 velocity=30.1 -> lower=-0.863 upper=0.863 effort=23.7 velocity=30.1
- joint RL_thigh_joint: limit lower=-0.663225115758 upper=2.96705972839 effort=23.7 velocity=30.1 -> lower=-0.686 upper=4.501 effort=23.7 velocity=30.1
- joint RR_calf_joint: limit lower=-2.72271363311 upper=-0.837758040957 effort=23.7 velocity=30.1 -> lower=-2.818 upper=-0.888 effort=35.55 velocity=20.06
- joint RR_hip_joint: limit lower=-1.0471975512 upper=1.0471975512 effort=23.7 velocity=30.1 -> lower=-0.863 upper=0.863 effort=23.7 velocity=30.1
- joint RR_thigh_joint: limit lower=-0.663225115758 upper=2.96705972839 effort=23.7 velocity=30.1 -> lower=-0.686 upper=4.501 effort=23.7 velocity=30.1
- joint camera_joint_chin: origin xyz=0.2522 0.0125 -0.0436 rpy=3.14159265359 1.57079632679 0 -> xyz=0.2522 0.0125 -0.0436 rpy=3.141592653589793 1.5707963267948966 0
- joint camera_joint_face: origin xyz=0.2785 0.0125 0.0167 rpy=3.14159265359 0 0 -> xyz=0.2785 0.0125 0.0167 rpy=3.141592653589793 0 0
- joint camera_joint_left: origin xyz=-0.066 0.082 -0.0176 rpy=3.14159265359 0.2618 1.57079632679 -> xyz=-0.066 0.082 -0.0176 rpy=3.141592653589793 0.2618 1.5707963267948966
- joint camera_joint_rearDown: origin xyz=-0.0825 0.0125 -0.04365 rpy=3.14159265359 1.57079632679 0 -> xyz=-0.0825 0.0125 -0.04365 rpy=3.141592653589793 1.5707963267948966 0
- joint camera_joint_right: origin xyz=-0.041 -0.082 -0.0176 rpy=3.14159265359 0.2618 -1.57079632679 -> xyz=-0.041 -0.082 -0.0176 rpy=3.141592653589793 0.2618 -1.5707963267948966
- joint camera_optical_joint_chin: origin xyz=0 0 0 rpy=-1.57079632679 0 -1.57079632679 -> xyz=0 0 0 rpy=-1.5707963267948966 0 -1.5707963267948966
- joint camera_optical_joint_face: origin xyz=0 0 0 rpy=-1.57079632679 0 -1.57079632679 -> xyz=0 0 0 rpy=-1.5707963267948966 0 -1.5707963267948966
- joint camera_optical_joint_left: origin xyz=0 0 0 rpy=-1.57079632679 0 -1.57079632679 -> xyz=0 0 0 rpy=-1.5707963267948966 0 -1.5707963267948966
- joint camera_optical_joint_rearDown: origin xyz=0 0 0 rpy=-1.57079632679 0 -1.57079632679 -> xyz=0 0 0 rpy=-1.5707963267948966 0 -1.5707963267948966
- joint camera_optical_joint_right: origin xyz=0 0 0 rpy=-1.57079632679 0 -1.57079632679 -> xyz=0 0 0 rpy=-1.5707963267948966 0 -1.5707963267948966
- joint ultraSound_joint_left: origin xyz=-0.0535  0.0826 0.00868 rpy=0 0.2618 1.57079632679 -> xyz=-0.0535  0.0826 0.00868 rpy=0 0.2618 1.5707963267948966
- joint ultraSound_joint_right: origin xyz=-0.0535 -0.0826 0.00868 rpy=0 0.2618 -1.57079632679 -> xyz=-0.0535 -0.0826 0.00868 rpy=0 0.2618 -1.5707963267948966

File: robots/go1_description/xacro/const.xacro (robot description, xacro)
@@ -28,19 +28,38 @@
     <!-- <xacro:property name="trunk_offset_z" value="0.01675"/> -->
     <xacro:property name="hip_offset" value="0.08"/>
+    <!-- offset of link and rotor locations (left front) -->
+    <xacro:property name="hip_offset_x" value="0.1881"/>
+    <xacro:property name="hip_offset_y" value="0.04675"/>
+    <xacro:property name="hip_offset_z" value="0.0"/>
+    <xacro:property name="hip_rotor_offset_x" value="0.11215"/>
+    <xacro:property name="hip_rotor_offset_y" value="0.04675"/>
+    <xacro:property name="hip_rotor_offset_z" value="0.0"/>
+    <xacro:property name="thigh_offset_x" value="0"/>
+    <xacro:property name="thigh_offset_y" value="0.08"/>
+    <xacro:property name="thigh_offset_z" value="0.0"/>
+    <xacro:property name="thigh_rotor_offset_x" value="0.0"/>
+    <xacro:property name="thigh_rotor_offset_y" value="-0.00015"/>
+    <xacro:property name="thigh_rotor_offset_z" value="0.0"/>
+    <xacro:property name="calf_offset_x" value="0.0"/>
+    <xacro:property name="calf_offset_y" value="0.0"/>
+    <xacro:property name="calf_offset_z" value="-0.213"/>
+    <xacro:property name="calf_rotor_offset_x" value="0.0"/>
+    <xacro:property name="calf_rotor_offset_y" value="-0.03235"/>
+    <xacro:property name="calf_rotor_offset_z" value="0.0"/>
     <!-- joint limits -->
     <xacro:property name="damping" value="0.01"/>
     <xacro:property name="friction" value="0.2"/>
-    <xacro:property name="hip_max" value="60"/>
-    <xacro:property name="hip_min" value="-60"/>
+    <xacro:property name="hip_position_max" value="0.863"/>
+    <xacro:property name="hip_position_min" value="-0.863"/>
     <xacro:property name="hip_velocity_max" value="30.1"/>
     <xacro:property name="hip_torque_max" value="23.7"/>
-    <xacro:property name="thigh_max" value="170"/>
-    <xacro:property name="thigh_min" value="-38"/>
+    <xacro:property name="thigh_position_max" value="4.501"/>
+    <xacro:property name="thigh_position_min" value="-0.686"/>
     <xacro:property name="thigh_velocity_max" value="30.1"/>
     <xacro:property name="thigh_torque_max" value="23.7"/>
-    <xacro:property name="calf_max" value="-48"/>
-    <xacro:property name="calf_min" value="-156"/>
-    <xacro:property name="calf_velocity_max" value="30.1"/>
-    <xacro:property name="calf_torque_max" value="23.7"/>
+    <xacro:property name="calf_position_max" value="-0.888"/>
+    <xacro:property name="calf_position_min" value="-2.818"/>
+    <xacro:property name="calf_velocity_max" value="20.06"/>
+    <xacro:property name="calf_torque_max" value="35.55"/>
     <!-- dynamics inertial value        total 12.84kg -->
     <!-- trunk -->
@@ -49,43 +68,73 @@
     <xacro:property name="trunk_com_y" value="0.002"/>
     <xacro:property name="trunk_com_z" value="-0.0005"/>
-    <xacro:property name="trunk_ixx" value="0.0168352186"/>
-    <xacro:property name="trunk_ixy" value="0.0004636141"/>
-    <xacro:property name="trunk_ixz" value="0.0002367952"/>
-    <xacro:property name="trunk_iyy" value="0.0656071082"/>
-    <xacro:property name="trunk_iyz" value="0.000036671"/>
-    <xacro:property name="trunk_izz" value="0.0742720659"/>
+    <xacro:property name="trunk_ixx" value="0.0168128557"/>
+    <xacro:property name="trunk_ixy" value="-0.0002296769"/>
+    <xacro:property name="trunk_ixz" value="-0.0002945293"/>
+    <xacro:property name="trunk_iyy" value="0.063009565"/>
+    <xacro:property name="trunk_iyz" value="-0.0000418731"/>
+    <xacro:property name="trunk_izz" value="0.0716547275"/>
     <!-- hip (left front) -->
     <xacro:property name="hip_mass" value="0.591"/>
-    <xacro:property name="hip_com_x" value="-0.00541"/>
-    <xacro:property name="hip_com_y" value="-0.00074"/>
-    <xacro:property name="hip_com_z" value="0.000006"/>
-    <xacro:property name="hip_ixx" value="0.000374268192"/>
-    <xacro:property name="hip_ixy" value="0.000036844422"/>
-    <xacro:property name="hip_ixz" value="-0.000000986754"/>
-    <xacro:property name="hip_iyy" value="0.000635923669"/>
-    <xacro:property name="hip_iyz" value="-0.000001172894"/>
-    <xacro:property name="hip_izz" value="0.000457647394"/>
+    <xacro:property name="hip_com_x" value="-0.005657"/>
+    <xacro:property name="hip_com_y" value="-0.008752"/>
+    <xacro:property name="hip_com_z" value="-0.000102"/>
+    <xacro:property name="hip_ixx" value="0.000334008405"/>
+    <xacro:property name="hip_ixy" value="-0.000010826066"/>
+    <xacro:property name="hip_ixz" value="0.000001290732"/>
+    <xacro:property name="hip_iyy" value="0.000619101213"/>
+    <xacro:property name="hip_iyz" value="0.000001643194"/>
+    <xacro:property name="hip_izz" value="0.00040057614"/>
+    <xacro:property name="hip_rotor_mass" value="0.089"/>
+    <xacro:property name="hip_rotor_com_x" value="0.0"/>
+    <xacro:property name="hip_rotor_com_y" value="0.0"/>
+    <xacro:property name="hip_rotor_com_z" value="0.0"/>
+    <xacro:property name="hip_rotor_ixx" value="0.000111842"/>
+    <xacro:property name="hip_rotor_ixy" value="0.0"/>
+    <xacro:property name="hip_rotor_ixz" value="0.0"/>
+    <xacro:property name="hip_rotor_iyy" value="0.000059647"/>
+    <xacro:property name="hip_rotor_iyz" value="0.0"/>
+    <xacro:property name="hip_rotor_izz" value="0.000059647"/>
     <!-- thigh -->
     <xacro:property name="thigh_mass" value="0.92"/>
-    <xacro:property name="thigh_com_x" value="-0.003468"/>
-    <xacro:property name="thigh_com_y" value="-0.018947"/>
-    <xacro:property name="thigh_com_z" value="-0.032736"/>
-    <xacro:property name="thigh_ixx" value="0.005851561134"/>
-    <xacro:property name="thigh_ixy" value="0.000001783284"/>
-    <xacro:property name="thigh_ixz" value="0.000328291374"/>
-    <xacro:property name="thigh_iyy" value="0.005596155105"/>
-    <xacro:property name="thigh_iyz" value="0.000021430713"/>
-    <xacro:property name="thigh_izz" value="0.00107157026"/>
+    <xacro:property name="thigh_com_x" value="-0.003342"/>
+    <xacro:property name="thigh_com_y" value="-0.018054"/>
+    <xacro:property name="thigh_com_z" value="-0.033451"/>
+    <xacro:property name="thigh_ixx" value="0.004431760472"/>
+    <xacro:property name="thigh_ixy" value="0.000057496807"/>
+    <xacro:property name="thigh_ixz" value="-0.000218457134"/>
+    <xacro:property name="thigh_iyy" value="0.004485671726"/>
+    <xacro:property name="thigh_iyz" value="0.000572001265"/>
+    <xacro:property name="thigh_izz" value="0.000740309489"/>
+    <xacro:property name="thigh_rotor_mass" value="0.089"/>
+    <xacro:property name="thigh_rotor_com_x" value="0.0"/>
+    <xacro:property name="thigh_rotor_com_y" value="0.0"/>
+    <xacro:property name="thigh_rotor_com_z" value="0.0"/>
+    <xacro:property name="thigh_rotor_ixx" value="0.000059647"/>
+    <xacro:property name="thigh_rotor_ixy" value="0.0"/>
+    <xacro:property name="thigh_rotor_ixz" value="0.0"/>
+    <xacro:property name="thigh_rotor_iyy" value="0.000111842"/>
+    <xacro:property name="thigh_rotor_iyz" value="0.0"/>
+    <xacro:property name="thigh_rotor_izz" value="0.000059647"/>
     <!-- calf -->
-    <xacro:property name="calf_mass" value="0.131"/>
-    <xacro:property name="calf_com_x" value="0.006286"/>
-    <xacro:property name="calf_com_y" value="0.001307"/>
-    <xacro:property name="calf_com_z" value="-0.122269"/>
-    <xacro:property name="calf_ixx" value="0.002939186297"/>
-    <xacro:property name="calf_ixy" value="0.000001440899"/>
-    <xacro:property name="calf_ixz" value="-0.000105359550"/>
-    <xacro:property name="calf_iyy" value="0.00295576935"/>
-    <xacro:property name="calf_iyz" value="-0.000024397752"/>
-    <xacro:property name="calf_izz" value="0.000030273372"/>
+    <xacro:property name="calf_mass" value="0.135862"/>
+    <xacro:property name="calf_com_x" value="0.006197"/>
+    <xacro:property name="calf_com_y" value="0.001408"/>
+    <xacro:property name="calf_com_z" value="-0.116695"/>
+    <xacro:property name="calf_ixx" value="0.001088793059"/>
+    <xacro:property name="calf_ixy" value="-0.000000255679"/>
+    <xacro:property name="calf_ixz" value="0.000007117814"/>
+    <xacro:property name="calf_iyy" value="0.001100428748"/>
+    <xacro:property name="calf_iyz" value="0.000002077264"/>
+    <xacro:property name="calf_izz" value="0.000024787446"/>
+    <xacro:property name="calf_rotor_mass" value="0.089"/>
+    <xacro:property name="calf_rotor_com_x" value="0.0"/>
+    <xacro:property name="calf_rotor_com_y" value="0.0"/>
+    <xacro:property name="calf_rotor_com_z" value="0.0"/>
+    <xacro:property name="calf_rotor_ixx" value="0.000059647"/>
+    <xacro:property name="calf_rotor_ixy" value="0.0"/>
+    <xacro:property name="calf_rotor_ixz" value="0.0"/>
+    <xacro:property name="calf_rotor_iyy" value="0.000111842"/>
+    <xacro:property name="calf_rotor_iyz" value="0.0"/>
+    <xacro:property name="calf_rotor_izz" value="0.000059647"/>
     <!-- foot -->
     <xacro:property name="foot_mass" value="0.06"/>
