Commit message: remove unnecessary collisions

File: robots/aliengo_description/xacro/leg.xacro (robot description, xacro)
@@ -85,10 +85,10 @@
                 <material name="green"/>
             </visual>
-            <collision>
+            <!-- <collision>
                 <origin rpy="0 ${PI/2.0} 0" xyz="0 0 0"/>
                 <geometry>
                     <cylinder length="0.02" radius="0.035"/>
                 </geometry>
-            </collision>
+            </collision> -->
             <inertial>
                 <origin rpy="0 0 0" xyz="${hip_rotor_com_x} ${hip_rotor_com_y} ${hip_rotor_com_z}"/>
@@ -149,10 +149,10 @@
                 <material name="green"/>
             </visual>
-            <collision>
-                <origin rpy="${PI/2.0} 0 0" xyz="0 0 0"/>
-                <geometry>
-                    <cylinder length="0.02" radius="0.035"/>
-                </geometry>
-            </collision>
+            <!-- <collision>
+                <origin rpy="${PI/2.0} 0 0" xyz="0 0 0"/>
+                <geometry>
+                    <cylinder length="0.02" radius="0.035"/>
+                </geometry>
+            </collision> -->
             <inertial>
                 <origin rpy="0 0 0" xyz="${thigh_rotor_com_x} ${thigh_rotor_com_y} ${thigh_rotor_com_z}"/>
@@ -208,10 +208,10 @@
                 <material name="green"/>
             </visual>
-            <collision>
-                <origin rpy="${PI/2.0} 0 0" xyz="0 0 0"/>
-                <geometry>
-                    <cylinder length="0.02" radius="0.035"/>
-                </geometry>
-            </collision>
+            <!-- <collision>
+                <origin rpy="${PI/2.0} 0 0" xyz="0 0 0"/>
+                <geometry>
+                    <cylinder length="0.02" radius="0.035"/>
+                </geometry>
+            </collision> -->
             <inertial>
                 <origin rpy="0 0 0" xyz="${calf_rotor_com_x} ${calf_rotor_com_y} ${calf_rotor_com_z}"/>

File: robots/b1_description/xacro/leg.xacro (robot description, xacro)
@@ -85,10 +85,10 @@
                 <material name="green"/>
             </visual>
-            <collision>
+            <!-- <collision>
                 <origin rpy="0 ${PI/2.0} 0" xyz="0 0 0"/>
                 <geometry>
                     <cylinder length="0.02" radius="0.05"/>
                 </geometry>
-            </collision>
+            </collision> -->
             <inertial>
                 <origin rpy="0 0 0" xyz="${hip_rotor_com_x} ${hip_rotor_com_y} ${hip_rotor_com_z}"/>
@@ -149,10 +149,10 @@
                 <material name="green"/>
             </visual>
-            <collision>
-                <origin rpy="${PI/2.0} 0 0" xyz="0 0 0"/>
-                <geometry>
-                    <cylinder length="0.02" radius="0.05"/>
-                </geometry>
-            </collision>
+            <!-- <collision>
+                <origin rpy="${PI/2.0} 0 0" xyz="0 0 0"/>
+                <geometry>
+                    <cylinder length="0.02" radius="0.05"/>
+                </geometry>
+            </collision> -->
             <inertial>
                 <origin rpy="0 0 0" xyz="${thigh_rotor_com_x} ${thigh_rotor_com_y} ${thigh_rotor_com_z}"/>
@@ -208,10 +208,10 @@
                 <material name="green"/>
             </visual>
-            <collision>
-                <origin rpy="${PI/2.0} 0 0" xyz="0 0 0"/>
-                <geometry>
-                    <cylinder length="0.02" radius="0.05"/>
-                </geometry>
-            </collision>
+            <!-- <collision>
+                <origin rpy="${PI/2.0} 0 0" xyz="0 0 0"/>
+                <geometry>
+                    <cylinder length="0.02" radius="0.05"/>
+                </geometry>
+            </collision> -->
             <inertial>
                 <origin rpy="0 0 0" xyz="${calf_rotor_com_x} ${calf_rotor_com_y} ${calf_rotor_com_z}"/>
