Commit message: change b1 xacro collision shape

File: robots/b1_description/xacro/leg.xacro (robot description, xacro)
@@ -63,7 +63,18 @@
             </visual>
             <collision>
-                <origin rpy="${PI/2.0} 0 0" xyz="0 ${hip_offset*mirror} 0"/>
-                <geometry>
-                    <cylinder length="${hip_length}" radius="${hip_radius}"/>
+                <xacro:if value="${(mirror_dae == True) and (front_hind_dae == True)}">
+                    <origin rpy="0 0 0" xyz="0 0 0"/>
+                </xacro:if>
+                <xacro:if value="${(mirror_dae == False) and (front_hind_dae == True)}">
+                    <origin rpy="${PI} 0 0" xyz="0 0 0"/>
+                </xacro:if>
+                <xacro:if value="${(mirror_dae == True) and (front_hind_dae == False)}">
+                    <origin rpy="0 ${PI} 0" xyz="0 0 0"/>
+                </xacro:if>
+                <xacro:if value="${(mirror_dae == False) and (front_hind_dae == False)}">
+                    <origin rpy="${PI} ${PI} 0" xyz="0 0 0"/>
+                </xacro:if>
+                <geometry>
+                    <mesh filename="package://b1_description/meshes/hip.dae" scale="1 1 1"/>
                 </geometry>
             </collision>
@@ -127,7 +138,12 @@
             </visual>
             <collision>
-                <origin rpy="0 ${PI/2.0} 0" xyz="0 0 ${-thigh_length/2.0}"/>
-                <geometry>
-                    <box size="${thigh_length} ${thigh_width} ${thigh_height}"/>
+                <origin rpy="0 0 0" xyz="0 0 0"/>
+                <geometry>
+                    <xacro:if value="${mirror_dae == True}">
+                        <mesh filename="package://b1_description/meshes/thigh.dae" scale="1 1 1"/>
+                    </xacro:if>
+                    <xacro:if value="${mirror_dae == False}">
+                        <mesh filename="package://b1_description/meshes/thigh_mirror.dae" scale="1 1 1"/>
+                    </xacro:if>
                 </geometry>
             </collision>
@@ -186,7 +202,7 @@
             </visual>
             <collision>
-                <origin rpy="0 ${PI/2.0} 0" xyz="0 0 ${-calf_length/2.0}"/>
-                <geometry>
-                    <box size="${calf_length} ${calf_width} ${calf_height}"/>
+                <origin rpy="0 0 0" xyz="0 0 0"/>
+                <geometry>
+                    <mesh filename="package://b1_description/meshes/calf.dae" scale="1 1 1"/>
                 </geometry>
             </collision>

File: robots/b1_description/xacro/robot.xacro (robot description, xacro)
@@ -40,13 +40,7 @@
             <origin rpy="0 0 0" xyz="0 0 0"/>
             <geometry>
-                <box size="${trunk_length} ${trunk_width} ${trunk_height}"/>
+                <mesh filename="package://b1_description/meshes/trunk.dae" scale="1 1 1"/>
             </geometry>
         </collision>
-        <!-- <collision>
-            <origin rpy="0 0 0" xyz="0 0 0"/>
-            <geometry>
-                <mesh filename="package://b1_description/meshes/trunk.dae" scale="1 1 1"/>
-            </geometry>
-        </collision> -->
         <inertial>
             <origin rpy="0 0 0" xyz="${trunk_com_x} ${trunk_com_y} ${trunk_com_z}"/>

Commit message: update b1 xacro dae file

File: robots/b1_description/xacro/leg.xacro (robot description, xacro)
@@ -58,5 +58,5 @@
                 </xacro:if>
                 <geometry>
-                    <mesh filename="package://b1_description/meshes/hip.dae" scale="1 1 1"/>
+                    <mesh filename="package://b1_description/meshes/hipb.dae" scale="1 1 1"/>
                 </geometry>
                 <material name="orange"/>
@@ -76,5 +76,5 @@
                 </xacro:if>
                 <geometry>
-                    <mesh filename="package://b1_description/meshes/hip.dae" scale="1 1 1"/>
+                    <mesh filename="package://b1_description/meshes/hipb.dae" scale="1 1 1"/>
                 </geometry>
             </collision>
@@ -129,8 +129,8 @@
                 <geometry>
                     <xacro:if value="${mirror_dae == True}">
-                        <mesh filename="package://b1_description/meshes/thigh.dae" scale="1 1 1"/>
+                        <mesh filename="package://b1_description/meshes/thighb.dae" scale="1 1 1"/>
                     </xacro:if>
                     <xacro:if value="${mirror_dae == False}">
-                        <mesh filename="package://b1_description/meshes/thigh_mirror.dae" scale="1 1 1"/>
+                        <mesh filename="package://b1_description/meshes/thigh_mirrorb.dae" scale="1 1 1"/>
                     </xacro:if>
                 </geometry>
@@ -141,8 +141,8 @@
                 <geometry>
                     <xacro:if value="${mirror_dae == True}">
-                        <mesh filename="package://b1_description/meshes/thigh.dae" scale="1 1 1"/>
+                        <mesh filename="package://b1_description/meshes/thighb.dae" scale="1 1 1"/>
                     </xacro:if>
                     <xacro:if value="${mirror_dae == False}">
-                        <mesh filename="package://b1_description/meshes/thigh_mirror.dae" scale="1 1 1"/>
+                        <mesh filename="package://b1_description/meshes/thigh_mirrorb.dae" scale="1 1 1"/>
                     </xacro:if>
                 </geometry>
@@ -197,5 +197,5 @@
                 <origin rpy="0 0 0" xyz="0 0 0"/>
                 <geometry>
-                    <mesh filename="package://b1_description/meshes/calf.dae" scale="1 1 1"/>
+                    <mesh filename="package://b1_description/meshes/calfb.dae" scale="1 1 1"/>
                 </geometry>
                 <material name="orange"/>
@@ -204,5 +204,5 @@
                 <origin rpy="0 0 0" xyz="0 0 0"/>
                 <geometry>
-                    <mesh filename="package://b1_description/meshes/calf.dae" scale="1 1 1"/>
+                    <mesh filename="package://b1_description/meshes/calfb.dae" scale="1 1 1"/>
                 </geometry>
             </collision>

File: robots/b1_description/xacro/robot.xacro (robot description, xacro)
@@ -33,5 +33,5 @@
             <origin rpy="0 0 0" xyz="0 0 0"/>
             <geometry>
-                <mesh filename="package://b1_description/meshes/trunk.dae" scale="1 1 1"/>
+                <mesh filename="package://b1_description/meshes/trunkb.dae" scale="1 1 1"/>
             </geometry>
             <material name="orange"/>
@@ -40,5 +40,5 @@
             <origin rpy="0 0 0" xyz="0 0 0"/>
             <geometry>
-                <mesh filename="package://b1_description/meshes/trunk.dae" scale="1 1 1"/>
+                <mesh filename="package://b1_description/meshes/trunkb.dae" scale="1 1 1"/>
             </geometry>
         </collision>
