Commit message: add fake rotor links

File: robots/b1_description/xacro/b1.urdf (robot description, URDF)
Before this commit: robot b1_description, 19 links, 18 joints
Links:
- added link FL_calf_rotor, mass 0.266; collision cylinder length=0.02 radius=0.05; visual cylinder length=0.02 radius=0.05
- added link FL_hip_rotor, mass 0.199; collision cylinder length=0.02 radius=0.05; visual cylinder length=0.02 radius=0.05
- added link FL_thigh_rotor, mass 0.266; collision cylinder length=0.02 radius=0.05; visual cylinder length=0.02 radius=0.05
- added link FR_calf_rotor, mass 0.266; collision cylinder length=0.02 radius=0.05; visual cylinder length=0.02 radius=0.05
- added link FR_hip_rotor, mass 0.199; collision cylinder length=0.02 radius=0.05; visual cylinder length=0.02 radius=0.05
- added link FR_thigh_rotor, mass 0.266; collision cylinder length=0.02 radius=0.05; visual cylinder length=0.02 radius=0.05
- added link RL_calf_rotor, mass 0.266; collision cylinder length=0.02 radius=0.05; visual cylinder length=0.02 radius=0.05
- added link RL_hip_rotor, mass 0.199; collision cylinder length=0.02 radius=0.05; visual cylinder length=0.02 radius=0.05
- added link RL_thigh_rotor, mass 0.266; collision cylinder length=0.02 radius=0.05; visual cylinder length=0.02 radius=0.05
- added link RR_calf_rotor, mass 0.266; collision cylinder length=0.02 radius=0.05; visual cylinder length=0.02 radius=0.05
- added link RR_hip_rotor, mass 0.199; collision cylinder length=0.02 radius=0.05; visual cylinder length=0.02 radius=0.05
- added link RR_thigh_rotor, mass 0.266; collision cylinder length=0.02 radius=0.05; visual cylinder length=0.02 radius=0.05
- link FL_calf: mass 0.207 -> 0.857; geometry collision box size=0.35 0.04 0.05; visual mesh filename=package://b1_description/meshes/calf.dae scale=1 1 1
- link FL_foot: mass 0.06 -> 0.05
- link FL_hip: mass 1.993 -> 2.1
- link FL_thigh: mass 0.639 -> 3.934
- link FR_calf: mass 0.207 -> 0.857; geometry collision box size=0.35 0.04 0.05; visual mesh filename=package://b1_description/meshes/calf.dae scale=1 1 1
- link FR_foot: mass 0.06 -> 0.05
- link FR_hip: mass 1.993 -> 2.1
- link FR_thigh: mass 0.639 -> 3.934
- link RL_calf: mass 0.207 -> 0.857; geometry collision box size=0.35 0.04 0.05; visual mesh filename=package://b1_description/meshes/calf.dae scale=1 1 1
- link RL_foot: mass 0.06 -> 0.05
- link RL_hip: mass 1.993 -> 2.1
- link RL_thigh: mass 0.639 -> 3.934
- link RR_calf: mass 0.207 -> 0.857; geometry collision box size=0.35 0.04 0.05; visual mesh filename=package://b1_description/meshes/calf.dae scale=1 1 1
- link RR_foot: mass 0.06 -> 0.05
- link RR_hip: mass 1.993 -> 2.1
- link RR_thigh: mass 0.639 -> 3.934
- link trunk: mass 9.041 -> 25
Joints:
- added joint FL_calf_rotor_joint: type fixed, parent FL_thigh, child FL_calf_rotor, origin xyz=0.0 -0.0519 0 rpy=0 0 0
- added joint FL_hip_rotor_joint: type fixed, parent trunk, child FL_hip_rotor, origin xyz=0.1955 0.072 0 rpy=0 0 0
- added joint FL_thigh_rotor_joint: type fixed, parent FL_hip, child FL_thigh_rotor, origin xyz=0.0 0.00935 0 rpy=0 0 0
- added joint FR_calf_rotor_joint: type fixed, parent FR_thigh, child FR_calf_rotor, origin xyz=0.0 0.0519 0 rpy=0 0 0
- added joint FR_hip_rotor_joint: type fixed, parent trunk, child FR_hip_rotor, origin xyz=0.1955 -0.072 0 rpy=0 0 0
- added joint FR_thigh_rotor_joint: type fixed, parent FR_hip, child FR_thigh_rotor, origin xyz=0.0 -0.00935 0 rpy=0 0 0
- added joint RL_calf_rotor_joint: type fixed, parent RL_thigh, child RL_calf_rotor, origin xyz=0.0 -0.0519 0 rpy=0 0 0
- added joint RL_hip_rotor_joint: type fixed, parent trunk, child RL_hip_rotor, origin xyz=-0.1955 0.072 0 rpy=0 0 0
- added joint RL_thigh_rotor_joint: type fixed, parent RL_hip, child RL_thigh_rotor, origin xyz=0.0 0.00935 0 rpy=0 0 0
- added joint RR_calf_rotor_joint: type fixed, parent RR_thigh, child RR_calf_rotor, origin xyz=0.0 0.0519 0 rpy=0 0 0
- added joint RR_hip_rotor_joint: type fixed, parent trunk, child RR_hip_rotor, origin xyz=-0.1955 -0.072 0 rpy=0 0 0
- added joint RR_thigh_rotor_joint: type fixed, parent RR_hip, child RR_thigh_rotor, origin xyz=0.0 -0.00935 0 rpy=0 0 0
- joint FL_calf_joint: limit lower=-2.6 upper=-0.6 effort=100 velocity=20 -> lower=-2.6 upper=-0.6 effort=140 velocity=15.55
- joint FL_hip_joint: limit lower=-0.75 upper=0.75 effort=100 velocity=20 -> lower=-0.75 upper=0.75 effort=91.0035 velocity=19.69
- joint FL_thigh_joint: limit lower=-1.0 upper=3.5 effort=100 velocity=20 -> lower=-1.0 upper=3.5 effort=93.33 velocity=23.32; type continuous -> revolute
- joint FR_calf_joint: limit lower=-2.6 upper=-0.6 effort=100 velocity=20 -> lower=-2.6 upper=-0.6 effort=140 velocity=15.55
- joint FR_hip_joint: limit lower=-0.75 upper=0.75 effort=100 velocity=20 -> lower=-0.75 upper=0.75 effort=91.0035 velocity=19.69
- joint FR_thigh_joint: limit lower=-1.0 upper=3.5 effort=100 velocity=20 -> lower=-1.0 upper=3.5 effort=93.33 velocity=23.32; type continuous -> revolute
- joint RL_calf_joint: limit lower=-2.6 upper=-0.6 effort=100 velocity=20 -> lower=-2.6 upper=-0.6 effort=140 velocity=15.55
- joint RL_hip_joint: limit lower=-0.75 upper=0.75 effort=100 velocity=20 -> lower=-0.75 upper=0.75 effort=91.0035 velocity=19.69
- joint RL_thigh_joint: limit lower=-1.0 upper=3.5 effort=100 velocity=20 -> lower=-1.0 upper=3.5 effort=93.33 velocity=23.32; type continuous -> revolute
- joint RR_calf_joint: limit lower=-2.6 upper=-0.6 effort=100 velocity=20 -> lower=-2.6 upper=-0.6 effort=140 velocity=15.55
- joint RR_hip_joint: limit lower=-0.75 upper=0.75 effort=100 velocity=20 -> lower=-0.75 upper=0.75 effort=91.0035 velocity=19.69
- joint RR_thigh_joint: limit lower=-1.0 upper=3.5 effort=100 velocity=20 -> lower=-1.0 upper=3.5 effort=93.33 velocity=23.32; type continuous -> revolute

File: robots/b1_description/xacro/const.xacro (robot description, xacro)
@@ -57,9 +57,9 @@
     <xacro:property name="thigh_position_min" value="-1.0"/>
     <xacro:property name="thigh_velocity_max" value="23.32"/>
-    <xacro:property name="thigh_torque_max" value="138.672"/>
+    <xacro:property name="thigh_torque_max" value="93.33"/>
     <xacro:property name="calf_position_max" value="-0.6"/>
     <xacro:property name="calf_position_min" value="-2.6"/>
     <xacro:property name="calf_velocity_max" value="15.55"/>
-    <xacro:property name="calf_torque_max" value="208"/>
+    <xacro:property name="calf_torque_max" value="140"/>
     <!-- dynamics inertial value -->
     <!-- trunk -->

File: robots/b1_description/xacro/leg.xacro (robot description, xacro)
@@ -2,7 +2,18 @@
 <robot xmlns:xacro="http://www.ros.org/wiki/xacro">
     <xacro:include filename="$(find b1_description)/xacro/transmission.xacro"/>
-    <xacro:macro name="leg" params="name mirror mirror_dae front_hind front_hind_dae *origin">
+    <xacro:macro name="leg" params="name mirror mirror_dae front_hind front_hind_dae">
         <joint name="${name}_hip_joint" type="revolute">
-            <xacro:insert_block name="origin"/>
+            <xacro:if value="${(mirror_dae == False) and (front_hind_dae == True)}">
+                <origin rpy="0 0 0" xyz="${leg_offset_x} ${-leg_offset_y} 0"/>
+            </xacro:if>
+            <xacro:if value="${(mirror_dae == True) and (front_hind_dae == True)}">
+                <origin rpy="0 0 0" xyz="${leg_offset_x} ${leg_offset_y} 0"/>
+            </xacro:if>
+            <xacro:if value="${(mirror_dae == False) and (front_hind_dae == False)}">
+                <origin rpy="0 0 0" xyz="${-leg_offset_x} ${-leg_offset_y} 0"/>
+            </xacro:if>
+            <xacro:if value="${(mirror_dae == True) and (front_hind_dae == False)}">
+                <origin rpy="0 0 0" xyz="${-leg_offset_x} ${leg_offset_y} 0"/>
+            </xacro:if>
             <parent link="trunk"/>
             <child link="${name}_hip"/>
@@ -16,4 +27,20 @@
             </xacro:if>
         </joint>
+        <joint name="${name}_hip_rotor_joint" type="fixed">
+            <xacro:if value="${(mirror_dae == False) and (front_hind_dae == True)}">
+                <origin rpy="0 0 0" xyz="${hip_rotor_offset_x} ${-hip_rotor_offset_y} 0"/>
+            </xacro:if>
+            <xacro:if value="${(mirror_dae == True) and (front_hind_dae == True)}">
+                <origin rpy="0 0 0" xyz="${hip_rotor_offset_x} ${hip_rotor_offset_y} 0"/>
+            </xacro:if>
+            <xacro:if value="${(mirror_dae == False) and (front_hind_dae == False)}">
+                <origin rpy="0 0 0" xyz="${-hip_rotor_offset_x} ${-hip_rotor_offset_y} 0"/>
+            </xacro:if>
+            <xacro:if value="${(mirror_dae == True) and (front_hind_dae == False)}">
+                <origin rpy="0 0 0" xyz="${-hip_rotor_offset_x} ${hip_rotor_offset_y} 0"/>
+            </xacro:if>
+            <parent link="trunk"/>
+            <child link="${name}_hip_rotor"/>
+        </joint>
         <link name="${name}_hip">
             <visual>
@@ -50,18 +77,27 @@
             </inertial>
         </link>
-        <!-- <joint name="${name}_hip_fixed" type="fixed">
-            <origin rpy="0 0 0" xyz="0 ${(thigh_shoulder_length/2.0+hip_offset)*mirror} 0"/>
-            <parent link="${name}_hip"/>
-            <child link="${name}_thigh_shoulder"/>
-        </joint> -->
-        <!-- this link is only for collision -->
-        <!-- <link name="${name}_thigh_shoulder">
-            <collision>
-                <origin rpy="${PI/2.0} 0 0" xyz="0 0 0"/>
-                <geometry>
-                    <cylinder length="${thigh_shoulder_length}" radius="${thigh_shoulder_radius}"/>
-                </geometry>
-            </collision>
-        </link> -->
+        <link name="${name}_hip_rotor">
+            <visual>
+                <origin rpy="0 ${PI/2.0} 0" xyz="0 0 0"/>
+                <geometry>
+                    <cylinder length="0.02" radius="0.05"/>
+                </geometry>
+                <material name="green"/>
+            </visual>
+            <collision>
+                <origin rpy="0 ${PI/2.0} 0" xyz="0 0 0"/>
+                <geometry>
+                    <cylinder length="0.02" radius="0.05"/>
+                </geometry>
+            </collision>
+            <inertial>
+                <origin rpy="0 0 0" xyz="${hip_rotor_com_x} ${hip_rotor_com_y} ${hip_rotor_com_z}"/>
+                <mass value="${hip_rotor_mass}"/>
+                <inertia
+                    ixx="${hip_rotor_ixx}" ixy="${hip_rotor_ixy}" ixz="${hip_rotor_ixz}"
+                    iyy="${hip_rotor_iyy}" iyz="${hip_rotor_iyz}"
+                    izz="${hip_rotor_izz}"/>
+            </inertial>
+        </link>
         <joint name="${name}_thigh_joint" type="revolute">
             <origin rpy="0 0 0" xyz="0 ${thigh_offset*mirror} 0"/>
@@ -72,4 +108,9 @@
             <limit effort="${thigh_torque_max}" velocity="${thigh_velocity_max}" lower="${thigh_position_min}" upper="${thigh_position_max}"/>
         </joint>
+        <joint name="${name}_thigh_rotor_joint" type="fixed">
+            <origin rpy="0 0 0" xyz="${thigh_rotor_offset_x} ${thigh_rotor_offset_y*mirror} 0"/>
+            <parent link="${name}_hip"/>
+            <child link="${name}_thigh_rotor"/>
+        </joint>
         <link name="${name}_thigh">
             <visual>
@@ -98,4 +139,27 @@
                     iyy="${thigh_iyy}" iyz="${thigh_iyz*mirror}"
                     izz="${thigh_izz}"/>
+            </inertial>
+        </link>
+        <link name="${name}_thigh_rotor">
+            <visual>
+                <origin rpy="${PI/2.0} 0 0" xyz="0 0 0"/>
+                <geometry>
+                    <cylinder length="0.02" radius="0.05"/>
+                </geometry>
+                <material name="green"/>
+            </visual>
+            <collision>
+                <origin rpy="${PI/2.0} 0 0" xyz="0 0 0"/>
+                <geometry>
+                    <cylinder length="0.02" radius="0.05"/>
+                </geometry>
+            </collision>
+            <inertial>
+                <origin rpy="0 0 0" xyz="${thigh_rotor_com_x} ${thigh_rotor_com_y} ${thigh_rotor_com_z}"/>
+                <mass value="${thigh_rotor_mass}"/>
+                <inertia
+                    ixx="${thigh_rotor_ixx}" ixy="${thigh_rotor_ixy}" ixz="${thigh_rotor_ixz}"
+                    iyy="${thigh_rotor_iyy}" iyz="${thigh_rotor_iyz}"
+                    izz="${thigh_rotor_izz}"/>
             </inertial>
         </link>
@@ -108,4 +172,9 @@
             <limit effort="${calf_torque_max}" velocity="${calf_velocity_max}" lower="${calf_position_min}" upper="${calf_position_max}"/>
         </joint>
+        <joint name="${name}_calf_rotor_joint" type="fixed">
+            <origin rpy="0 0 0" xyz="${calf_rotor_offset_x} ${calf_rotor_offset_y*mirror} 0"/>
+            <parent link="${name}_thigh"/>
+            <child link="${name}_calf_rotor"/>
+        </joint>
         <link name="${name}_calf">
             <visual>
@@ -129,4 +198,27 @@
                     iyy="${calf_iyy}" iyz="${calf_iyz}"
                     izz="${calf_izz}"/>
+            </inertial>
+        </link>
+        <link name="${name}_calf_rotor">
+            <visual>
+                <origin rpy="${PI/2.0} 0 0" xyz="0 0 0"/>
+                <geometry>
+                    <cylinder length="0.02" radius="0.05"/>
+                </geometry>
+                <material name="green"/>
+            </visual>
+            <collision>
+                <origin rpy="${PI/2.0} 0 0" xyz="0 0 0"/>
+                <geometry>
+                    <cylinder length="0.02" radius="0.05"/>
+                </geometry>
+            </collision>
+            <inertial>
+                <origin rpy="0 0 0" xyz="${calf_rotor_com_x} ${calf_rotor_com_y} ${calf_rotor_com_z}"/>
+                <mass value="${calf_rotor_mass}"/>
+                <inertia
+                    ixx="${calf_rotor_ixx}" ixy="${calf_rotor_ixy}" ixz="${calf_rotor_ixz}"
+                    iyy="${calf_rotor_iyy}" iyz="${calf_rotor_iyz}"
+                    izz="${calf_rotor_izz}"/>
             </inertial>
         </link>

File: robots/b1_description/xacro/robot.xacro (robot description, xacro)
@@ -5,6 +5,6 @@
     <xacro:include filename="$(find b1_description)/xacro/leg.xacro"/>
     <xacro:include filename="$(find b1_description)/xacro/gazebo.xacro"/>
-    <!-- Rollover Protection mode will add an additional stick on the top, use "true" or "false" to switch it. -->
-    <xacro:property name="rolloverProtection" value="false"/>
+    <!-- Rotor related joint and link is only for demonstrate location. -->
+    <!-- Actually, the rotor will rotate and the joint is not fixed. Reduction ratio should be considered. -->
     <!-- Debug mode will hung up the robot, use "true" or "false" to switch it. -->
     <!-- <xacro:if value="$(arg DEBUG)">
@@ -58,33 +58,4 @@
         </inertial>
     </link>
-    <xacro:if value="${(rolloverProtection == 'true')}">
-        <joint name="stick_joint" type="fixed">
-            <parent link="trunk"/>
-            <child link="stick_link"/>
-            <origin rpy="0 0 0" xyz="${0.18} 0 ${stick_length/2.0+0.08}"/>
-        </joint>
-        <link name="stick_link">
-            <visual>
-                <geometry>
-                    <cylinder length="${stick_length}" radius="${stick_radius}"/>
-                </geometry>
-                <origin rpy="0 0 0" xyz="0 0 0"/>
-                <material name="white"/>
-            </visual>
-            <collision>
-                <geometry>
-                    <cylinder length="${stick_length}" radius="${stick_radius}"/>
-                </geometry>
-                <origin rpy="0 0 0" xyz="0 0 0"/>
-            </collision>
-            <inertial>
-                <mass value="${stick_mass}"/>
-                <inertia
-                    ixx="${stick_mass / 2.0 * (stick_radius*stick_radius)}" ixy="0.0" ixz="0.0"
-                    iyy="${stick_mass / 12.0 * (3*stick_radius*stick_radius + stick_length*stick_length)}" iyz="0.0"
-                    izz="${stick_mass / 12.0 * (3*stick_radius*stick_radius + stick_length*stick_length)}"/>
-            </inertial>
-        </link>
-    </xacro:if>
     <joint name="imu_joint" type="fixed">
         <parent link="trunk"/>
@@ -112,16 +83,8 @@
         </collision>
     </link>
-    <xacro:leg name="FR" mirror="-1" mirror_dae= "False" front_hind="1" front_hind_dae="True">
-        <origin rpy="0 0 0" xyz="${leg_offset_x} ${-leg_offset_y} 0"/>
-    </xacro:leg>
-    <xacro:leg name="FL" mirror="1" mirror_dae="True" front_hind="1" front_hind_dae="True">
-        <origin rpy="0 0 0" xyz="${leg_offset_x} ${leg_offset_y} 0"/>
-    </xacro:leg>
-    <xacro:leg name="RR" mirror="-1" mirror_dae="False" front_hind="-1" front_hind_dae="False">
-        <origin rpy="0 0 0" xyz="${-leg_offset_x} ${-leg_offset_y} 0"/>
-    </xacro:leg>
-    <xacro:leg name="RL" mirror="1" mirror_dae="True" front_hind="-1" front_hind_dae="False">
-        <origin rpy="0 0 0" xyz="${-leg_offset_x} ${leg_offset_y} 0"/>
-    </xacro:leg>
+    <xacro:leg name="FR" mirror="-1" mirror_dae= "False" front_hind="1"  front_hind_dae="True"  />
+    <xacro:leg name="FL" mirror="1"  mirror_dae="True"   front_hind="1"  front_hind_dae="True"  />
+    <xacro:leg name="RR" mirror="-1" mirror_dae="False"  front_hind="-1" front_hind_dae="False" />
+    <xacro:leg name="RL" mirror="1"  mirror_dae="True"   front_hind="-1" front_hind_dae="False" />
     <!-- <xacro:stairs stairs="15" xpos="0" ypos="2.0" zpos="0" /> -->
 </robot>

Commit message: change b1 URDF collision shape

File: robots/b1_description/xacro/b1.urdf (robot description, URDF)
Before this commit: robot b1_description, 31 links, 30 joints
Links:
- link FL_calf: geometry collision mesh filename=package://b1_description/meshes/calf.dae scale=1 1 1; visual mesh filename=package://b1_description/meshes/calf.dae scale=1 1 1
- link FL_hip: geometry collision mesh filename=package://b1_description/meshes/hip.dae scale=1 1 1; visual mesh filename=package://b1_description/meshes/hip.dae scale=1 1 1
- link FL_thigh: geometry collision mesh filename=package://b1_description/meshes/thigh.dae scale=1 1 1; visual mesh filename=package://b1_description/meshes/thigh.dae scale=1 1 1
- link FR_calf: geometry collision mesh filename=package://b1_description/meshes/calf.dae scale=1 1 1; visual mesh filename=package://b1_description/meshes/calf.dae scale=1 1 1
- link FR_hip: geometry collision mesh filename=package://b1_description/meshes/hip.dae scale=1 1 1; visual mesh filename=package://b1_description/meshes/hip.dae scale=1 1 1
- link FR_thigh: geometry collision mesh filename=package://b1_description/meshes/thigh_mirror.dae scale=1 1 1; visual mesh filename=package://b1_description/meshes/thigh_mirror.dae scale=1 1 1
- link RL_calf: geometry collision mesh filename=package://b1_description/meshes/calf.dae scale=1 1 1; visual mesh filename=package://b1_description/meshes/calf.dae scale=1 1 1
- link RL_hip: geometry collision mesh filename=package://b1_description/meshes/hip.dae scale=1 1 1; visual mesh filename=package://b1_description/meshes/hip.dae scale=1 1 1
- link RL_thigh: geometry collision mesh filename=package://b1_description/meshes/thigh.dae scale=1 1 1; visual mesh filename=package://b1_description/meshes/thigh.dae scale=1 1 1
- link RR_calf: geometry collision mesh filename=package://b1_description/meshes/calf.dae scale=1 1 1; visual mesh filename=package://b1_description/meshes/calf.dae scale=1 1 1
- link RR_hip: geometry collision mesh filename=package://b1_description/meshes/hip.dae scale=1 1 1; visual mesh filename=package://b1_description/meshes/hip.dae scale=1 1 1
- link RR_thigh: geometry collision mesh filename=package://b1_description/meshes/thigh_mirror.dae scale=1 1 1; visual mesh filename=package://b1_description/meshes/thigh_mirror.dae scale=1 1 1
- link trunk: geometry collision mesh filename=package://b1_description/meshes/trunk.dae scale=1 1 1; visual mesh filename=package://b1_description/meshes/trunk.dae scale=1 1 1

Commit message: update b1 URDF mass

File: robots/b1_description/xacro/b1.urdf (robot description, URDF)
Before this commit: robot b1_description, 31 links, 30 joints
Links:
- link FL_calf: mass 0.857 -> 1.05
- link FL_hip: mass 2.1 -> 2.15
- link FL_thigh: mass 3.934 -> 4.3
- link FR_calf: mass 0.857 -> 1.05
- link FR_hip: mass 2.1 -> 2.15
- link FR_thigh: mass 3.934 -> 4.3
- link RL_calf: mass 0.857 -> 1.05
- link RL_hip: mass 2.1 -> 2.15
- link RL_thigh: mass 3.934 -> 4.3
- link RR_calf: mass 0.857 -> 1.05
- link RR_hip: mass 2.1 -> 2.15
- link RR_thigh: mass 3.934 -> 4.3
- link trunk: mass 25 -> 29.45
