Commit message: update b1 URDF dae file

File: robots/b1_description/xacro/b1.urdf (robot description, URDF)
Before this commit: robot b1_description, 31 links, 30 joints
Links:
- link FL_calf: geometry collision mesh filename=package://b1_description/meshes/calfb.dae scale=1 1 1; visual mesh filename=package://b1_description/meshes/calfb.dae scale=1 1 1
- link FL_hip: geometry collision mesh filename=package://b1_description/meshes/hipb.dae scale=1 1 1; visual mesh filename=package://b1_description/meshes/hipb.dae scale=1 1 1
- link FL_thigh: geometry collision mesh filename=package://b1_description/meshes/thighb.dae scale=1 1 1; visual mesh filename=package://b1_description/meshes/thighb.dae scale=1 1 1
- link FR_calf: geometry collision mesh filename=package://b1_description/meshes/calfb.dae scale=1 1 1; visual mesh filename=package://b1_description/meshes/calfb.dae scale=1 1 1
- link FR_hip: geometry collision mesh filename=package://b1_description/meshes/hipb.dae scale=1 1 1; visual mesh filename=package://b1_description/meshes/hipb.dae scale=1 1 1
- link FR_thigh: geometry collision mesh filename=package://b1_description/meshes/thigh_mirrorb.dae scale=1 1 1; visual mesh filename=package://b1_description/meshes/thigh_mirrorb.dae scale=1 1 1
- link RL_calf: geometry collision mesh filename=package://b1_description/meshes/calfb.dae scale=1 1 1; visual mesh filename=package://b1_description/meshes/calfb.dae scale=1 1 1
- link RL_hip: geometry collision mesh filename=package://b1_description/meshes/hipb.dae scale=1 1 1; visual mesh filename=package://b1_description/meshes/hipb.dae scale=1 1 1
- link RL_thigh: geometry collision mesh filename=package://b1_description/meshes/thighb.dae scale=1 1 1; visual mesh filename=package://b1_description/meshes/thighb.dae scale=1 1 1
- link RR_calf: geometry collision mesh filename=package://b1_description/meshes/calfb.dae scale=1 1 1; visual mesh filename=package://b1_description/meshes/calfb.dae scale=1 1 1
- link RR_hip: geometry collision mesh filename=package://b1_description/meshes/hipb.dae scale=1 1 1; visual mesh filename=package://b1_description/meshes/hipb.dae scale=1 1 1
- link RR_thigh: geometry collision mesh filename=package://b1_description/meshes/thigh_mirrorb.dae scale=1 1 1; visual mesh filename=package://b1_description/meshes/thigh_mirrorb.dae scale=1 1 1
- link trunk: geometry collision mesh filename=package://b1_description/meshes/trunkb.dae scale=1 1 1; visual mesh filename=package://b1_description/meshes/trunkb.dae scale=1 1 1

Commit message: add b1 realsense link to URDF

File: robots/b1_description/xacro/b1.urdf (robot description, URDF)
Before this commit: robot b1_description, 31 links, 30 joints
Links:
- added link head_camera_1_link, mass 0.001
- added link head_camera_2_link, mass 0.001
- added link left_side_camera_link, mass 0.001
- added link right_side_camera_link, mass 0.001
- added link tail_camera_link, mass 0.001
Joints:
- added joint head_camera_1_joint: type fixed, parent trunk, child head_camera_1_link, origin xyz=0.48883 0 0.0255 rpy=0 0 0
- added joint head_camera_2_joint: type fixed, parent trunk, child head_camera_2_link, origin xyz=0.45430 0 -0.081 rpy=0 0 0
- added joint left_side_camera_joint: type fixed, parent trunk, child left_side_camera_link, origin xyz=-0.1086 0.1371 -0.03077 rpy=-0.331612 0 0
- added joint right_side_camera_joint: type fixed, parent trunk, child right_side_camera_link, origin xyz=-0.10190 -0.1371 -0.03077 rpy=0.331612 0 0
- added joint tail_camera_joint: type fixed, parent trunk, child tail_camera_link, origin xyz=-0.459 0 -0.081 rpy=0 0 0
