Commit message: add b1 realsense link to xacro

File: robots/b1_description/xacro/robot.xacro (robot description, xacro)
@@ -77,4 +77,65 @@
         </collision>
     </link>
+    <joint name="left_side_camera_joint" type="fixed">
+	    <parent link="trunk"/>
+	    <child link="left_side_camera_link"/>
+	    <origin rpy="-0.331612 0 0" xyz="-0.1086 0.1371 -0.03077"/>
+    </joint>
+    <link name="left_side_camera_link">
+        <inertial>
+            <mass value="0.001"/>
+            <origin rpy="0 0 0" xyz="0 0 0"/>
+            <inertia ixx="0.0001" ixy="0" ixz="0" iyy="0.0001" iyz="0" izz="0.0001"/>
+        </inertial>
+    </link>
+    <joint name="right_side_camera_joint" type="fixed">
+	    <parent link="trunk"/>
+	    <child link="right_side_camera_link"/>
+	    <origin rpy="0.331612 0 0" xyz="-0.10190 -0.1371 -0.03077"/>
+    </joint>
+    <link name="right_side_camera_link">
+        <inertial>
+            <mass value="0.001"/>
+            <origin rpy="0 0 0" xyz="0 0 0"/>
+            <inertia ixx="0.0001" ixy="0" ixz="0" iyy="0.0001" iyz="0" izz="0.0001"/>
+        </inertial>
+    </link>
+-
+    <joint name="head_camera_1_joint" type="fixed">
+	    <parent link="trunk"/>
+	    <child link="head_camera_1_link"/>
+	    <origin rpy="0 0 0" xyz="0.48883 0 0.0255"/>
+    </joint>
+    <link name="head_camera_1_link">
+        <inertial>
+            <mass value="0.001"/>
+            <origin rpy="0 0 0" xyz="0 0 0"/>
+            <inertia ixx="0.0001" ixy="0" ixz="0" iyy="0.0001" iyz="0" izz="0.0001"/>
+        </inertial>
+    </link>
+    <joint name="head_camera_2_joint" type="fixed">
+	    <parent link="trunk"/>
+	    <child link="head_camera_2_link"/>
+	    <origin rpy="0 0 0" xyz="0.45430 0 -0.081"/>
+    </joint>
+    <link name="head_camera_2_link">
+        <inertial>
+            <mass value="0.001"/>
+            <origin rpy="0 0 0" xyz="0 0 0"/>
+            <inertia ixx="0.0001" ixy="0" ixz="0" iyy="0.0001" iyz="0" izz="0.0001"/>
+        </inertial>
+    </link>
+    <joint name="tail_camera_joint" type="fixed">
+	    <parent link="trunk"/>
+	    <child link="tail_camera_link"/>
+	    <origin rpy="0 0 0" xyz="-0.459 0 -0.081"/>
+    </joint>
+    <link name="tail_camera_link">
+        <inertial>
+            <mass value="0.001"/>
+            <origin rpy="0 0 0" xyz="0 0 0"/>
+            <inertia ixx="0.0001" ixy="0" ixz="0" iyy="0.0001" iyz="0" izz="0.0001"/>
+        </inertial>
+    </link>
     <xacro:leg name="FR" mirror="-1" mirror_dae= "False" front_hind="1"  front_hind_dae="True"  />
     <xacro:leg name="FL" mirror="1"  mirror_dae="True"   front_hind="1"  front_hind_dae="True"  />

Commit message: Add xacro macro for B1

File: robots/b1_description/xacro/robot.xacro (robot description, xacro)
@@ -1,10 +1,7 @@
 <?xml version="1.0"?>
 <robot name="b1_description" xmlns:xacro="http://www.ros.org/wiki/xacro">
-    <xacro:include filename="$(find b1_description)/xacro/const.xacro"/>
-    <xacro:include filename="$(find b1_description)/xacro/materials.xacro"/>
-    <xacro:include filename="$(find b1_description)/xacro/leg.xacro"/>
+    <xacro:arg name="DEBUG" default="false"/>
+    <xacro:include filename="$(find b1_description)/xacro/b1.xacro"/>
     <xacro:include filename="$(find b1_description)/xacro/gazebo.xacro"/>
-    <!-- Rotor related joint and link is only for demonstrate location. -->
-    <!-- Actually, the rotor will rotate and the joint is not fixed. Reduction ratio should be considered. -->
     <!-- Debug mode will hung up the robot, use "true" or "false" to switch it. -->
     <xacro:if value="$(arg DEBUG)">
@@ -16,75 +13,5 @@
         </joint>
     </xacro:if>
-    <link name="base">
-        <visual>
-            <origin rpy="0 0 0" xyz="0 0 0"/>
-            <geometry>
-                <box size="0.001 0.001 0.001"/>
-            </geometry>
-        </visual>
-    </link>
-    <joint name="floating_base" type="fixed">
-        <origin rpy="0 0 0" xyz="0 0 0"/>
-        <parent link="base"/>
-        <child link="trunk"/>
-    </joint>
-    <link name="trunk">
-        <visual>
-            <origin rpy="0 0 0" xyz="0 0 0"/>
-            <geometry>
-                <mesh filename="package://b1_description/meshes/trunk.dae" scale="1 1 1"/>
-            </geometry>
-            <material name="orange"/>
-        </visual>
-        <collision>
-            <origin rpy="0 0 0" xyz="0 0 0"/>
-            <geometry>
-                <box size="${trunk_length} ${trunk_width} ${trunk_height}"/>
-            </geometry>
-        </collision>
-        <!-- <collision>
-            <origin rpy="0 0 0" xyz="0 0 0"/>
-            <geometry>
-                <mesh filename="package://b1_description/meshes/trunk.dae" scale="1 1 1"/>
-            </geometry>
-        </collision> -->
-        <inertial>
-            <origin rpy="0 0 0" xyz="${trunk_com_x} ${trunk_com_y} ${trunk_com_z}"/>
-            <mass value="${trunk_mass}"/>
-            <inertia
-                ixx="${trunk_ixx}" ixy="${trunk_ixy}" ixz="${trunk_ixz}"
-                iyy="${trunk_iyy}" iyz="${trunk_iyz}"
-                izz="${trunk_izz}"/>
-        </inertial>
-    </link>
-    <joint name="imu_joint" type="fixed">
-        <parent link="trunk"/>
-        <child link="imu_link"/>
-        <origin rpy="0 0 0" xyz="0 0 0"/>
-    </joint>
-    <link name="imu_link">
-        <inertial>
-            <mass value="0.001"/>
-            <origin rpy="0 0 0" xyz="0 0 0"/>
-            <inertia ixx="0.0001" ixy="0" ixz="0" iyy="0.0001" iyz="0" izz="0.0001"/>
-        </inertial>
-        <visual>
-            <origin rpy="0 0 0" xyz="0 0 0"/>
-            <geometry>
-                <box size="0.001 0.001 0.001"/>
-            </geometry>
-            <material name="red"/>
-        </visual>
-        <collision>
-            <origin rpy="0 0 0" xyz="0 0 0"/>
-            <geometry>
-                <box size=".001 .001 .001"/>
-            </geometry>
-        </collision>
-    </link>
-    <xacro:leg name="FR" mirror="-1" mirror_dae= "False" front_hind="1"  front_hind_dae="True"  />
-    <xacro:leg name="FL" mirror="1"  mirror_dae="True"   front_hind="1"  front_hind_dae="True"  />
-    <xacro:leg name="RR" mirror="-1" mirror_dae="False"  front_hind="-1" front_hind_dae="False" />
-    <xacro:leg name="RL" mirror="1"  mirror_dae="True"   front_hind="-1" front_hind_dae="False" />
+    <xacro:b1/>
     <!-- <xacro:stairs stairs="15" xpos="0" ypos="2.0" zpos="0" /> -->
 </robot>
