Commit message: add documentation

File: robots/b1_description/xacro/b1.xacro (robot description, xacro)
@@ -1,4 +1,5 @@
 <?xml version="1.0"?>
 <robot name="b1_description" xmlns:xacro="http://www.ros.org/wiki/xacro">
+    <!-- B1 macro: describes Unitree B1 quadruped robot -->
     <xacro:macro name="b1">
         <xacro:include filename="$(find b1_description)/xacro/const.xacro"/>

File: robots/b1_description/xacro/robot.xacro (robot description, xacro)
@@ -1,9 +1,15 @@
 <?xml version="1.0"?>
+<!-- b1_description: Unitree B1 quadruped robot -->
 <robot name="b1_description" xmlns:xacro="http://www.ros.org/wiki/xacro">
-    <xacro:arg name="DEBUG" default="false"/>
+    <!-- define arguments -->
+    <xacro:arg name="DEBUG" default="false"/> <!-- debug mode switch -->
+    <!-- include xacro files -->
     <xacro:include filename="$(find b1_description)/xacro/b1.xacro"/>
     <xacro:include filename="$(find b1_description)/xacro/gazebo.xacro"/>
-    <!-- Debug mode will hung up the robot, use "true" or "false" to switch it. -->
+    <!-- B1 macro: expands to describe B1 quadruped robot -->
+    <xacro:b1/>
+    <!-- debug mode configuration -->
     <xacro:if value="$(arg DEBUG)">
+        <!-- statically affix B1 base to world; i.e. "hang up" the robot -->
         <link name="world"/>
         <joint name="base_static_joint" type="fixed">
@@ -13,5 +19,3 @@
         </joint>
     </xacro:if>
-    <xacro:b1/>
-    <!-- <xacro:stairs stairs="15" xpos="0" ypos="2.0" zpos="0" /> -->
 </robot>

File: robots/b1z1_description/xacro/gazebo.xacro (robot description, xacro)
@@ -1,5 +1,6 @@
 <?xml version="1.0"?>
+<!-- Gazebo-specific elements for b1z1_description -->
 <robot>
-      <!-- ros_control plugin -->
+    <!-- ros_control plugin -->
     <gazebo>
         <plugin name="gazebo_ros_control" filename="libgazebo_ros_control.so">

File: robots/b1z1_description/xacro/robot.xacro (robot description, xacro)
@@ -10,5 +10,5 @@
     <xacro:include filename="$(find b1z1_description)/xacro/const.xacro"/>
     <xacro:include filename="$(find b1z1_description)/xacro/gazebo.xacro"/>
-    <!-- B1 macro: expands to describe B1 quadruped -->
+    <!-- B1 macro: expands to describe B1 quadruped robot -->
     <xacro:b1/>
     <!-- Z1 macro: expands to describe Z1 robotic arm -->
@@ -17,5 +17,6 @@
     <joint name="trunk_arm_joint" type="fixed">
         <!-- Z1 mounting point wrt B1 trunk; configurable in const.xacro -->
-        <origin rpy="${arm_offset_r} ${arm_offset_p} ${arm_offset_yaw}" xyz="${arm_offset_x} ${arm_offset_y} ${arm_offset_z}"/>
+        <origin rpy="${arm_offset_r} ${arm_offset_p} ${arm_offset_yaw}"
+            xyz="${arm_offset_x} ${arm_offset_y} ${arm_offset_z}"/>
         <!-- define parent and child links -->
         <parent link="trunk"/>
@@ -24,5 +25,5 @@
     <!-- debug mode configuration -->
     <xacro:if value="$(arg DEBUG)">
-        <!-- debug mode hangs up the robot; i.e., statically affixes B1 base to world -->
+        <!-- statically affix B1 base to world; i.e. "hang up" the robot -->
         <link name="world"/>
         <joint name="base_static_joint" type="fixed">

File: robots/z1_description/xacro/robot.xacro (robot description, xacro)
@@ -1,13 +1,20 @@
 <?xml version="1.0"?>
+<!-- z1_description: Unitree Z1 robotic arm -->
 <robot name="z1_description" xmlns:xacro="http://www.ros.org/wiki/xacro">
-    <xacro:arg name="UnitreeGripper" default="false"/>
+    <!-- define arguments -->
+    <xacro:arg name="UnitreeGripper" default="false"/> <!-- include default end-effector -->
+    <!-- include xacro files -->
     <xacro:include filename="$(find z1_description)/xacro/z1.xacro"/>
     <xacro:include filename="$(find z1_description)/xacro/gazebo.xacro"/>
+    <!-- Z1 macro: expands to describe Z1 robotic arm -->
+    <xacro:z1 UnitreeGripper="$(arg UnitreeGripper)"/>
+    <!-- define world link and statically affix Z1 -->
     <link name="world"/>
     <joint name="base_static_joint" type="fixed">
+        <!-- Z1 mounting point wrt origin (configurable) -->
         <origin rpy="0 0 0" xyz="0 0 0"/>
+        <!-- define parent and child links -->
         <parent link="world"/>
         <child link="link00"/>
     </joint>
-    <xacro:z1 UnitreeGripper="$(arg UnitreeGripper)"/>
 </robot>

File: robots/z1_description/xacro/z1.xacro (robot description, xacro)
@@ -1,4 +1,5 @@
 <?xml version="1.0"?>
 <robot name="z1_description" xmlns:xacro="http://www.ros.org/wiki/xacro">
+    <!-- Z1 macro: describes Unitree Z1 robotic arm -->
     <xacro:macro name="z1" params="UnitreeGripper:=false">
         <xacro:include filename="$(find z1_description)/xacro/const.xacro"/>
