Commit message: reconfirm Aliengo inertial params

File: robots/aliengo_description/urdf/aliengo.urdf (robot description, URDF)
Before this commit: robot aliengo, 19 links, 18 joints
Links:
- added link FL_calf_rotor, mass 0.132; collision cylinder length=0.02 radius=0.035; visual cylinder length=0.02 radius=0.035
- added link FL_hip_rotor, mass 0.146; collision cylinder length=0.02 radius=0.035; visual cylinder length=0.02 radius=0.035
- added link FL_thigh_rotor, mass 0.146; collision cylinder length=0.02 radius=0.035; visual cylinder length=0.02 radius=0.035
- added link FR_calf_rotor, mass 0.132; collision cylinder length=0.02 radius=0.035; visual cylinder length=0.02 radius=0.035
- added link FR_hip_rotor, mass 0.146; collision cylinder length=0.02 radius=0.035; visual cylinder length=0.02 radius=0.035
- added link FR_thigh_rotor, mass 0.146; collision cylinder length=0.02 radius=0.035; visual cylinder length=0.02 radius=0.035
- added link RL_calf_rotor, mass 0.132; collision cylinder length=0.02 radius=0.035; visual cylinder length=0.02 radius=0.035
- added link RL_hip_rotor, mass 0.146; collision cylinder length=0.02 radius=0.035; visual cylinder length=0.02 radius=0.035
- added link RL_thigh_rotor, mass 0.146; collision cylinder length=0.02 radius=0.035; visual cylinder length=0.02 radius=0.035
- added link RR_calf_rotor, mass 0.132; collision cylinder length=0.02 radius=0.035; visual cylinder length=0.02 radius=0.035
- added link RR_hip_rotor, mass 0.146; collision cylinder length=0.02 radius=0.035; visual cylinder length=0.02 radius=0.035
- added link RR_thigh_rotor, mass 0.146; collision cylinder length=0.02 radius=0.035; visual cylinder length=0.02 radius=0.035
- link trunk: mass 9.041 -> 11.644
Joints:
- added joint FL_calf_rotor_joint: type fixed, parent FL_thigh, child FL_calf_rotor, origin xyz=0.0 -0.0997 0 rpy=0 0 0
- added joint FL_hip_rotor_joint: type fixed, parent trunk, child FL_hip_rotor, origin xyz=0.139985 0.051 0 rpy=0 0 0
- added joint FL_thigh_rotor_joint: type fixed, parent FL_hip, child FL_thigh_rotor, origin xyz=0.0 0.0298 0 rpy=0 0 0
- added joint FR_calf_rotor_joint: type fixed, parent FR_thigh, child FR_calf_rotor, origin xyz=0.0 0.0997 0 rpy=0 0 0
- added joint FR_hip_rotor_joint: type fixed, parent trunk, child FR_hip_rotor, origin xyz=0.139985 -0.051 0 rpy=0 0 0
- added joint FR_thigh_rotor_joint: type fixed, parent FR_hip, child FR_thigh_rotor, origin xyz=0.0 -0.0298 0 rpy=0 0 0
- added joint RL_calf_rotor_joint: type fixed, parent RL_thigh, child RL_calf_rotor, origin xyz=0.0 -0.0997 0 rpy=0 0 0
- added joint RL_hip_rotor_joint: type fixed, parent trunk, child RL_hip_rotor, origin xyz=-0.139985 0.051 0 rpy=0 0 0
- added joint RL_thigh_rotor_joint: type fixed, parent RL_hip, child RL_thigh_rotor, origin xyz=0.0 0.0298 0 rpy=0 0 0
- added joint RR_calf_rotor_joint: type fixed, parent RR_thigh, child RR_calf_rotor, origin xyz=0.0 0.0997 0 rpy=0 0 0
- added joint RR_hip_rotor_joint: type fixed, parent trunk, child RR_hip_rotor, origin xyz=-0.139985 -0.051 0 rpy=0 0 0
- added joint RR_thigh_rotor_joint: type fixed, parent RR_hip, child RR_thigh_rotor, origin xyz=0.0 -0.0298 0 rpy=0 0 0
- joint FL_calf_joint: limit lower=-2.77507351067 upper=-0.645771823238 effort=55 velocity=16 -> lower=-2.775073510670984 upper=-0.6457718232379019 effort=44.4 velocity=15.89
- joint FL_hip_joint: limit lower=-1.2217304764 upper=1.2217304764 effort=44 velocity=20 -> lower=-1.2217304763960306 upper=1.2217304763960306 effort=35.278 velocity=20; origin xyz=0.2399 0.051 0 rpy=0 0 0 -> xyz=0.2407 0.051 0 rpy=0 0 0
- joint FL_thigh_joint: limit effort=44 velocity=20 -> effort=35.278 velocity=20; origin xyz=0 0.083 0 rpy=0 0 0 -> xyz=0 0.0868 0 rpy=0 0 0
- joint FR_calf_joint: limit lower=-2.77507351067 upper=-0.645771823238 effort=55 velocity=16 -> lower=-2.775073510670984 upper=-0.6457718232379019 effort=44.4 velocity=15.89
- joint FR_hip_joint: limit lower=-1.2217304764 upper=1.2217304764 effort=44 velocity=20 -> lower=-1.2217304763960306 upper=1.2217304763960306 effort=35.278 velocity=20; origin xyz=0.2399 -0.051 0 rpy=0 0 0 -> xyz=0.2407 -0.051 0 rpy=0 0 0
- joint FR_thigh_joint: limit effort=44 velocity=20 -> effort=35.278 velocity=20; origin xyz=0 -0.083 0 rpy=0 0 0 -> xyz=0 -0.0868 0 rpy=0 0 0
- joint RL_calf_joint: limit lower=-2.77507351067 upper=-0.645771823238 effort=55 velocity=16 -> lower=-2.775073510670984 upper=-0.6457718232379019 effort=44.4 velocity=15.89
- joint RL_hip_joint: limit lower=-1.2217304764 upper=1.2217304764 effort=44 velocity=20 -> lower=-1.2217304763960306 upper=1.2217304763960306 effort=35.278 velocity=20; origin xyz=-0.2399 0.051 0 rpy=0 0 0 -> xyz=-0.2407 0.051 0 rpy=0 0 0
- joint RL_thigh_joint: limit effort=44 velocity=20 -> effort=35.278 velocity=20; origin xyz=0 0.083 0 rpy=0 0 0 -> xyz=0 0.0868 0 rpy=0 0 0
- joint RR_calf_joint: limit lower=-2.77507351067 upper=-0.645771823238 effort=55 velocity=16 -> lower=-2.775073510670984 upper=-0.6457718232379019 effort=44.4 velocity=15.89
- joint RR_hip_joint: limit lower=-1.2217304764 upper=1.2217304764 effort=44 velocity=20 -> lower=-1.2217304763960306 upper=1.2217304763960306 effort=35.278 velocity=20; origin xyz=-0.2399 -0.051 0 rpy=0 0 0 -> xyz=-0.2407 -0.051 0 rpy=0 0 0
- joint RR_thigh_joint: limit effort=44 velocity=20 -> effort=35.278 velocity=20; origin xyz=0 -0.083 0 rpy=0 0 0 -> xyz=0 -0.0868 0 rpy=0 0 0

File: robots/aliengo_description/xacro/const.xacro (robot description, xacro)
@@ -28,4 +28,23 @@
     <xacro:property name="trunk_offset_z" value="0.01675"/>
     <xacro:property name="hip_offset" value="0.083"/>
+    <!-- offset of link and rotor locations (left front) -->
+    <xacro:property name="hip_offset_x" value="0.2407"/>
+    <xacro:property name="hip_offset_y" value="0.051"/>
+    <xacro:property name="hip_offset_z" value="0.0"/>
+    <xacro:property name="hip_rotor_offset_x" value="0.139985"/>
+    <xacro:property name="hip_rotor_offset_y" value="0.051"/>
+    <xacro:property name="hip_rotor_offset_z" value="0.0"/>
+    <xacro:property name="thigh_offset_x" value="0"/>
+    <xacro:property name="thigh_offset_y" value="0.0868"/>
+    <xacro:property name="thigh_offset_z" value="0.0"/>
+    <xacro:property name="thigh_rotor_offset_x" value="0.0"/>
+    <xacro:property name="thigh_rotor_offset_y" value="0.0298"/>
+    <xacro:property name="thigh_rotor_offset_z" value="0.0"/>
+    <xacro:property name="calf_offset_x" value="0.0"/>
+    <xacro:property name="calf_offset_y" value="0.0"/>
+    <xacro:property name="calf_offset_z" value="-0.25"/>
+    <xacro:property name="calf_rotor_offset_x" value="0.0"/>
+    <xacro:property name="calf_rotor_offset_y" value="-0.0997"/>
+    <xacro:property name="calf_rotor_offset_z" value="0.0"/>
     <!-- joint limits -->
     <xacro:property name="damping" value="0"/>
@@ -43,16 +62,16 @@
     <xacro:property name="calf_velocity_max" value="15.89"/>
     <xacro:property name="calf_torque_max" value="44.4"/>
-    <!-- dynamics inertial value        total 22.0kg -->
+    <!-- dynamics inertial value        total 23.0kg -->
     <!-- trunk -->
-    <xacro:property name="trunk_mass" value="11.041"/>
-    <xacro:property name="trunk_com_x" value="0.008465"/>
-    <xacro:property name="trunk_com_y" value="0.004045"/>
-    <xacro:property name="trunk_com_z" value="-0.000763"/>
-    <xacro:property name="trunk_ixx" value="0.050874"/>
-    <xacro:property name="trunk_ixy" value="-0.000451628"/>
-    <xacro:property name="trunk_ixz" value="0.000487603"/>
-    <xacro:property name="trunk_iyy" value="0.64036"/>
-    <xacro:property name="trunk_iyz" value="0.000048356"/>
-    <xacro:property name="trunk_izz" value="0.65655"/>
+    <xacro:property name="trunk_mass" value="11.644"/>
+    <xacro:property name="trunk_com_x" value="0.008811"/>
+    <xacro:property name="trunk_com_y" value="0.003839"/>
+    <xacro:property name="trunk_com_z" value="0.000273"/>
+    <xacro:property name="trunk_ixx" value="0.051944892"/>
+    <xacro:property name="trunk_ixy" value="0.001703617"/>
+    <xacro:property name="trunk_ixz" value="0.000235941"/>
+    <xacro:property name="trunk_iyy" value="0.24693924"/>
+    <xacro:property name="trunk_iyz" value="0.000119783"/>
+    <xacro:property name="trunk_izz" value="0.270948307"/>
     <!-- hip (left front) -->
     <xacro:property name="hip_mass" value="1.993"/>
@@ -60,10 +79,20 @@
     <xacro:property name="hip_com_y" value="0.015144"/>
     <xacro:property name="hip_com_z" value="-0.000015"/>
-    <xacro:property name="hip_ixx" value="0.002903894"/>
-    <xacro:property name="hip_ixy" value="-0.000071850"/>
-    <xacro:property name="hip_ixz" value="-0.000001262"/>
-    <xacro:property name="hip_iyy" value="0.004907517"/>
-    <xacro:property name="hip_iyz" value="-0.00000175"/>
-    <xacro:property name="hip_izz" value="0.005586944"/>
+    <xacro:property name="hip_ixx" value="0.002446735"/>
+    <xacro:property name="hip_ixy" value="-0.00059805"/>
+    <xacro:property name="hip_ixz" value="0.000001945"/>
+    <xacro:property name="hip_iyy" value="0.003925876"/>
+    <xacro:property name="hip_iyz" value="0.000001284"/>
+    <xacro:property name="hip_izz" value="0.004148145"/>
+    <xacro:property name="hip_rotor_mass" value="0.146"/>
+    <xacro:property name="hip_rotor_com_x" value="0.0"/>
+    <xacro:property name="hip_rotor_com_y" value="0.0"/>
+    <xacro:property name="hip_rotor_com_z" value="0.0"/>
+    <xacro:property name="hip_rotor_ixx" value="0.000138702"/>
+    <xacro:property name="hip_rotor_ixy" value="0.0"/>
+    <xacro:property name="hip_rotor_ixz" value="0.0"/>
+    <xacro:property name="hip_rotor_iyy" value="0.000083352"/>
+    <xacro:property name="hip_rotor_iyz" value="0.0"/>
+    <xacro:property name="hip_rotor_izz" value="0.000083352"/>
     <!-- thigh -->
     <xacro:property name="thigh_mass" value="0.639"/>
@@ -71,10 +100,20 @@
     <xacro:property name="thigh_com_y" value="-0.003877"/>
     <xacro:property name="thigh_com_z" value="-0.048199"/>
-    <xacro:property name="thigh_ixx" value="0.005666803"/>
-    <xacro:property name="thigh_ixy" value="0.000003597"/>
-    <xacro:property name="thigh_ixz" value="0.000491446"/>
-    <xacro:property name="thigh_iyy" value="0.005847229"/>
-    <xacro:property name="thigh_iyz" value="0.000010086"/>
-    <xacro:property name="thigh_izz" value="0.000369811"/>
+    <xacro:property name="thigh_ixx" value="0.004173855"/>
+    <xacro:property name="thigh_ixy" value="0.000010284"/>
+    <xacro:property name="thigh_ixz" value="-0.000318874"/>
+    <xacro:property name="thigh_iyy" value="0.004343802"/>
+    <xacro:property name="thigh_iyz" value="0.000109233"/>
+    <xacro:property name="thigh_izz" value="0.000340136"/>
+    <xacro:property name="thigh_rotor_mass" value="0.146"/>
+    <xacro:property name="thigh_rotor_com_x" value="0.0"/>
+    <xacro:property name="thigh_rotor_com_y" value="0.0"/>
+    <xacro:property name="thigh_rotor_com_z" value="0.0"/>
+    <xacro:property name="thigh_rotor_ixx" value="0.000083352"/>
+    <xacro:property name="thigh_rotor_ixy" value="0.0"/>
+    <xacro:property name="thigh_rotor_ixz" value="0.0"/>
+    <xacro:property name="thigh_rotor_iyy" value="0.000138702"/>
+    <xacro:property name="thigh_rotor_iyz" value="0.0"/>
+    <xacro:property name="thigh_rotor_izz" value="0.000083352"/>
     <!-- calf -->
     <xacro:property name="calf_mass" value="0.207"/>
@@ -82,10 +121,20 @@
     <xacro:property name="calf_com_y" value="0.000063"/>
     <xacro:property name="calf_com_z" value="-0.142518"/>
-    <xacro:property name="calf_ixx" value="0.006341369"/>
-    <xacro:property name="calf_ixy" value="-0.000000003"/>
-    <xacro:property name="calf_ixz" value="-0.000087951"/>
-    <xacro:property name="calf_iyy" value="0.006355157"/>
-    <xacro:property name="calf_iyz" value="-0.000001336"/>
-    <xacro:property name="calf_izz" value="0.000039188"/>
+    <xacro:property name="calf_ixx" value="0.002129279"/>
+    <xacro:property name="calf_ixy" value="0.000000039"/>
+    <xacro:property name="calf_ixz" value="0.000005757"/>
+    <xacro:property name="calf_iyy" value="0.002141463"/>
+    <xacro:property name="calf_iyz" value="-0.000000516"/>
+    <xacro:property name="calf_izz" value="0.000037583"/>
+    <xacro:property name="calf_rotor_mass" value="0.132"/>
+    <xacro:property name="calf_rotor_com_x" value="0.0"/>
+    <xacro:property name="calf_rotor_com_y" value="0.0"/>
+    <xacro:property name="calf_rotor_com_z" value="0.0"/>
+    <xacro:property name="calf_rotor_ixx" value="0.000145463"/>
+    <xacro:property name="calf_rotor_ixy" value="0.0"/>
+    <xacro:property name="calf_rotor_ixz" value="0.0"/>
+    <xacro:property name="calf_rotor_iyy" value="0.000133031"/>
+    <xacro:property name="calf_rotor_iyz" value="0.0"/>
+    <xacro:property name="calf_rotor_izz" value="0.000145463"/>
     <!-- foot -->
     <xacro:property name="foot_mass" value="0.06"/>

File: robots/aliengo_description/xacro/leg.xacro (robot description, xacro)
@@ -2,7 +2,18 @@
 <robot xmlns:xacro="http://www.ros.org/wiki/xacro">
     <xacro:include filename="$(find aliengo_description)/xacro/transmission.xacro"/>
-    <xacro:macro name="leg" params="name mirror mirror_dae front_hind front_hind_dae *origin">
+    <xacro:macro name="leg" params="name mirror mirror_dae front_hind front_hind_dae">
         <joint name="${name}_hip_joint" type="revolute">
-            <xacro:insert_block name="origin"/>
+            <xacro:if value="${(mirror_dae == False) and (front_hind_dae == True)}">
+                <origin rpy="0 0 0" xyz="${leg_offset_x} ${-leg_offset_y} 0"/>
+            </xacro:if>
+            <xacro:if value="${(mirror_dae == True) and (front_hind_dae == True)}">
+                <origin rpy="0 0 0" xyz="${leg_offset_x} ${leg_offset_y} 0"/>
+            </xacro:if>
+            <xacro:if value="${(mirror_dae == False) and (front_hind_dae == False)}">
+                <origin rpy="0 0 0" xyz="${-leg_offset_x} ${-leg_offset_y} 0"/>
+            </xacro:if>
+            <xacro:if value="${(mirror_dae == True) and (front_hind_dae == False)}">
+                <origin rpy="0 0 0" xyz="${-leg_offset_x} ${leg_offset_y} 0"/>
+            </xacro:if>
             <parent link="trunk"/>
             <child link="${name}_hip"/>
@@ -16,4 +27,20 @@
             </xacro:if>
         </joint>
+        <joint name="${name}_hip_rotor_joint" type="fixed">
+            <xacro:if value="${(mirror_dae == False) and (front_hind_dae == True)}">
+                <origin rpy="0 0 0" xyz="${hip_rotor_offset_x} ${-hip_rotor_offset_y} 0"/>
+            </xacro:if>
+            <xacro:if value="${(mirror_dae == True) and (front_hind_dae == True)}">
+                <origin rpy="0 0 0" xyz="${hip_rotor_offset_x} ${hip_rotor_offset_y} 0"/>
+            </xacro:if>
+            <xacro:if value="${(mirror_dae == False) and (front_hind_dae == False)}">
+                <origin rpy="0 0 0" xyz="${-hip_rotor_offset_x} ${-hip_rotor_offset_y} 0"/>
+            </xacro:if>
+            <xacro:if value="${(mirror_dae == True) and (front_hind_dae == False)}">
+                <origin rpy="0 0 0" xyz="${-hip_rotor_offset_x} ${hip_rotor_offset_y} 0"/>
+            </xacro:if>
+            <parent link="trunk"/>
+            <child link="${name}_hip_rotor"/>
+        </joint>
         <link name="${name}_hip">
             <visual>
@@ -50,18 +77,27 @@
             </inertial>
         </link>
-        <!-- <joint name="${name}_hip_fixed" type="fixed">
-            <origin rpy="0 0 0" xyz="0 ${(thigh_shoulder_length/2.0+hip_offset)*mirror} 0"/>
-            <parent link="${name}_hip"/>
-            <child link="${name}_thigh_shoulder"/>
-        </joint> -->
-        <!-- this link is only for collision -->
-        <!-- <link name="${name}_thigh_shoulder">
-            <collision>
-                <origin rpy="${PI/2.0} 0 0" xyz="0 0 0"/>
-                <geometry>
-                    <cylinder length="${thigh_shoulder_length}" radius="${thigh_shoulder_radius}"/>
-                </geometry>
-            </collision>
-        </link> -->
+        <link name="${name}_hip_rotor">
+            <visual>
+                <origin rpy="0 ${PI/2.0} 0" xyz="0 0 0"/>
+                <geometry>
+                    <cylinder length="0.02" radius="0.035"/>
+                </geometry>
+                <material name="green"/>
+            </visual>
+            <collision>
+                <origin rpy="0 ${PI/2.0} 0" xyz="0 0 0"/>
+                <geometry>
+                    <cylinder length="0.02" radius="0.035"/>
+                </geometry>
+            </collision>
+            <inertial>
+                <origin rpy="0 0 0" xyz="${hip_rotor_com_x} ${hip_rotor_com_y} ${hip_rotor_com_z}"/>
+                <mass value="${hip_rotor_mass}"/>
+                <inertia
+                    ixx="${hip_rotor_ixx}" ixy="${hip_rotor_ixy}" ixz="${hip_rotor_ixz}"
+                    iyy="${hip_rotor_iyy}" iyz="${hip_rotor_iyz}"
+                    izz="${hip_rotor_izz}"/>
+            </inertial>
+        </link>
         <joint name="${name}_thigh_joint" type="continuous">
             <origin rpy="0 0 0" xyz="0 ${thigh_offset*mirror} 0"/>
@@ -72,4 +108,9 @@
             <limit effort="${thigh_torque_max}" velocity="${thigh_velocity_max}"/>
         </joint>
+        <joint name="${name}_thigh_rotor_joint" type="fixed">
+            <origin rpy="0 0 0" xyz="${thigh_rotor_offset_x} ${thigh_rotor_offset_y*mirror} 0"/>
+            <parent link="${name}_hip"/>
+            <child link="${name}_thigh_rotor"/>
+        </joint>
         <link name="${name}_thigh">
             <visual>
@@ -98,4 +139,27 @@
                     iyy="${thigh_iyy}" iyz="${thigh_iyz*mirror}"
                     izz="${thigh_izz}"/>
+            </inertial>
+        </link>
+        <link name="${name}_thigh_rotor">
+            <visual>
+                <origin rpy="${PI/2.0} 0 0" xyz="0 0 0"/>
+                <geometry>
+                    <cylinder length="0.02" radius="0.035"/>
+                </geometry>
+                <material name="green"/>
+            </visual>
+            <collision>
+                <origin rpy="${PI/2.0} 0 0" xyz="0 0 0"/>
+                <geometry>
+                    <cylinder length="0.02" radius="0.035"/>
+                </geometry>
+            </collision>
+            <inertial>
+                <origin rpy="0 0 0" xyz="${thigh_rotor_com_x} ${thigh_rotor_com_y} ${thigh_rotor_com_z}"/>
+                <mass value="${thigh_rotor_mass}"/>
+                <inertia
+                    ixx="${thigh_rotor_ixx}" ixy="${thigh_rotor_ixy}" ixz="${thigh_rotor_ixz}"
+                    iyy="${thigh_rotor_iyy}" iyz="${thigh_rotor_iyz}"
+                    izz="${thigh_rotor_izz}"/>
             </inertial>
         </link>
@@ -108,4 +172,9 @@
             <limit effort="${calf_torque_max}" velocity="${calf_velocity_max}" lower="${calf_position_min}" upper="${calf_position_max}"/>
         </joint>
+        <joint name="${name}_calf_rotor_joint" type="fixed">
+            <origin rpy="0 0 0" xyz="${calf_rotor_offset_x} ${calf_rotor_offset_y*mirror} 0"/>
+            <parent link="${name}_thigh"/>
+            <child link="${name}_calf_rotor"/>
+        </joint>
         <link name="${name}_calf">
             <visual>
@@ -129,4 +198,27 @@
                     iyy="${calf_iyy}" iyz="${calf_iyz}"
                     izz="${calf_izz}"/>
+            </inertial>
+        </link>
+        <link name="${name}_calf_rotor">
+            <visual>
+                <origin rpy="${PI/2.0} 0 0" xyz="0 0 0"/>
+                <geometry>
+                    <cylinder length="0.02" radius="0.035"/>
+                </geometry>
+                <material name="green"/>
+            </visual>
+            <collision>
+                <origin rpy="${PI/2.0} 0 0" xyz="0 0 0"/>
+                <geometry>
+                    <cylinder length="0.02" radius="0.035"/>
+                </geometry>
+            </collision>
+            <inertial>
+                <origin rpy="0 0 0" xyz="${calf_rotor_com_x} ${calf_rotor_com_y} ${calf_rotor_com_z}"/>
+                <mass value="${calf_rotor_mass}"/>
+                <inertia
+                    ixx="${calf_rotor_ixx}" ixy="${calf_rotor_ixy}" ixz="${calf_rotor_ixz}"
+                    iyy="${calf_rotor_iyy}" iyz="${calf_rotor_iyz}"
+                    izz="${calf_rotor_izz}"/>
             </inertial>
         </link>
