Commit message: update aliengoZ1_description based on new version of aliengo_description

File: robots/aliengoZ1_description/xacro/robot.xacro (robot description, xacro)
@@ -106,5 +106,5 @@
         </inertial>
     </link>
-    <joint name="joint1" type="revolute">
+   <joint name="joint1" type="revolute">
         <origin rpy="0 0 0" xyz="0 0 0.0585"/>
         <parent link="link00"/>
@@ -121,10 +121,10 @@
             </geometry>
         </visual>
-        <!-- <collision>
+        <collision>
             <geometry>
                 <cylinder length="${2*motor_height}" radius="${motor_diameter}"/>
             </geometry>
             <origin rpy="0 0 0" xyz="0 0 0"/>
-        </collision> -->
+        </collision>
         <inertial>
             <origin rpy="0 0 0" xyz="${L01_ComX} ${L01_ComY} ${L01_ComZ}"/>
@@ -366,15 +366,7 @@
     <xacro:motorTransmission name="5"/>
     <xacro:motorTransmission name="6"/>
-    <xacro:leg name="FR" mirror="-1" mirror_dae= "False" front_hind="1" front_hind_dae="True">
-        <origin rpy="0 0 0" xyz="${leg_offset_x} ${-leg_offset_y} 0"/>
-    </xacro:leg>
-    <xacro:leg name="FL" mirror="1" mirror_dae="True" front_hind="1" front_hind_dae="True">
-        <origin rpy="0 0 0" xyz="${leg_offset_x} ${leg_offset_y} 0"/>
-    </xacro:leg>
-    <xacro:leg name="RR" mirror="-1" mirror_dae="False" front_hind="-1" front_hind_dae="False">
-        <origin rpy="0 0 0" xyz="${-leg_offset_x} ${-leg_offset_y} 0"/>
-    </xacro:leg>
-    <xacro:leg name="RL" mirror="1" mirror_dae="True" front_hind="-1" front_hind_dae="False">
-        <origin rpy="0 0 0" xyz="${-leg_offset_x} ${leg_offset_y} 0"/>
-    </xacro:leg>
+    <xacro:leg name="FR" mirror="-1" mirror_dae= "False" front_hind="1"  front_hind_dae="True"  />
+    <xacro:leg name="FL" mirror="1"  mirror_dae="True"   front_hind="1"  front_hind_dae="True"  />
+    <xacro:leg name="RR" mirror="-1" mirror_dae="False"  front_hind="-1" front_hind_dae="False" />
+    <xacro:leg name="RL" mirror="1"  mirror_dae="True"   front_hind="-1" front_hind_dae="False" />
 </robot>

Commit message: modify z1_urdf

File: robots/aliengoZ1_description/xacro/robot.xacro (robot description, xacro)
@@ -203,5 +203,5 @@
                 <cylinder length="0.059" radius="${motor_diameter}"/>
             </geometry>
-            <origin rpy="0 ${PI/2.0} 0" xyz="${0.065+0.185-0.059/2.0} 0 0.055"/>
+            <origin rpy="0 ${PI/2.0} ${PI/2.0}" xyz="${0.065+0.185-0.059/2.0} 0 0.055"/>
         </collision>
         <inertial>
@@ -231,7 +231,7 @@
         <collision>
             <geometry>
-                <cylinder length="0.073" radius="${motor_diameter}"/>
-            </geometry>
-            <origin rpy="${PI/2.0} 0 0" xyz="0.0472 0 0"/>
+                <cylinder length="${motor_height + 2*0.008}" radius="${motor_diameter}"/>
+            </geometry>
+            <origin rpy="0 0 0" xyz="0.072 0 0"/>
         </collision>
         <inertial>

File: robots/z1_description/xacro/const.xacro (robot description, xacro)
@@ -103,20 +103,18 @@
     <xacro:property name="GripperMover_Izz" value="0.00035728"/>
     <!-- joint limits -->
-    <!-- <xacro:property name="jointDamping" value="3.0"/> -->
-    <!-- <xacro:property name="jointFriction" value="2.0"/> -->
     <xacro:property name="jointDamping" value="1.0"/>
     <xacro:property name="jointFriction" value="1.0"/>
     <xacro:property name="torqueMax" value="30.0"/>
-    <xacro:property name="velocityMax" value="10"/>
+    <xacro:property name="velocityMax" value="3.1415"/>
     <xacro:property name="joint1_PositionMin" value="${-PI*150/180}"/>
     <xacro:property name="joint1_PositionMax" value="${PI*150/180}"/>
     <xacro:property name="joint2_PositionMin" value="0.0"/>
-    <xacro:property name="joint2_PositionMax" value="${PI}"/>
-    <xacro:property name="joint3_PositionMin" value="${-PI*274/180}"/>
+    <xacro:property name="joint2_PositionMax" value="${PI*170/180}"/>
+    <xacro:property name="joint3_PositionMin" value="${-PI*165/180}"/>
     <xacro:property name="joint3_PositionMax" value="0.0"/>
-    <xacro:property name="joint4_PositionMin" value="${-PI*100/180}"/>
-    <xacro:property name="joint4_PositionMax" value="${PI*90/180}"/>
-    <xacro:property name="joint5_PositionMin" value="${-PI*99/180}"/>
-    <xacro:property name="joint5_PositionMax" value="${PI*99/180}"/>
+    <xacro:property name="joint4_PositionMin" value="${-PI*87/180}"/>
+    <xacro:property name="joint4_PositionMax" value="${PI*87/180}"/>
+    <xacro:property name="joint5_PositionMin" value="${-PI*77/180}"/>
+    <xacro:property name="joint5_PositionMax" value="${PI*77/180}"/>
     <xacro:property name="joint6_PositionMin" value="${-PI*160/180}"/>
     <xacro:property name="joint6_PositionMax" value="${PI*160/180}"/>

File: robots/z1_description/xacro/robot.xacro (robot description, xacro)
@@ -48,10 +48,4 @@
             </geometry>
         </visual>
-        <!-- <collision>
-            <geometry>
-                <cylinder length="${2*motor_height}" radius="${motor_diameter}"/>
-            </geometry>
-            <origin rpy="0 0 0" xyz="0 0 0"/>
-        </collision> -->
         <inertial>
             <origin rpy="0 0 0" xyz="${L01_ComX} ${L01_ComY} ${L01_ComZ}"/>
@@ -130,5 +124,5 @@
                 <cylinder length="0.059" radius="${motor_diameter}"/>
             </geometry>
-            <origin rpy="0 ${PI/2.0} 0" xyz="${0.065+0.185-0.059/2.0} 0 0.055"/>
+            <origin rpy="0 ${PI/2.0} ${PI/2.0}" xyz="${0.065+0.185-0.059/2.0} 0 0.055"/>
         </collision>
         <inertial>
@@ -158,7 +152,7 @@
         <collision>
             <geometry>
-                <cylinder length="0.073" radius="${motor_diameter}"/>
-            </geometry>
-            <origin rpy="${PI/2.0} 0 0" xyz="0.0472 0 0"/>
+                <cylinder length="${motor_height + 2*0.008}" radius="${motor_diameter}"/>
+            </geometry>
+            <origin rpy="0 0 0" xyz="0.072 0 0"/>
         </collision>
         <inertial>

File: robots/z1_description/xacro/z1.urdf (robot description, URDF)
Before this commit: robot z1_description, 8 links, 7 joints
Links:
- link link00: geometry collision cylinder length=0.051 radius=0.0325; visual mesh filename=package://z1_description/meshes/visual/z1_Link00.dae scale=1 1 1
- link link01: geometry visual mesh filename=package://z1_description/meshes/visual/z1_Link01.dae scale=1 1 1
- link link02: geometry collision cylinder length=0.051 radius=0.0325; collision cylinder length=0.102 radius=0.0325
- link link03: geometry collision cylinder length=0.059 radius=0.0325; collision cylinder length=0.116 radius=0.02
- link link04: geometry collision cylinder length=0.067 radius=0.0325; visual mesh filename=package://z1_description/meshes/visual/z1_Link04.dae scale=1 1 1
- link link05: geometry visual mesh filename=package://z1_description/meshes/visual/z1_Link05.dae scale=1 1 1
- link link06: geometry collision cylinder length=0.051 radius=0.0325; visual mesh filename=package://z1_description/meshes/visual/z1_Link06.dae scale=1 1 1
Joints:
- joint joint2: limit lower=0.0 upper=3.141592653589793 effort=60.0 velocity=10 -> lower=0.0 upper=2.9670597283903604 effort=60.0 velocity=10
- joint joint3: limit lower=-4.782202150464463 upper=0.0 effort=30.0 velocity=10 -> lower=-2.8797932657906435 upper=0.0 effort=30.0 velocity=10
- joint joint4: limit lower=-1.7453292519943295 upper=1.5707963267948966 effort=30.0 velocity=10 -> lower=-1.5184364492350666 upper=1.5184364492350666 effort=30.0 velocity=10
- joint joint5: limit lower=-1.7278759594743864 upper=1.7278759594743864 effort=30.0 velocity=10 -> lower=-1.3439035240356338 upper=1.3439035240356338 effort=30.0 velocity=10
