Commit message: Fix Z1 inertia error

File: robots/z1_description/xacro/const.xacro (robot description, xacro)
@@ -9,8 +9,8 @@
     <xacro:property name="L00_ComZ" value="0.02495843"/>
     <xacro:property name="L00_Ixx" value="0.00037937"/>
-    <xacro:property name="L00_Ixy" value="0.00000035"/>
-    <xacro:property name="L00_Ixz" value="0.00001037"/>
+    <xacro:property name="L00_Ixy" value="-0.00000035"/>
+    <xacro:property name="L00_Ixz" value="-0.00001037"/>
     <xacro:property name="L00_Iyy" value="0.00041521"/>
-    <xacro:property name="L00_Iyz" value="0.00000099"/>
+    <xacro:property name="L00_Iyz" value="-0.00000099"/>
     <xacro:property name="L00_Izz" value="0.00053066"/>
     <!-- Link 01 -->
@@ -20,8 +20,8 @@
     <xacro:property name="L01_ComZ" value="0.02317169"/>
     <xacro:property name="L01_Ixx" value="0.00128328"/>
-    <xacro:property name="L01_Ixy" value="0.00000006"/>
-    <xacro:property name="L01_Ixz" value="0.00000040"/>
+    <xacro:property name="L01_Ixy" value="-0.00000006"/>
+    <xacro:property name="L01_Ixz" value="-0.00000040"/>
     <xacro:property name="L01_Iyy" value="0.00071931"/>
-    <xacro:property name="L01_Iyz" value="-0.00000050"/>
+    <xacro:property name="L01_Iyz" value="0.00000050"/>
     <xacro:property name="L01_Izz" value="0.00083936"/>
     <!-- Link 02 -->
@@ -31,8 +31,8 @@
     <xacro:property name="L02_ComZ" value="0.00158266"/>
     <xacro:property name="L02_Ixx" value="0.00102138"/>
-    <xacro:property name="L02_Ixy" value="-0.00062358"/>
-    <xacro:property name="L02_Ixz" value="-0.00000513"/>
+    <xacro:property name="L02_Ixy" value="0.00062358"/>
+    <xacro:property name="L02_Ixz" value="0.00000513"/>
     <xacro:property name="L02_Iyy" value="0.02429457"/>
-    <xacro:property name="L02_Iyz" value="0.00000210"/>
+    <xacro:property name="L02_Iyz" value="-0.00000210"/>
     <xacro:property name="L02_Izz" value="0.02466114"/>
     <!-- Link 03 -->
@@ -42,8 +42,8 @@
     <xacro:property name="L03_ComZ" value="0.03476383"/>
     <xacro:property name="L03_Ixx" value="0.00108061"/>
-    <xacro:property name="L03_Ixy" value="0.00008669"/>
-    <xacro:property name="L03_Ixz" value="0.00208102"/>
+    <xacro:property name="L03_Ixy" value="-0.00008669"/>
+    <xacro:property name="L03_Ixz" value="-0.00208102"/>
     <xacro:property name="L03_Iyy" value="0.00954238"/>
-    <xacro:property name="L03_Iyz" value="0.00001332"/>
+    <xacro:property name="L03_Iyz" value="-0.00001332"/>
     <xacro:property name="L03_Izz" value="0.00886621"/>
     <!-- Link 04 -->
@@ -53,8 +53,8 @@
     <xacro:property name="L04_ComZ" value="-0.00170192"/>
     <xacro:property name="L04_Ixx" value="0.00031576"/>
-    <xacro:property name="L04_Ixy" value="-0.00008130"/>
-    <xacro:property name="L04_Ixz" value="-0.00004091"/>
+    <xacro:property name="L04_Ixy" value="0.00008130"/>
+    <xacro:property name="L04_Ixz" value="0.00004091"/>
     <xacro:property name="L04_Iyy" value="0.00092996"/>
-    <xacro:property name="L04_Iyz" value="0.00000596"/>
+    <xacro:property name="L04_Iyz" value="-0.00000596"/>
     <xacro:property name="L04_Izz" value="0.00097912"/>
     <!-- Link 05 -->
@@ -64,8 +64,8 @@
     <xacro:property name="L05_ComZ" value="0.00646316"/>
     <xacro:property name="L05_Ixx" value="0.00017605"/>
-    <xacro:property name="L05_Ixy" value="-0.00000040"/>
-    <xacro:property name="L05_Ixz" value="-0.00005689"/>
+    <xacro:property name="L05_Ixy" value="0.00000040"/>
+    <xacro:property name="L05_Ixz" value="0.00005689"/>
     <xacro:property name="L05_Iyy" value="0.00055896"/>
-    <xacro:property name="L05_Iyz" value="0.00000013"/>
+    <xacro:property name="L05_Iyz" value="-0.00000013"/>
     <xacro:property name="L05_Izz" value="0.00053860"/>
     <!-- Link 06 -->
@@ -75,8 +75,8 @@
     <xacro:property name="L06_ComZ" value="-0.00143876"/>
     <xacro:property name="L06_Ixx" value="0.00018328"/>
-    <xacro:property name="L06_Ixy" value="-0.00000122"/>
-    <xacro:property name="L06_Ixz" value="-0.00000054"/>
+    <xacro:property name="L06_Ixy" value="0.00000122"/>
+    <xacro:property name="L06_Ixz" value="0.00000054"/>
     <xacro:property name="L06_Iyy" value="0.00014750"/>
-    <xacro:property name="L06_Iyz" value="-0.00000008"/>
+    <xacro:property name="L06_Iyz" value="0.00000008"/>
     <xacro:property name="L06_Izz" value="0.00014680"/>
     <!-- Link Gripper Stator -->
@@ -86,8 +86,8 @@
     <xacro:property name="GripperStator_ComZ" value="-0.00249162"/>
     <xacro:property name="GripperStator_Ixx" value="0.00038683"/>
-    <xacro:property name="GripperStator_Ixy" value="0.00000359"/>
-    <xacro:property name="GripperStator_Ixz" value="-0.00007662"/>
+    <xacro:property name="GripperStator_Ixy" value="-0.00000359"/>
+    <xacro:property name="GripperStator_Ixz" value="0.00007662"/>
     <xacro:property name="GripperStator_Iyy" value="0.00068614"/>
-    <xacro:property name="GripperStator_Iyz" value="-0.00000209"/>
+    <xacro:property name="GripperStator_Iyz" value="0.00000209"/>
     <xacro:property name="GripperStator_Izz" value="0.00066293"/>
     <!-- Link Gripper Mover -->
@@ -97,8 +97,8 @@
     <xacro:property name="GripperMover_ComZ" value="0.00380534"/>
     <xacro:property name="GripperMover_Ixx" value="0.00017716"/>
-    <xacro:property name="GripperMover_Ixy" value="-0.00001683"/>
-    <xacro:property name="GripperMover_Ixz" value="0.00001786"/>
+    <xacro:property name="GripperMover_Ixy" value="0.00001683"/>
+    <xacro:property name="GripperMover_Ixz" value="-0.00001786"/>
     <xacro:property name="GripperMover_Iyy" value="0.00026787"/>
-    <xacro:property name="GripperMover_Iyz" value="-0.00000262"/>
+    <xacro:property name="GripperMover_Iyz" value="0.00000262"/>
     <xacro:property name="GripperMover_Izz" value="0.00035728"/>
     <!-- joint limits -->
