Commit message: update z1.urdf

File: robots/z1_description/xacro/z1.urdf (robot description, URDF)
Before this commit: robot z1_description, 8 links, 7 joints
Joints:
- joint joint1: limit lower=-2.6179938779914944 upper=2.6179938779914944 effort=30.0 velocity=10 -> lower=-2.6179938779914944 upper=2.6179938779914944 effort=30.0 velocity=3.1415
- joint joint2: limit lower=0.0 upper=2.9670597283903604 effort=60.0 velocity=10 -> lower=0.0 upper=2.9670597283903604 effort=60.0 velocity=3.1415
- joint joint3: limit lower=-2.8797932657906435 upper=0.0 effort=30.0 velocity=10 -> lower=-2.8797932657906435 upper=0.0 effort=30.0 velocity=3.1415
- joint joint4: limit lower=-1.5184364492350666 upper=1.5184364492350666 effort=30.0 velocity=10 -> lower=-1.5184364492350666 upper=1.5184364492350666 effort=30.0 velocity=3.1415
- joint joint5: limit lower=-1.3439035240356338 upper=1.3439035240356338 effort=30.0 velocity=10 -> lower=-1.3439035240356338 upper=1.3439035240356338 effort=30.0 velocity=3.1415
- joint joint6: limit lower=-2.792526803190927 upper=2.792526803190927 effort=30.0 velocity=10 -> lower=-2.792526803190927 upper=2.792526803190927 effort=30.0 velocity=3.1415
