Commit message: update inertial params and add _isaacgym files

File: robots/h1_description/urdf/h1_isaacgym.urdf (robot description, URDF)
Before this commit: robot h1_description, 22 links, 21 joints
Links:
- link logo_link: geometry visual mesh filename=package://h1_description/meshes/logo_link_gray.dae

File: robots/h1_description/urdf/h1_with_hand_isaacgym.urdf (robot description, URDF)
Before this commit: robot h1, 49 links, 48 joints
Links:
- link logo_link: geometry collision mesh filename=package://h1_description/meshes/logo_link.STL; visual mesh filename=package://h1_description/meshes/logo_link_gray.dae
