Commit message: fix collision for H1 with hand

File: robots/h1_description/urdf/h1_with_hand.urdf (robot description, URDF)
Before this commit: robot h1, 49 links, 48 joints
Links:
- link left_hip_yaw_link: geometry collision cylinder length=0.07 radius=0.06; visual mesh filename=package://h1_description/meshes/left_hip_yaw_link.STL
- link right_hip_yaw_link: geometry collision cylinder length=0.07 radius=0.06; visual mesh filename=package://h1_description/meshes/right_hip_yaw_link.STL

File: robots/h1_description/urdf/h1_with_hand_isaacgym.urdf (robot description, URDF)
Before this commit: robot h1, 49 links, 48 joints
Links:
- link left_hip_yaw_link: geometry collision cylinder length=0.07 radius=0.06; visual mesh filename=package://h1_description/meshes/left_hip_yaw_link.STL
- link right_hip_yaw_link: geometry collision cylinder length=0.07 radius=0.06; visual mesh filename=package://h1_description/meshes/right_hip_yaw_link.STL
