Commit message: update hip pitch joint limit

File: robots/h1_description/urdf/h1.urdf (robot description, URDF)
Before this commit: robot h1_description, 22 links, 21 joints
Joints:
- joint left_hip_pitch_joint: limit lower=-1.57 upper=1.57 effort=200 velocity=23 -> lower=-3.14 upper=2.53 effort=200 velocity=23
- joint right_hip_pitch_joint: limit lower=-1.57 upper=1.57 effort=200 velocity=23 -> lower=-3.14 upper=2.53 effort=200 velocity=23

File: robots/h1_description/urdf/h1_isaacgym.urdf (robot description, URDF)
Before this commit: robot h1_description, 22 links, 21 joints
Joints:
- joint left_hip_pitch_joint: limit lower=-1.57 upper=1.57 effort=200 velocity=23 -> lower=-3.14 upper=2.53 effort=200 velocity=23
- joint right_hip_pitch_joint: limit lower=-1.57 upper=1.57 effort=200 velocity=23 -> lower=-3.14 upper=2.53 effort=200 velocity=23

File: robots/h1_description/urdf/h1_with_hand.urdf (robot description, URDF)
Before this commit: robot h1, 49 links, 48 joints
Joints:
- joint left_hip_pitch_joint: limit lower=-1.57 upper=0.56 effort=200 velocity=23 -> lower=-3.14 upper=2.53 effort=200 velocity=23
- joint right_hip_pitch_joint: limit lower=-1.57 upper=0.56 effort=200 velocity=23 -> lower=-3.14 upper=2.53 effort=200 velocity=23

File: robots/h1_description/urdf/h1_with_hand_isaacgym.urdf (robot description, URDF)
Before this commit: robot h1, 49 links, 48 joints
Joints:
- joint left_hip_pitch_joint: limit lower=-1.57 upper=0.56 effort=200 velocity=23 -> lower=-3.14 upper=2.53 effort=200 velocity=23
- joint right_hip_pitch_joint: limit lower=-1.57 upper=0.56 effort=200 velocity=23 -> lower=-3.14 upper=2.53 effort=200 velocity=23

Commit message: update H1 urdf for isaac gym

File: robots/h1_description/urdf/h1.urdf (robot description, URDF)
Before this commit: robot h1_description, 22 links, 21 joints
Links:
- link left_ankle_link: geometry collision box size=0.28 0.03 0.024; visual mesh filename=package://h1_description/meshes/left_ankle_link.dae
- link left_elbow_link: mass 0.669 -> 0.723; geometry collision cylinder length=0.09 radius=0.03; visual mesh filename=package://h1_description/meshes/left_elbow_link.dae
- link left_hip_pitch_link: geometry collision cylinder length=0.2 radius=0.05; visual mesh filename=package://h1_description/meshes/left_hip_pitch_link.dae
- link left_hip_roll_link: geometry collision cylinder length=0.01 radius=0.02; visual mesh filename=package://h1_description/meshes/left_hip_roll_link.dae
- link left_hip_yaw_link: geometry collision cylinder length=0.02 radius=0.01; visual mesh filename=package://h1_description/meshes/left_hip_yaw_link.dae
- link left_knee_link: geometry collision cylinder length=0.2 radius=0.05; visual mesh filename=package://h1_description/meshes/left_knee_link.dae
- link left_shoulder_pitch_link: geometry collision cylinder length=0.04 radius=0.03; visual mesh filename=package://h1_description/meshes/left_shoulder_pitch_link.dae
- link left_shoulder_roll_link: geometry collision cylinder length=0.01 radius=0.04; visual mesh filename=package://h1_description/meshes/left_shoulder_roll_link.dae
- link left_shoulder_yaw_link: geometry collision cylinder length=0.01 radius=0.04; visual mesh filename=package://h1_description/meshes/left_shoulder_yaw_link.dae
- link logo_link: geometry visual mesh filename=package://h1_description/meshes/logo_link.dae
- link pelvis: geometry collision sphere radius=0.05; visual mesh filename=package://h1_description/meshes/pelvis.dae
- link right_ankle_link: geometry collision box size=0.28 0.03 0.024; visual mesh filename=package://h1_description/meshes/right_ankle_link.dae
- link right_elbow_link: mass 0.669 -> 0.723; geometry collision cylinder length=0.09 radius=0.03; visual mesh filename=package://h1_description/meshes/right_elbow_link.dae
- link right_hip_pitch_link: geometry collision cylinder length=0.2 radius=0.05; visual mesh filename=package://h1_description/meshes/right_hip_pitch_link.dae
- link right_hip_roll_link: geometry collision cylinder length=0.01 radius=0.02; visual mesh filename=package://h1_description/meshes/right_hip_roll_link.dae
- link right_hip_yaw_link: geometry collision cylinder length=0.02 radius=0.01; visual mesh filename=package://h1_description/meshes/right_hip_yaw_link.dae
- link right_knee_link: geometry collision cylinder length=0.2 radius=0.05; visual mesh filename=package://h1_description/meshes/right_knee_link.dae
- link right_shoulder_pitch_link: geometry collision cylinder length=0.04 radius=0.03; visual mesh filename=package://h1_description/meshes/right_shoulder_pitch_link.d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
- link right_shoulder_roll_link: geometry collision cylinder length=0.01 radius=0.04; visual mesh filename=package://h1_description/meshes/right_shoulder_roll_link.dae
- link right_shoulder_yaw_link: geometry collision cylinder length=0.01 radius=0.04; visual mesh filename=package://h1_description/meshes/right_shoulder_yaw_link.dae
- link torso_link: geometry collision box size=0.08 0.16 0.1; visual mesh filename=package://h1_description/meshes/torso_link.dae

File: robots/h1_description/urdf/h1_with_hand.urdf (robot description, URDF)
Before this commit: robot h1, 49 links, 48 joints
Links:
- link L_hand_base_link: geometry collision mesh filename=package://h1_description/meshes/L_hand_base_link.STL; visual mesh filename=package://h1_description/meshes/L_hand_base_link.dae
- link L_index_intermediate: geometry collision mesh filename=package://h1_description/meshes/Link16_L.STL; visual mesh filename=package://h1_description/meshes/Link16_L.dae
- link L_index_proximal: geometry collision mesh filename=package://h1_description/meshes/Link15_L.STL; visual mesh filename=package://h1_description/meshes/Link15_L.dae
- link L_middle_intermediate: geometry collision mesh filename=package://h1_description/meshes/Link18_L.STL; visual mesh filename=package://h1_description/meshes/Link18_L.dae
- link L_middle_proximal: geometry collision mesh filename=package://h1_description/meshes/Link17_L.STL; visual mesh filename=package://h1_description/meshes/Link17_L.dae
- link L_pinky_intermediate: geometry collision mesh filename=package://h1_description/meshes/Link22_L.STL; visual mesh filename=package://h1_description/meshes/Link22_L.dae
- link L_pinky_proximal: geometry collision mesh filename=package://h1_description/meshes/Link21_L.STL; visual mesh filename=package://h1_description/meshes/Link21_L.dae
- link L_ring_intermediate: geometry collision mesh filename=package://h1_description/meshes/Link20_L.STL; visual mesh filename=package://h1_description/meshes/Link20_L.dae
- link L_ring_proximal: geometry collision mesh filename=package://h1_description/meshes/Link19_L.STL; visual mesh filename=package://h1_description/meshes/Link19_L.dae
- link L_thumb_distal: geometry collision mesh filename=package://h1_description/meshes/Link14_L.STL; visual mesh filename=package://h1_description/meshes/Link14_L.dae
- link L_thumb_intermediate: geometry collision mesh filename=package://h1_description/meshes/Link13_L.STL; visual mesh filename=package://h1_description/meshes/Link13_L.dae
- link L_thumb_proximal: geometry collision mesh filename=package://h1_description/meshes/Link12_L.STL; visual mesh filename=package://h1_description/meshes/Link12_L.dae
- link L_thumb_proximal_base: geometry collision mesh filename=package://h1_description/meshes/Link11_L.STL; visual mesh filename=package://h1_description/meshes/Link11_L.dae
- link R_hand_base_link: geometry collision mesh filename=package://h1_description/meshes/R_hand_base_link.STL; visual mesh filename=package://h1_description/meshes/R_hand_base_link.dae
- link R_index_intermediate: geometry collision mesh filename=package://h1_description/meshes/Link16_R.STL; visual mesh filename=package://h1_description/meshes/Link16_R.dae
- link R_index_proximal: geometry collision mesh filename=package://h1_description/meshes/Link15_R.STL; visual mesh filename=package://h1_description/meshes/Link15_R.dae
- link R_middle_intermediate: geometry collision mesh filename=package://h1_description/meshes/Link18_R.STL; visual mesh filename=package://h1_description/meshes/Link18_R.dae
- link R_middle_proximal: geometry collision mesh filename=package://h1_description/meshes/Link17_R.STL; visual mesh filename=package://h1_description/meshes/Link17_R.dae
- link R_pinky_intermediate: geometry collision mesh filename=package://h1_description/meshes/Link22_R.STL; visual mesh filename=package://h1_description/meshes/Link22_R.dae
- link R_pinky_proximal: geometry collision mesh filename=package://h1_description/meshes/Link21_R.STL; visual mesh filename=package://h1_description/meshes/Link21_R.dae
- link R_ring_intermediate: geometry collision mesh filename=package://h1_description/meshes/Link20_R.STL; visual mesh filename=package://h1_description/meshes/Link20_R.dae
- link R_ring_proximal: geometry collision mesh filename=package://h1_description/meshes/Link19_R.STL; visual mesh filename=package://h1_description/meshes/Link19_R.dae
- link R_thumb_distal: geometry collision mesh filename=package://h1_description/meshes/Link14_R.STL; visual mesh filename=package://h1_description/meshes/Link14_R.dae
- link R_thumb_intermediate: geometry collision mesh filename=package://h1_description/meshes/Link13_R.STL; visual mesh filename=package://h1_description/meshes/Link13_R.dae
- link R_thumb_proximal: geometry collision mesh filename=package://h1_description/meshes/Link12_R.STL; visual mesh filename=package://h1_description/meshes/Link12_R.dae
- link R_thumb_proximal_base: geometry collision mesh filename=package://h1_description/meshes/Link11_R.STL; visual mesh filename=package://h1_description/meshes/Link11_R.dae
- link left_ankle_link: geometry collision box size=0.28 0.03 0.024; visual mesh filename=package://h1_description/meshes/left_ankle_link.dae
- link left_elbow_link: geometry collision cylinder length=0.09 radius=0.03; visual mesh filename=package://h1_description/meshes/left_elbow_link.dae
- link left_hand_link: geometry collision mesh filename=package://h1_description/meshes/left_hand_link.STL; visual mesh filename=package://h1_description/meshes/left_hand_link.dae
- link left_hip_pitch_link: geometry collision cylinder length=0.2 radius=0.05; visual mesh filename=package://h1_description/meshes/left_hip_pitch_link.dae
- link left_hip_roll_link: geometry collision cylinder length=0.01 radius=0.02; visual mesh filename=package://h1_description/meshes/left_hip_roll_link.dae
- link left_hip_yaw_link: geometry collision cylinder length=0.02 radius=0.01; visual mesh filename=package://h1_description/meshes/left_hip_yaw_link.dae
- link left_knee_link: geometry collision cylinder length=0.2 radius=0.05; visual mesh filename=package://h1_description/meshes/left_knee_link.dae
- link left_shoulder_pitch_link: geometry collision cylinder length=0.04 radius=0.03; visual mesh filename=package://h1_description/meshes/left_shoulder_pitch_link.dae
- link left_shoulder_roll_link: geometry collision cylinder length=0.01 radius=0.04; visual mesh filename=package://h1_description/meshes/left_shoulder_roll_link.dae
- link left_shoulder_yaw_link: geometry collision cylinder length=0.01 radius=0.04; visual mesh filename=package://h1_description/meshes/left_shoulder_yaw_link.dae
- link logo_link: geometry visual mesh filename=package://h1_description/meshes/logo_link.dae
- link pelvis: geometry collision sphere radius=0.05; visual mesh filename=package://h1_description/meshes/pelvis.dae
- link right_ankle_link: geometry collision box size=0.28 0.03 0.024; visual mesh filename=package://h1_description/meshes/right_ankle_link.dae
- link right_elbow_link: geometry collision cylinder length=0.09 radius=0.03; visual mesh filename=package://h1_description/meshes/right_elbow_link.dae
- link right_hand_link: geometry collision mesh filename=package://h1_description/meshes/right_hand_link.STL; visual mesh filename=package://h1_description/meshes/right_hand_link.dae
- link right_hip_pitch_link: geometry collision cylinder length=0.2 radius=0.05; visual mesh filename=package://h1_description/meshes/right_hip_pitch_link.dae
- link right_hip_roll_link: geometry collision cylinder length=0.01 radius=0.02; visual mesh filename=package://h1_description/meshes/right_hip_roll_link.dae
- link right_hip_yaw_link: geometry collision cylinder length=0.02 radius=0.01; visual mesh filename=package://h1_description/meshes/right_hip_yaw_link.dae
- link right_knee_link: geometry collision cylinder length=0.2 radius=0.05; visual mesh filename=package://h1_description/meshes/right_knee_link.dae
- link right_shoulder_pitch_link: geometry collision cylinder length=0.04 radius=0.03; visual mesh filename=package://h1_description/meshes/right_shoulder_pitch_link.d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
- link right_shoulder_roll_link: geometry collision cylinder length=0.01 radius=0.04; visual mesh filename=package://h1_description/meshes/right_shoulder_roll_link.dae
- link right_shoulder_yaw_link: geometry collision cylinder length=0.01 radius=0.04; visual mesh filename=package://h1_description/meshes/right_shoulder_yaw_link.dae
- link torso_link: geometry collision box size=0.08 0.16 0.1; visual mesh filename=package://h1_description/meshes/torso_link.dae

Commit message: add camera and ladar links/joints in H1 urdf

File: robots/h1_description/urdf/h1.urdf (robot description, URDF)
Before this commit: robot h1_description, 22 links, 21 joints
Links:
- added link d435_left_imager_link; collision sphere radius=0.001; visual sphere radius=0.001
- added link d435_rgb_module_link; collision sphere radius=0.001; visual sphere radius=0.001
- added link mid360_link; collision sphere radius=0.001; visual sphere radius=0.001
Joints:
- added joint d435_left_imager_joint: type fixed, parent torso_link, child d435_left_imager_link, origin xyz=0.10848474394 0.0175 0.69317107367 rpy=-2.45735 0 -1.57080, axis 0 0 0
- added joint d435_rgb_module_joint: type fixed, parent torso_link, child d435_rgb_module_link, origin xyz=0.10848474394 0.0325 0.69317107367 rpy=-2.45735 0 -1.57080, axis 0 0 0
- added joint mid360_joint: type fixed, parent torso_link, child mid360_link, origin xyz=0.04729990180 0 0.67492878653 rpy=0 0.243124 0, axis 0 0 0

File: robots/h1_description/urdf/h1_with_hand.urdf (robot description, URDF)
Before this commit: robot h1, 49 links, 48 joints
Links:
- added link d435_left_imager_link; collision sphere radius=0.001; visual sphere radius=0.001
- added link d435_rgb_module_link; collision sphere radius=0.001; visual sphere radius=0.001
- added link mid360_link; collision sphere radius=0.001; visual sphere radius=0.001
Joints:
- added joint d435_left_imager_joint: type fixed, parent torso_link, child d435_left_imager_link, origin xyz=0.10848474394 0.0175 0.69317107367 rpy=-2.45735 0 -1.57080, axis 0 0 0
- added joint d435_rgb_module_joint: type fixed, parent torso_link, child d435_rgb_module_link, origin xyz=0.10848474394 0.0325 0.69317107367 rpy=-2.45735 0 -1.57080, axis 0 0 0
- added joint mid360_joint: type fixed, parent torso_link, child mid360_link, origin xyz=0.04729990180 0 0.67492878653 rpy=0 0.243124 0, axis 0 0 0

Commit message: change h1 torso_link mass

File: robots/h1_description/urdf/h1.urdf (robot description, URDF)
Before this commit: robot h1_description, 25 links, 24 joints
Links:
- link torso_link: mass 17.789 -> 21.189

File: robots/h1_description/urdf/h1_with_hand.urdf (robot description, URDF)
Before this commit: robot h1, 52 links, 51 joints
Links:
- link torso_link: mass 17.789 -> 21.189

Commit message: update h1 urdf (mass&inertial)

File: robots/h1_description/urdf/h1.urdf (robot description, URDF)
Before this commit: robot h1_description, 25 links, 24 joints
Links:
- link left_ankle_link: mass 0.474 -> 0.725; geometry collision box size=0.28 0.03 0.024; visual mesh filename=package://h1_description/meshes/left_ankle_link.STL
- link left_elbow_link: mass 0.723 -> 0.745; geometry collision cylinder length=0.09 radius=0.03; visual mesh filename=package://h1_description/meshes/left_elbow_link.STL
- link left_hip_pitch_link: mass 4.152 -> 4.953; geometry collision cylinder length=0.2 radius=0.05; visual mesh filename=package://h1_description/meshes/left_hip_pitch_link.STL
- link left_hip_roll_link: mass 2.232 -> 2.7150; geometry collision cylinder length=0.01 radius=0.02; visual mesh filename=package://h1_description/meshes/left_hip_roll_link.STL
- link left_hip_yaw_link: mass 2.244 -> 2.965; geometry collision cylinder length=0.02 radius=0.01; visual mesh filename=package://h1_description/meshes/left_hip_yaw_link.STL
- link left_knee_link: mass 1.721 -> 2.824; geometry collision cylinder length=0.2 radius=0.05; visual mesh filename=package://h1_description/meshes/left_knee_link.STL
- link left_shoulder_pitch_link: mass 1.033 -> 1.142; geometry collision cylinder length=0.04 radius=0.03; visual mesh filename=package://h1_description/meshes/left_shoulder_pitch_link.STL
- link left_shoulder_roll_link: mass 0.793 -> 0.852; geometry collision cylinder length=0.01 radius=0.04; visual mesh filename=package://h1_description/meshes/left_shoulder_roll_link.STL
- link left_shoulder_yaw_link: mass 0.839 -> 0.862; geometry collision cylinder length=0.01 radius=0.04; visual mesh filename=package://h1_description/meshes/left_shoulder_yaw_link.STL
- link logo_link: geometry visual mesh filename=package://h1_description/meshes/logo_link.STL
- link pelvis: mass 5.39 -> 5.983; geometry collision sphere radius=0.05; visual mesh filename=package://h1_description/meshes/pelvis.STL
- link right_ankle_link: mass 0.474 -> 0.725; geometry collision box size=0.28 0.03 0.024; visual mesh filename=package://h1_description/meshes/right_ankle_link.STL
- link right_elbow_link: mass 0.723 -> 0.745; geometry collision cylinder length=0.09 radius=0.03; visual mesh filename=package://h1_description/meshes/right_elbow_link.STL
- link right_hip_pitch_link: mass 4.152 -> 4.953; geometry collision cylinder length=0.2 radius=0.05; visual mesh filename=package://h1_description/meshes/right_hip_pitch_link.STL
- link right_hip_roll_link: mass 2.232 -> 2.7150; geometry collision cylinder length=0.01 radius=0.02; visual mesh filename=package://h1_description/meshes/right_hip_roll_link.STL
- link right_hip_yaw_link: mass 2.244 -> 2.965; geometry collision cylinder length=0.02 radius=0.01; visual mesh filename=package://h1_description/meshes/right_hip_yaw_link.STL
- link right_knee_link: mass 1.721 -> 2.824; geometry collision cylinder length=0.2 radius=0.05; visual mesh filename=package://h1_description/meshes/right_knee_link.STL
- link right_shoulder_pitch_link: mass 1.033 -> 1.142; geometry collision cylinder length=0.04 radius=0.03; visual mesh filename=package://h1_description/meshes/right_shoulder_pitch_link.S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
- link right_shoulder_roll_link: mass 0.793 -> 0.852; geometry collision cylinder length=0.01 radius=0.04; visual mesh filename=package://h1_description/meshes/right_shoulder_roll_link.STL
- link right_shoulder_yaw_link: mass 0.839 -> 0.862; geometry collision cylinder length=0.01 radius=0.04; visual mesh filename=package://h1_description/meshes/right_shoulder_yaw_link.STL
- link torso_link: mass 21.189 -> 17.789; geometry collision box size=0.08 0.16 0.1; visual mesh filename=package://h1_description/meshes/torso_link.STL
