Commit message: cylinder foot to sphere foot

File: robots/b2_description/urdf/b2_description.urdf (robot description, URDF)
Before this commit: robot b2_description, 37 links, 36 joints
Links:
- link FL_foot: geometry collision sphere radius=0.032
- link FR_foot: geometry collision sphere radius=0.032
- link RL_foot: geometry collision sphere radius=0.032
- link RR_foot: geometry collision sphere radius=0.032

File: robots/b2_description/xacro/leg.xacro (robot description, xacro)
@@ -234,5 +234,5 @@
                 rpy="0 0 0" />
             <geometry>
-                <cylinder length="0.05" radius="0.032" />
+                <sphere radius="0.032" />
             </geometry>
             </collision>

Commit message: modify some inertial parameters in B2 and B2W

File: robots/b2_description/urdf/b2_description.urdf (robot description, URDF)
Before this commit: robot b2_description, 37 links, 36 joints
Links:
- link FL_calf: mass 0.58094 -> 0.404
- link FL_foot: mass 0.098183 -> 0.126
- link FL_hip: mass 2.256 -> 2.673
- link FL_thigh: mass 3.591 -> 4.536
- link FR_calf: mass 0.58094 -> 0.404
- link FR_foot: mass 0.098183 -> 0.126
- link FR_thigh: mass 3.591 -> 4.536
- link RL_calf: mass 0.58094 -> 0.404
- link RL_foot: mass 0.098183 -> 0.126
- link RL_thigh: mass 3.591 -> 4.536
- link RR_calf: mass 0.58094 -> 0.404
- link RR_foot: mass 0.098183 -> 0.126
- link RR_hip: mass 2.256 -> 2.673
- link RR_thigh: mass 3.591 -> 4.536
- link base_link: mass 35.606 -> 35.86
- link f_dc_link: mass 6.54E-08 -> 4.19E-15
- link f_oc_link: mass 6.55E-08 -> 4.19E-15
- link head_Link: mass 3.366 -> 3.6885
- link imu_link: mass 6.54E-08 -> 4.19E-15
- link lidar_link: mass 6.55E-08 -> 4.19E-15
- link r_dc_link: mass 6.55E-08 -> 4.19E-15
- link r_oc_link: mass 6.55E-08 -> 4.19E-12
- link tail_link: mass 0.777 -> 0.795

File: robots/b2w_description/urdf/b2w_description.urdf (robot description, URDF)
Before this commit: robot b2w_description, 26 links, 25 joints
Links:
- link FL_calf: mass 2.053 -> 2.2906
- link FL_foot: mass 0.918 -> 1.083
- link FL_hip: mass 2.256 -> 2.673
- link FL_thigh: mass 3.591 -> 4.536
- link FR_calf: mass 2.053 -> 2.290557
- link FR_foot: mass 0.918 -> 1.083
- link FR_hip: mass 2.256 -> 2.673
- link FR_thigh: mass 3.591 -> 4.536
- link RL_calf: mass 2.053 -> 2.2906
- link RL_foot: mass 0.918 -> 1.083
- link RL_hip: mass 2.256 -> 2.673
- link RL_thigh: mass 3.591 -> 4.536
- link RR_calf: mass 2.053 -> 2.2906
- link RR_foot: mass 0.918 -> 1.083
- link RR_hip: mass 2.256 -> 2.673
- link RR_thigh: mass 3.591 -> 4.536
- link head_Link: mass 3.366 -> 3.6885
- link tail_link: mass 0.777 -> 0.795

Commit message: revise b2 urdf

File: robots/b2_description/urdf/b2_description.urdf (robot description, URDF)
Before this commit: robot b2_description, 37 links, 36 joints
Links:
- link FR_hip: mass 2.256 -> 2.673
- link RL_hip: mass 2.256 -> 2.673
