Commit message: rename G1 fingers

File: robots/g1_description/g1_29dof_with_hand.urdf (robot description, URDF)
Before this commit: robot g1_29dof_with_hand, 51 links, 50 joints
Links:
- removed link left_hand_five_link
- removed link left_hand_four_link
- removed link left_hand_one_link
- removed link left_hand_six_link
- removed link left_hand_three_link
- removed link left_hand_two_link
- removed link left_hand_zero_link
- removed link right_hand_five_link
- removed link right_hand_four_link
- removed link right_hand_one_link
- removed link right_hand_six_link
- removed link right_hand_three_link
- removed link right_hand_two_link
- removed link right_hand_zero_link
- added link left_hand_index_0_link, mass 0.05619628; collision mesh filename=meshes/left_hand_index_0_link.STL; visual mesh filename=meshes/left_hand_index_0_link.STL
- added link left_hand_index_1_link, mass 0.02487314; collision mesh filename=meshes/left_hand_index_1_link.STL; visual mesh filename=meshes/left_hand_index_1_link.STL
- added link left_hand_middle_0_link, mass 0.05619628; collision mesh filename=meshes/left_hand_middle_0_link.STL; visual mesh filename=meshes/left_hand_middle_0_link.STL
- added link left_hand_middle_1_link, mass 0.02487314; collision mesh filename=meshes/left_hand_middle_1_link.STL; visual mesh filename=meshes/left_hand_middle_1_link.STL
- added link left_hand_thumb_0_link, mass 0.08033018; collision mesh filename=meshes/left_hand_thumb_0_link.STL; visual mesh filename=meshes/left_hand_thumb_0_link.STL
- added link left_hand_thumb_1_link, mass 0.05619628; collision box size=0.02 0.03 0.02; visual mesh filename=meshes/left_hand_thumb_1_link.STL
- added link left_hand_thumb_2_link, mass 0.02487314; collision mesh filename=meshes/left_hand_thumb_2_link.STL; visual mesh filename=meshes/left_hand_thumb_2_link.STL
- added link right_hand_index_0_link, mass 0.05619628; collision mesh filename=meshes/right_hand_index_0_link.STL; visual mesh filename=meshes/right_hand_index_0_link.STL
- added link right_hand_index_1_link, mass 0.02487314; collision mesh filename=meshes/right_hand_index_1_link.STL; visual mesh filename=meshes/right_hand_index_1_link.STL
- added link right_hand_middle_0_link, mass 0.05619628; collision mesh filename=meshes/right_hand_middle_0_link.STL; visual mesh filename=meshes/right_hand_middle_0_link.STL
- added link right_hand_middle_1_link, mass 0.02487314; collision mesh filename=meshes/right_hand_middle_1_link.STL; visual mesh filename=meshes/right_hand_middle_1_link.STL
- added link right_hand_thumb_0_link, mass 0.08033018; collision mesh filename=meshes/right_hand_thumb_0_link.STL; visual mesh filename=meshes/right_hand_thumb_0_link.STL
- added link right_hand_thumb_1_link, mass 0.05619628; collision box size=0.02 0.03 0.02; visual mesh filename=meshes/right_hand_thumb_1_link.STL
- added link right_hand_thumb_2_link, mass 0.02487314; collision mesh filename=meshes/right_hand_thumb_2_link.STL; visual mesh filename=meshes/right_hand_thumb_2_link.STL
Joints:
- removed joint left_hand_five_joint
- removed joint left_hand_four_joint
- removed joint left_hand_one_joint
- removed joint left_hand_six_joint
- removed joint left_hand_three_joint
- removed joint left_hand_two_joint
- removed joint left_hand_zero_joint
- removed joint right_hand_five_joint
- removed joint right_hand_four_joint
- removed joint right_hand_one_joint
- removed joint right_hand_six_joint
- removed joint right_hand_three_joint
- removed joint right_hand_two_joint
- removed joint right_hand_zero_joint
- added joint left_hand_index_0_joint: type revolute, parent left_hand_palm_link, child left_hand_index_0_link, origin xyz=0.1 -0.0017 0.0285 rpy=0 0 0, axis 0 0 1, limit lower=-1.83259571 upper=0.19198621 effort=0.7 velocity=24
- added joint left_hand_index_1_joint: type revolute, parent left_hand_index_0_link, child left_hand_index_1_link, origin xyz=0.0528 -0.0055 0 rpy=0 0 0, axis 0 0 1, limit lower=-2.09439510 upper=0 effort=0.7 velocity=24
- added joint left_hand_middle_0_joint: type revolute, parent left_hand_palm_link, child left_hand_middle_0_link, origin xyz=0.1 -0.0017 -0.0285 rpy=0 0 0, axis 0 0 1, limit lower=-1.83259571 upper=0.19198621 effort=0.7 velocity=24
- added joint left_hand_middle_1_joint: type revolute, parent left_hand_middle_0_link, child left_hand_middle_1_link, origin xyz=0.0528 -0.0055 0 rpy=0 0 0, axis 0 0 1, limit lower=-2.09439510 upper=0 effort=0.7 velocity=24
- added joint left_hand_thumb_0_joint: type revolute, parent left_hand_palm_link, child left_hand_thumb_0_link, origin xyz=0.028 0 0 rpy=0 0 0, axis 0 1 0, limit lower=-1.04719755 upper=1.04719755 effort=2.45 velocity=6.857
- added joint left_hand_thumb_1_joint: type revolute, parent left_hand_thumb_0_link, child left_hand_thumb_1_link, origin xyz=0 -0.0246 0 rpy=0 0 0, axis 0 0 1, limit lower=-0.72431163 upper=1.04719755 effort=0.7 velocity=24
- added joint left_hand_thumb_2_joint: type revolute, parent left_hand_thumb_1_link, child left_hand_thumb_2_link, origin xyz=0.0055 -0.0528 0 rpy=0 0 0, axis 0 0 1, limit lower=0 upper=2.09439510 effort=0.7 velocity=24
- added joint right_hand_index_0_joint: type revolute, parent right_hand_palm_link, child right_hand_index_0_link, origin xyz=0.1 0.0017 0.0285 rpy=0 0 0, axis 0 0 1, limit lower=-0.19198621 upper=1.83259571 effort=0.7 velocity=24
- added joint right_hand_index_1_joint: type revolute, parent right_hand_index_0_link, child right_hand_index_1_link, origin xyz=0.0528 0.0055 0 rpy=0 0 0, axis 0 0 1, limit lower=0 upper=2.09439510 effort=0.7 velocity=24
- added joint right_hand_middle_0_joint: type revolute, parent right_hand_palm_link, child right_hand_middle_0_link, origin xyz=0.1 0.0017 -0.0285 rpy=0 0 0, axis 0 0 1, limit lower=-0.19198621 upper=1.83259571 effort=0.7 velocity=24
- added joint right_hand_middle_1_joint: type revolute, parent right_hand_middle_0_link, child right_hand_middle_1_link, origin xyz=0.0528 0.0055 0 rpy=0 0 0, axis 0 0 1, limit lower=0 upper=2.09439510 effort=0.7 velocity=24
- added joint right_hand_thumb_0_joint: type revolute, parent right_hand_palm_link, child right_hand_thumb_0_link, origin xyz=0.028 0 0 rpy=0 0 0, axis 0 1 0, limit lower=-1.04719755 upper=1.04719755 effort=2.45 velocity=6.857
- added joint right_hand_thumb_1_joint: type revolute, parent right_hand_thumb_0_link, child right_hand_thumb_1_link, origin xyz=0 0.0246 0 rpy=0 0 0, axis 0 0 1, limit lower=-1.04719755 upper=0.72431163 effort=0.7 velocity=24
- added joint right_hand_thumb_2_joint: type revolute, parent right_hand_thumb_1_link, child right_hand_thumb_2_link, origin xyz=0.0055 0.0528 0 rpy=0 0 0, axis 0 0 1, limit lower=-2.09439510 upper=0 effort=0.7 velocity=24

Commit message: update g1_29dof_with_hand model

File: robots/g1_description/g1_29dof_with_hand.urdf (robot description, URDF)
Before this commit: robot g1_29dof_with_hand, 53 links, 52 joints
Links:
- link left_hand_index_0_link: mass 0.05619628 -> 0.05885070
- link left_hand_index_1_link: mass 0.02487314 -> 0.02030626
- link left_hand_middle_0_link: mass 0.05619628 -> 0.05885070
- link left_hand_middle_1_link: mass 0.02487314 -> 0.02030626
- link left_hand_thumb_0_link: mass 0.08033018 -> 0.08623657
- link left_hand_thumb_1_link: mass 0.05619628 -> 0.05885070
- link left_hand_thumb_2_link: mass 0.02487314 -> 0.02030626
- link right_hand_index_0_link: mass 0.05619628 -> 0.05885070
- link right_hand_index_1_link: mass 0.02487314 -> 0.02030626
- link right_hand_middle_0_link: mass 0.05619628 -> 0.05885070
- link right_hand_middle_1_link: mass 0.02487314 -> 0.02030626
- link right_hand_thumb_0_link: mass 0.08033018 -> 0.08623657
- link right_hand_thumb_1_link: mass 0.05619628 -> 0.05885070
- link right_hand_thumb_2_link: mass 0.02487314 -> 0.02030626
Joints:
- joint left_hand_index_0_joint: limit lower=-1.83259571 upper=0.19198621 effort=0.7 velocity=24 -> lower=-1.57079632 upper=0 effort=1.4 velocity=12; origin xyz=0.1 -0.0017 0.0285 rpy=0 0 0 -> xyz=0.0777 0.0016 0.0285 rpy=0 0 0
- joint left_hand_index_1_joint: limit lower=-2.09439510 upper=0 effort=0.7 velocity=24 -> lower=-1.74532925 upper=0 effort=1.4 velocity=12; origin xyz=0.0528 -0.0055 0 rpy=0 0 0 -> xyz=0.0458 0 0 rpy=0 0 0
- joint left_hand_middle_0_joint: limit lower=-1.83259571 upper=0.19198621 effort=0.7 velocity=24 -> lower=-1.57079632 upper=0 effort=1.4 velocity=12; origin xyz=0.1 -0.0017 -0.0285 rpy=0 0 0 -> xyz=0.0777 0.0016 -0.0285 rpy=0 0 0
- joint left_hand_middle_1_joint: limit lower=-2.09439510 upper=0 effort=0.7 velocity=24 -> lower=-1.74532925 upper=0 effort=1.4 velocity=12; origin xyz=0.0528 -0.0055 0 rpy=0 0 0 -> xyz=0.0458 0 0 rpy=0 0 0
- joint left_hand_thumb_0_joint: origin xyz=0.028 0 0 rpy=0 0 0 -> xyz=0.0255 0 0 rpy=0 0 0
- joint left_hand_thumb_1_joint: limit lower=-0.72431163 upper=1.04719755 effort=0.7 velocity=24 -> lower=-0.72431163 upper=1.04719755 effort=1.4 velocity=12; origin xyz=0 -0.0246 0 rpy=0 0 0 -> xyz=-0.0025 -0.0193 0 rpy=0 0 0
- joint left_hand_thumb_2_joint: limit lower=0 upper=2.09439510 effort=0.7 velocity=24 -> lower=0 upper=1.74532925 effort=1.4 velocity=12; origin xyz=0.0055 -0.0528 0 rpy=0 0 0 -> xyz=0 -0.0458 0 rpy=0 0 0
- joint right_hand_index_0_joint: limit lower=-0.19198621 upper=1.83259571 effort=0.7 velocity=24 -> lower=0 upper=1.57079632 effort=1.4 velocity=12; origin xyz=0.1 0.0017 0.0285 rpy=0 0 0 -> xyz=0.0777 -0.0016 0.0285 rpy=0 0 0
- joint right_hand_index_1_joint: limit lower=0 upper=2.09439510 effort=0.7 velocity=24 -> lower=0 upper=1.74532925 effort=1.4 velocity=12; origin xyz=0.0528 0.0055 0 rpy=0 0 0 -> xyz=0.0458 0 0 rpy=0 0 0
- joint right_hand_middle_0_joint: limit lower=-0.19198621 upper=1.83259571 effort=0.7 velocity=24 -> lower=0 upper=1.57079632 effort=1.4 velocity=12; origin xyz=0.1 0.0017 -0.0285 rpy=0 0 0 -> xyz=0.0777 -0.0016 -0.0285 rpy=0 0 0
- joint right_hand_middle_1_joint: limit lower=0 upper=2.09439510 effort=0.7 velocity=24 -> lower=0 upper=1.74532925 effort=1.4 velocity=12; origin xyz=0.0528 0.0055 0 rpy=0 0 0 -> xyz=0.0458 0 0 rpy=0 0 0
- joint right_hand_thumb_0_joint: origin xyz=0.028 0 0 rpy=0 0 0 -> xyz=0.0255 0 0 rpy=0 0 0
- joint right_hand_thumb_1_joint: limit lower=-1.04719755 upper=0.72431163 effort=0.7 velocity=24 -> lower=-1.04719755 upper=0.72431163 effort=1.4 velocity=12; origin xyz=0 0.0246 0 rpy=0 0 0 -> xyz=-0.0025 0.0193 0 rpy=0 0 0
- joint right_hand_thumb_2_joint: limit lower=-2.09439510 upper=0 effort=0.7 velocity=24 -> lower=-1.74532925 upper=0 effort=1.4 velocity=12; origin xyz=0.0055 0.0528 0 rpy=0 0 0 -> xyz=0 0.0458 0 rpy=0 0 0
