Commit message: add inspire hand for g1

File: robots/g1_description/dex3_1_l.urdf (robot description, URDF)
Before this commit: robot g1_29dof_with_hand_rev_1_0, 8 links, 7 joints
Joints:
- joint left_hand_thumb_0_joint: limit lower=-1.04719755 upper=1.04719755 effort=2.45 velocity=6.857 -> lower=-1.04719755 upper=1.04719755 effort=2.45 velocity=3.14

File: robots/g1_description/dex3_1_r.urdf (robot description, URDF)
Before this commit: robot g1_29dof_with_hand_rev_1_0, 8 links, 7 joints
Joints:
- joint right_hand_thumb_0_joint: limit lower=-1.04719755 upper=1.04719755 effort=2.45 velocity=6.857 -> lower=-1.04719755 upper=1.04719755 effort=2.45 velocity=3.14

File: robots/g1_description/g1_29dof_lock_waist_with_hand_rev_1_0.urdf (robot description, URDF)
Before this commit: robot g1_29dof_lock_waist_with_hand_rev_1_0, 53 links, 52 joints
Joints:
- joint left_hand_thumb_0_joint: limit lower=-1.04719755 upper=1.04719755 effort=2.45 velocity=6.857 -> lower=-1.04719755 upper=1.04719755 effort=2.45 velocity=3.14
- joint right_hand_thumb_0_joint: limit lower=-1.04719755 upper=1.04719755 effort=2.45 velocity=6.857 -> lower=-1.04719755 upper=1.04719755 effort=2.45 velocity=3.14

File: robots/g1_description/g1_29dof_with_hand.urdf (robot description, URDF)
Before this commit: robot g1_29dof_with_hand, 54 links, 53 joints
Joints:
- joint left_hand_thumb_0_joint: limit lower=-1.04719755 upper=1.04719755 effort=2.45 velocity=6.857 -> lower=-1.04719755 upper=1.04719755 effort=2.45 velocity=3.14
- joint right_hand_thumb_0_joint: limit lower=-1.04719755 upper=1.04719755 effort=2.45 velocity=6.857 -> lower=-1.04719755 upper=1.04719755 effort=2.45 velocity=3.14

File: robots/g1_description/g1_29dof_with_hand_rev_1_0.urdf (robot description, URDF)
Before this commit: robot g1_29dof_with_hand_rev_1_0, 53 links, 52 joints
Joints:
- joint left_hand_thumb_0_joint: limit lower=-1.04719755 upper=1.04719755 effort=2.45 velocity=6.857 -> lower=-1.04719755 upper=1.04719755 effort=2.45 velocity=3.14
- joint right_hand_thumb_0_joint: limit lower=-1.04719755 upper=1.04719755 effort=2.45 velocity=6.857 -> lower=-1.04719755 upper=1.04719755 effort=2.45 velocity=3.14
