Commit message: update g1_comp

File: robots/g1_description/g1_comp.urdf (robot description, URDF)
Before this commit: robot g1_comp, 34 links, 33 joints
Links:
- link d455_link: geometry collision cylinder length=0.1 radius=0.015; visual mesh filename=meshes/d455_link.STL
- link xl330_link: geometry visual mesh filename=meshes/xl330_link.STL
