Commit message: update g1 pelvis mesh

File: robots/g1_description/g1_23dof_mode_10.urdf (robot description, URDF)
Before this commit: robot g1_23dof_mode_10, 31 links, 30 joints
Links:
- removed link pelvis_contour_link
- link pelvis: geometry visual mesh filename=meshes/pelvis_ver0529.STL
Joints:
- removed joint pelvis_contour_joint

File: robots/g1_description/g1_29dof_mode_11.urdf (robot description, URDF)
Before this commit: robot g1_29dof_mode_11, 39 links, 38 joints
Links:
- removed link pelvis_contour_link
- link pelvis: geometry visual mesh filename=meshes/pelvis_ver0529.STL
Joints:
- removed joint pelvis_contour_joint

File: robots/g1_description/g1_29dof_mode_12.urdf (robot description, URDF)
Before this commit: robot g1_29dof_mode_12, 39 links, 38 joints
Links:
- removed link pelvis_contour_link
- link pelvis: geometry visual mesh filename=meshes/pelvis_ver0529.STL
Joints:
- removed joint pelvis_contour_joint

File: robots/g1_description/g1_29dof_mode_15.urdf (robot description, URDF)
Before this commit: robot g1_29dof_mode_15, 39 links, 38 joints
Links:
- removed link pelvis_contour_link
- link pelvis: geometry visual mesh filename=meshes/pelvis_ver0529.STL
Joints:
- removed joint pelvis_contour_joint

File: robots/g1_description/g1_29dof_mode_15_with_dex1_1.urdf (robot description, URDF)
Before this commit: robot g1_29dof_mode_15, 43 links, 42 joints
Links:
- removed link pelvis_contour_link
- link pelvis: geometry visual mesh filename=meshes/pelvis_ver0529.STL
Joints:
- removed joint pelvis_contour_joint

File: robots/g1_description/g1_29dof_mode_16.urdf (robot description, URDF)
Before this commit: robot g1_29dof_mode_16, 39 links, 38 joints
Links:
- removed link pelvis_contour_link
- link pelvis: geometry visual mesh filename=meshes/pelvis_ver0529.STL
Joints:
- removed joint pelvis_contour_joint

File: robots/g1_with_brainco_hand/g1_29dof_mode_15_brainco_hand.urdf (robot description, URDF)
Before this commit: robot g1_29dof_mode_15_brainco_hand, 73 links, 72 joints
Links:
- removed link pelvis_contour_link
- link pelvis: geometry visual mesh filename=meshes/pelvis_ver0529.STL
Joints:
- removed joint pelvis_contour_joint

Commit message: fix g1 mid360_joint transform

File: robots/g1_description/g1_23dof_mode_10.urdf (robot description, URDF)
Before this commit: robot g1_23dof_mode_10, 30 links, 29 joints
Joints:
- joint mid360_joint: origin xyz=0.0002835 0.00003 0.41618 rpy=0 0.04014257279586953 0 -> xyz=0.0002835 0.00003 0.428434 rpy=3.141592653589793 0.05112069379091391 0

File: robots/g1_description/g1_23dof_rev_1_0.urdf (robot description, URDF)
Before this commit: robot g1_23dof_rev_1_0, 31 links, 30 joints
Joints:
- joint mid360_joint: origin xyz=0.0002835 0.00003 0.41618 rpy=0 0.04014257279586953 0 -> xyz=0.0002835 0.00003 0.428434 rpy=3.141592653589793 0.05112069379091391 0

File: robots/g1_description/g1_29dof_lock_waist_rev_1_0.urdf (robot description, URDF)
Before this commit: robot g1_29dof_lock_waist_rev_1_0, 39 links, 38 joints
Joints:
- joint mid360_joint: origin xyz=0.0002835 0.00003 0.41618 rpy=0 0.04014257279586953 0 -> xyz=0.0002835 0.00003 0.428434 rpy=3.141592653589793 0.05112069379091391 0

File: robots/g1_description/g1_29dof_lock_waist_with_hand_rev_1_0.urdf (robot description, URDF)
Before this commit: robot g1_29dof_lock_waist_with_hand_rev_1_0, 53 links, 52 joints
Joints:
- joint mid360_joint: origin xyz=0.0002835 0.00003 0.41618 rpy=0 0.04014257279586953 0 -> xyz=0.0002835 0.00003 0.428434 rpy=3.141592653589793 0.05112069379091391 0

File: robots/g1_description/g1_29dof_mode_11.urdf (robot description, URDF)
Before this commit: robot g1_29dof_mode_11, 38 links, 37 joints
Joints:
- joint mid360_joint: origin xyz=0.0002835 0.00003 0.41618 rpy=0 0.04014257279586953 0 -> xyz=0.0002835 0.00003 0.428434 rpy=3.141592653589793 0.05112069379091391 0

File: robots/g1_description/g1_29dof_mode_12.urdf (robot description, URDF)
Before this commit: robot g1_29dof_mode_12, 38 links, 37 joints
Joints:
- joint mid360_joint: origin xyz=0.0002835 0.00003 0.41618 rpy=0 0.04014257279586953 0 -> xyz=0.0002835 0.00003 0.428434 rpy=3.141592653589793 0.05112069379091391 0

File: robots/g1_description/g1_29dof_mode_13.urdf (robot description, URDF)
Before this commit: robot g1_29dof_mode_13, 39 links, 38 joints
Joints:
- joint mid360_joint: origin xyz=0.0002835 0.00003 0.41618 rpy=0 0.04014257279586953 0 -> xyz=0.0002835 0.00003 0.428434 rpy=3.141592653589793 0.05112069379091391 0

File: robots/g1_description/g1_29dof_mode_14.urdf (robot description, URDF)
Before this commit: robot g1_29dof_mode_14, 39 links, 38 joints
Joints:
- joint mid360_joint: origin xyz=0.0002835 0.00003 0.41618 rpy=0 0.04014257279586953 0 -> xyz=0.0002835 0.00003 0.428434 rpy=3.141592653589793 0.05112069379091391 0

File: robots/g1_description/g1_29dof_mode_15.urdf (robot description, URDF)
Before this commit: robot g1_29dof_mode_15, 38 links, 37 joints
Joints:
- joint mid360_joint: origin xyz=0.0002835 0.00003 0.41618 rpy=0 0.04014257279586953 0 -> xyz=0.0002835 0.00003 0.428434 rpy=3.141592653589793 0.05112069379091391 0

File: robots/g1_description/g1_29dof_mode_15_with_dex1_1.urdf (robot description, URDF)
Before this commit: robot g1_29dof_mode_15, 42 links, 41 joints
Joints:
- joint mid360_joint: origin xyz=0.0002835 0.00003 0.41618 rpy=0 0.04014257279586953 0 -> xyz=0.0002835 0.00003 0.428434 rpy=3.141592653589793 0.05112069379091391 0

File: robots/g1_description/g1_29dof_mode_16.urdf (robot description, URDF)
Before this commit: robot g1_29dof_mode_16, 38 links, 37 joints
Joints:
- joint mid360_joint: origin xyz=0.0002835 0.00003 0.41618 rpy=0 0.04014257279586953 0 -> xyz=0.0002835 0.00003 0.428434 rpy=3.141592653589793 0.05112069379091391 0

File: robots/g1_description/g1_29dof_rev_1_0.urdf (robot description, URDF)
Before this commit: robot g1_29dof_rev_1_0, 39 links, 38 joints
Joints:
- joint mid360_joint: origin xyz=0.0002835 0.00003 0.41618 rpy=0 0.04014257279586953 0 -> xyz=0.0002835 0.00003 0.428434 rpy=3.141592653589793 0.05112069379091391 0

File: robots/g1_description/g1_29dof_rev_1_0_with_inspire_hand_DFQ.urdf (robot description, URDF)
Before this commit: robot g1_29dof_rev_1_0_with_inspire_hand_DFQ, 63 links, 62 joints
Joints:
- joint mid360_joint: origin xyz=0.0002835 0.00003 0.41618 rpy=0 0.04014257279586953 0 -> xyz=0.0002835 0.00003 0.428434 rpy=3.141592653589793 0.05112069379091391 0

File: robots/g1_description/g1_29dof_rev_1_0_with_inspire_hand_FTP.urdf (robot description, URDF)
Before this commit: robot g1_29dof_rev_1_0_with_inspire_hand_FTP, 97 links, 96 joints
Joints:
- joint mid360_joint: origin xyz=0.0002835 0.00003 0.41618 rpy=0 0.04014257279586953 0 -> xyz=0.0002835 0.00003 0.428434 rpy=3.141592653589793 0.05112069379091391 0

File: robots/g1_description/g1_29dof_with_hand_rev_1_0.urdf (robot description, URDF)
Before this commit: robot g1_29dof_with_hand_rev_1_0, 53 links, 52 joints
Joints:
- joint mid360_joint: origin xyz=0.0002835 0.00003 0.41618 rpy=0 0.04014257279586953 0 -> xyz=0.0002835 0.00003 0.428434 rpy=3.141592653589793 0.05112069379091391 0

File: robots/g1_description/g1_comp.urdf (robot description, URDF)
Before this commit: robot g1_comp, 34 links, 33 joints
Joints:
- joint mid360_joint: origin xyz=0.0002835 0.00003 0.41618 rpy=0 0.04014257279586953 0 -> xyz=0.0002835 0.00003 0.428434 rpy=3.141592653589793 0.05112069379091391 0
