Commit message: update g1+ motor infos

File: robots/g1_description/g1_29dof_mode_18_with_2dof_head.urdf (robot description, URDF)
Before this commit: robot g1_29dof_mode_18_with_2dof_head, 43 links, 42 joints
Links:
- link waist_yaw_link: mass 0.3537 -> 0.214
Joints:
- joint left_ankle_pitch_joint: limit lower=-0.87267 upper=0.5236 effort=35 velocity=30 -> lower=-0.87267 upper=0.5236 effort=41 velocity=34.1
- joint left_ankle_roll_joint: limit lower=-0.2618 upper=0.2618 effort=35 velocity=30 -> lower=-0.2618 upper=0.2618 effort=41 velocity=34.1
- joint left_elbow_joint: limit lower=-1.0472 upper=2.0944 effort=25 velocity=37 -> lower=-1.0472 upper=2.0944 effort=41 velocity=34.1
- joint left_hip_pitch_joint: limit lower=-2.5307 upper=2.8798 effort=139 velocity=20 -> lower=-2.5307 upper=2.8798 effort=77 velocity=34.9
- joint left_hip_roll_joint: limit lower=-0.5236 upper=2.9671 effort=139 velocity=20 -> lower=-0.5236 upper=2.9671 effort=121 velocity=22.1
- joint left_hip_yaw_joint: limit lower=-2.7576 upper=2.7576 effort=88 velocity=32 -> lower=-2.7576 upper=2.7576 effort=121 velocity=22.1
- joint left_knee_joint: limit lower=-0.087267 upper=2.8798 effort=139 velocity=20 -> lower=-0.087267 upper=2.8798 effort=121 velocity=22.1
- joint left_shoulder_pitch_joint: limit lower=-3.0892 upper=2.6704 effort=100 velocity=26.9 -> lower=-3.0892 upper=2.6704 effort=60 velocity=30.6
- joint left_shoulder_roll_joint: limit lower=-1.5882 upper=2.2515 effort=25 velocity=37 -> lower=-1.5882 upper=2.2515 effort=41 velocity=34.1
- joint left_shoulder_yaw_joint: limit lower=-2.618 upper=2.618 effort=25 velocity=37 -> lower=-2.618 upper=2.618 effort=41 velocity=34.1
- joint left_wrist_pitch_joint: limit lower=-1.614429558 upper=1.614429558 effort=13.4 velocity=27 -> lower=-1.614429558 upper=1.614429558 effort=13.4 velocity=41.5
- joint left_wrist_roll_joint: limit lower=-1.972222054 upper=1.972222054 effort=25 velocity=37 -> lower=-1.972222054 upper=1.972222054 effort=41 velocity=34.1
- joint left_wrist_yaw_joint: limit lower=-1.614429558 upper=1.614429558 effort=13.4 velocity=27 -> lower=-1.614429558 upper=1.614429558 effort=13.4 velocity=41.5
- joint neck_pitch_joint: limit lower=-0.43633 upper=0.62832 effort=25 velocity=37 -> lower=-0.43633 upper=0.62832 effort=41 velocity=34.1
- joint neck_yaw_joint: limit lower=-2.0071 upper=2.0071 effort=13.4 velocity=27 -> lower=-2.0071 upper=2.0071 effort=13.4 velocity=41.5
- joint right_ankle_pitch_joint: limit lower=-0.87267 upper=0.5236 effort=35 velocity=30 -> lower=-0.87267 upper=0.5236 effort=41 velocity=34.1
- joint right_ankle_roll_joint: limit lower=-0.2618 upper=0.2618 effort=35 velocity=30 -> lower=-0.2618 upper=0.2618 effort=41 velocity=34.1
- joint right_elbow_joint: limit lower=-1.0472 upper=2.0944 effort=25 velocity=37 -> lower=-1.0472 upper=2.0944 effort=41 velocity=34.1
- joint right_hip_pitch_joint: limit lower=-2.5307 upper=2.8798 effort=139 velocity=20 -> lower=-2.5307 upper=2.8798 effort=77 velocity=34.9
- joint right_hip_roll_joint: limit lower=-2.9671 upper=0.5236 effort=139 velocity=20 -> lower=-2.9671 upper=0.5236 effort=121 velocity=22.1
- joint right_hip_yaw_joint: limit lower=-2.7576 upper=2.7576 effort=88 velocity=32 -> lower=-2.7576 upper=2.7576 effort=121 velocity=22.1
- joint right_knee_joint: limit lower=-0.087267 upper=2.8798 effort=139 velocity=20 -> lower=-0.087267 upper=2.8798 effort=121 velocity=22.1
- joint right_shoulder_pitch_joint: limit lower=-3.0892 upper=2.6704 effort=100 velocity=26.9 -> lower=-3.0892 upper=2.6704 effort=60 velocity=30.6
- joint right_shoulder_roll_joint: limit lower=-2.2515 upper=1.5882 effort=25 velocity=37 -> lower=-2.2515 upper=1.5882 effort=41 velocity=34.1
- joint right_shoulder_yaw_joint: limit lower=-2.618 upper=2.618 effort=25 velocity=37 -> lower=-2.618 upper=2.618 effort=41 velocity=34.1
- joint right_wrist_pitch_joint: limit lower=-1.614429558 upper=1.614429558 effort=13.4 velocity=27 -> lower=-1.614429558 upper=1.614429558 effort=13.4 velocity=41.5
- joint right_wrist_roll_joint: limit lower=-1.972222054 upper=1.972222054 effort=25 velocity=37 -> lower=-1.972222054 upper=1.972222054 effort=41 velocity=34.1
- joint right_wrist_yaw_joint: limit lower=-1.614429558 upper=1.614429558 effort=13.4 velocity=27 -> lower=-1.614429558 upper=1.614429558 effort=13.4 velocity=41.5
- joint waist_pitch_joint: limit lower=-0.52 upper=0.52 effort=35 velocity=30 -> lower=-0.52 upper=0.52 effort=60 velocity=30.6
- joint waist_roll_joint: limit lower=-0.52 upper=0.52 effort=35 velocity=30 -> lower=-0.52 upper=0.52 effort=60 velocity=30.6; origin xyz=-0.003943 -0.000004 0.047 rpy=0 0 0 -> xyz=-0.0039635 0 0.044 rpy=0 0 0
- joint waist_yaw_joint: limit lower=-2.618 upper=2.618 effort=88 velocity=32 -> lower=-2.618 upper=2.618 effort=77 velocity=34.9
