Commit message: add g1_plus

File: robots/g1_description/g1_plus.urdf (robot description, URDF)
Before this commit: robot g1_29dof_mode_18_with_2dof_head, 43 links, 42 joints
Joints:
- joint left_ankle_pitch_joint: limit lower=-0.87267 upper=0.5236 effort=41 velocity=34.1 -> lower=-0.87267 upper=0.5236 effort=61.5 velocity=34.1
- joint left_ankle_roll_joint: limit lower=-0.2618 upper=0.2618 effort=41 velocity=34.1 -> lower=-0.2618 upper=0.2618 effort=61.5 velocity=34.1
- joint right_ankle_pitch_joint: limit lower=-0.87267 upper=0.5236 effort=41 velocity=34.1 -> lower=-0.87267 upper=0.5236 effort=61.5 velocity=34.1
- joint right_ankle_roll_joint: limit lower=-0.2618 upper=0.2618 effort=41 velocity=34.1 -> lower=-0.2618 upper=0.2618 effort=61.5 velocity=34.1
- joint waist_pitch_joint: limit lower=-0.52 upper=0.52 effort=60 velocity=30.6 -> lower=-0.52 upper=0.52 effort=90 velocity=30.6
- joint waist_roll_joint: limit lower=-0.52 upper=0.52 effort=60 velocity=30.6 -> lower=-0.52 upper=0.52 effort=90 velocity=30.6
