Commit message: Update G1+ hip motor mapping

File: robots/g1_description/g1_pl.urdf (robot description, URDF)
Before this commit: robot g1_pl, 43 links, 42 joints
Joints:
- joint left_hip_pitch_joint: limit lower=-2.5307 upper=2.8798 effort=77 velocity=34.9 -> lower=-2.5307 upper=2.8798 effort=121 velocity=22.1
- joint left_hip_yaw_joint: limit lower=-2.7576 upper=2.7576 effort=121 velocity=22.1 -> lower=-2.7576 upper=2.7576 effort=77 velocity=34.9
- joint right_hip_pitch_joint: limit lower=-2.5307 upper=2.8798 effort=77 velocity=34.9 -> lower=-2.5307 upper=2.8798 effort=121 velocity=22.1
- joint right_hip_yaw_joint: limit lower=-2.7576 upper=2.7576 effort=121 velocity=22.1 -> lower=-2.7576 upper=2.7576 effort=77 velocity=34.9

Commit message: clean g1+

File: robots/g1_description/g1_pl.urdf (robot description, URDF)
Before this commit: robot g1_pl, 43 links, 42 joints
Links:
- removed link d435_link
- removed link mid360_link
Joints:
- removed joint d435_joint
- removed joint mid360_joint
