Commit message: modify knee joint info in go2's urdf

File: robots/go2_description/urdf/go2_description.urdf (robot description, URDF)
Before this commit: robot go2_description, 29 links, 28 joints
Joints:
- joint FL_calf_joint: limit lower=-2.7227 upper=-0.83776 effort=35.55 velocity=20.07 -> lower=-2.7227 upper=-0.83776 effort=45.43 velocity=15.70
- joint FR_calf_joint: limit lower=-2.7227 upper=-0.83776 effort=35.55 velocity=20.07 -> lower=-2.7227 upper=-0.83776 effort=45.43 velocity=15.70
- joint RL_calf_joint: limit lower=-2.7227 upper=-0.83776 effort=35.55 velocity=20.07 -> lower=-2.7227 upper=-0.83776 effort=45.43 velocity=15.70
- joint RR_calf_joint: limit lower=-2.7227 upper=-0.83776 effort=35.55 velocity=20.07 -> lower=-2.7227 upper=-0.83776 effort=45.43 velocity=15.70

Commit message: add go2 rotor inertial to g2's urdf

File: robots/go2_description/urdf/go2_description.urdf (robot description, URDF)
Before this commit: robot go2_description, 29 links, 28 joints
Links:
- added link FL_calf_rotor, mass 0.089
- added link FL_hip_rotor, mass 0.089
- added link FL_thigh_rotor, mass 0.089
- added link FR_calf_rotor, mass 0.089
- added link FR_hip_rotor, mass 0.089
- added link FR_thigh_rotor, mass 0.089
- added link RL_calf_rotor, mass 0.089
- added link RL_hip_rotor, mass 0.089
- added link RL_thigh_rotor, mass 0.089
- added link RR_calf_rotor, mass 0.089
- added link RR_hip_rotor, mass 0.089
- added link RR_thigh_rotor, mass 0.089
Joints:
- added joint FL_calf_rotor_joint: type fixed, parent FL_thigh, child FL_calf_rotor, origin xyz=0 -0.03235 0 rpy=0 0 0
- added joint FL_hip_rotor_joint: type fixed, parent base, child FL_hip_rotor, origin xyz=0.11215 0.04675 0 rpy=0 0 0
- added joint FL_thigh_rotor_joint: type fixed, parent FL_hip, child FL_thigh_rotor, origin xyz=0 -0.00015 0 rpy=0 0 0
- added joint FR_calf_rotor_joint: type fixed, parent FR_thigh, child FR_calf_rotor, origin xyz=0 0.03235 0 rpy=0 0 0
- added joint FR_hip_rotor_joint: type fixed, parent base, child FR_hip_rotor, origin xyz=0.11215 -0.04675 0 rpy=0 0 0
- added joint FR_thigh_rotor_joint: type fixed, parent FR_hip, child FR_thigh_rotor, origin xyz=0 0.00015 0 rpy=0 0 0
- added joint RL_calf_rotor_joint: type fixed, parent RL_thigh, child RL_calf_rotor, origin xyz=0 -0.03235 0 rpy=0 0 0
- added joint RL_hip_rotor_joint: type fixed, parent base, child RL_hip_rotor, origin xyz=-0.11215 0.04675 0 rpy=0 0 0
- added joint RL_thigh_rotor_joint: type fixed, parent RL_hip, child RL_thigh_rotor, origin xyz=0 -0.00015 0 rpy=0 0 0
- added joint RR_calf_rotor_joint: type fixed, parent RR_thigh, child RR_calf_rotor, origin xyz=0 0.03235 0 rpy=0 0 0
- added joint RR_hip_rotor_joint: type fixed, parent base, child RR_hip_rotor, origin xyz=-0.11215 -0.04675 0 rpy=0 0 0
- added joint RR_thigh_rotor_joint: type fixed, parent RR_hip, child RR_thigh_rotor, origin xyz=0 0.00015 0 rpy=0 0 0

Commit message: add go2 front_camera link

File: robots/go2_description/urdf/go2_description.urdf (robot description, URDF)
Before this commit: robot go2_description, 41 links, 40 joints
Links:
- added link front_camera
Joints:
- added joint front_camera_joint: type fixed, parent base, child front_camera, origin xyz=0.32715 -0.00003 0.04297 rpy=0 0 0

File: robots/go2_description/xacro/robot.xacro (robot description, xacro)
@@ -81,4 +81,11 @@
         </collision>
     </link>
+    <joint name="front_camera_joint" type="fixed">
+        <parent link="trunk"/>
+        <child link="front_camera"/>
+        <origin rpy="0 0 0" xyz="0.32715 -0.00003 0.04297"/>
+    </joint>
+    <link name="front_camera">
+    </link>
     <!--
     <joint name="load_joint" type="fixed">
