Commit message: update dex3_1 joint limit

File: robots/dexterous_hand_description/dex3_1/dex3_1_l.urdf (robot description, URDF)
Before this commit: robot dex3_1_l, 8 links, 7 joints
Joints:
- joint left_hand_thumb_1_joint: limit lower=-0.72431163 upper=1.04719755 effort=1.4 velocity=12 -> lower=-0.61086523 upper=1.04719755 effort=1.4 velocity=12

File: robots/dexterous_hand_description/dex3_1/dex3_1_r.urdf (robot description, URDF)
Before this commit: robot dex3_1_r, 8 links, 7 joints
Joints:
- joint right_hand_thumb_1_joint: limit lower=-1.04719755 upper=0.72431163 effort=1.4 velocity=12 -> lower=-1.04719755 upper=0.61086523 effort=1.4 velocity=12

File: robots/g1_description/g1_29dof_lock_waist_with_hand_rev_1_0.urdf (robot description, URDF)
Before this commit: robot g1_29dof_lock_waist_with_hand_rev_1_0, 53 links, 52 joints
Joints:
- joint left_hand_thumb_1_joint: limit lower=-0.72431163 upper=1.04719755 effort=1.4 velocity=12 -> lower=-0.61086523 upper=1.04719755 effort=1.4 velocity=12
- joint right_hand_thumb_1_joint: limit lower=-1.04719755 upper=0.72431163 effort=1.4 velocity=12 -> lower=-1.04719755 upper=0.61086523 effort=1.4 velocity=12

File: robots/g1_description/g1_29dof_with_hand.urdf (robot description, URDF)
Before this commit: robot g1_29dof_with_hand, 54 links, 53 joints
Joints:
- joint left_hand_thumb_1_joint: limit lower=-0.72431163 upper=1.04719755 effort=1.4 velocity=12 -> lower=-0.61086523 upper=1.04719755 effort=1.4 velocity=12
- joint right_hand_thumb_1_joint: limit lower=-1.04719755 upper=0.72431163 effort=1.4 velocity=12 -> lower=-1.04719755 upper=0.61086523 effort=1.4 velocity=12

File: robots/g1_description/g1_29dof_with_hand_rev_1_0.urdf (robot description, URDF)
Before this commit: robot g1_29dof_with_hand_rev_1_0, 53 links, 52 joints
Joints:
- joint left_hand_thumb_1_joint: limit lower=-0.72431163 upper=1.04719755 effort=1.4 velocity=12 -> lower=-0.61086523 upper=1.04719755 effort=1.4 velocity=12
- joint right_hand_thumb_1_joint: limit lower=-1.04719755 upper=0.72431163 effort=1.4 velocity=12 -> lower=-1.04719755 upper=0.61086523 effort=1.4 velocity=12
