Commit message: update dex5 urdf

File: robots/dexterous_hand_description/dex5_1/Dex5-URDF-L/Dex5-URDF-L.urdf (robot description, URDF)
Before this commit: robot Dex5-URDF-L, 21 links, 20 joints
Links:
- removed link base_link_L
- added link base_link00L, mass 0.732177466301149; collision mesh filename=meshes/base_link00L.STL; visual mesh filename=meshes/base_link00L.STL
Joints:
- joint Link_41L: parent base_link_L -> base_link00L
- joint Pitch_13L: limit lower=0 upper=1.9548 effort=0.93 velocity=4.18 -> lower=0 upper=1.7652 effort=0.93 velocity=4.18
- joint Roll_21L: parent base_link_L -> base_link00L
- joint Roll_31L: parent base_link_L -> base_link00L
- joint Roll_51L: parent base_link_L -> base_link00L
- joint Yaw_11L: limit lower=-0.57596 upper=0.76794 effort=0.93 velocity=4.18 -> lower=-0.5867 upper=0.6803 effort=0.93 velocity=4.18; parent base_link_L -> base_link00L

File: robots/dexterous_hand_description/dex5_1/Dex5-URDF-R/Dex5-URDF-R.urdf (robot description, URDF)
Before this commit: robot Dex5-URDF-R, 21 links, 20 joints
Links:
- removed link base_link_R
- added link base_link00, mass 0.685702; collision mesh filename=meshes/base_link00.STL; visual mesh filename=meshes/base_link00.STL
Joints:
- joint Pitch_13R: limit lower=0 upper=1.9548 effort=0.93 velocity=4.18 -> lower=0 upper=1.765226 effort=0.93 velocity=4.18
- joint Roll_21R: parent base_link_R -> base_link00
- joint Roll_31R: parent base_link_R -> base_link00
- joint Roll_41R: parent base_link_R -> base_link00
- joint Roll_51R: parent base_link_R -> base_link00
- joint Yaw_11R: limit lower=-0.57596 upper=0.76794 effort=0.93 velocity=4.18 -> lower=-0.5867 upper=0.6803 effort=0.93 velocity=4.18; parent base_link_R -> base_link00
