Commit message: feat: Changed tip joints to fixed instead of locked revolute joints
Signed-off-by: Tanner, Gilbert <gilbertta@edu.aau.at>

File: robots/g1_with_brainco_hand/g1_29dof_mode_15_brainco_hand.urdf (robot description, URDF)
Before this commit: robot g1_29dof_mode_15_brainco_hand, 73 links, 72 joints
Links:
- removed link left_index_distal_Link
- removed link left_index_proximal_Link
- removed link left_index_tip_Link
- removed link left_middle_distal_Link
- removed link left_middle_proximal_Link
- removed link left_middle_tip_Link
- removed link left_pinky_distal_Link
- removed link left_pinky_proximal_Link
- removed link left_pinky_tip_Link
- removed link left_ring_distal_Link
- removed link left_ring_proximal_Link
- removed link left_ring_tip_Link
- removed link left_thumb_distal_Link
- removed link left_thumb_metacarpal_Link
- removed link left_thumb_proximal_Link
- removed link left_thumb_tip_Link
- added link left_index_distal_link, mass 0.009; collision mesh filename=meshes/left_index_distal_link.STL; visual mesh filename=meshes/left_index_distal_link.STL
- added link left_index_proximal_link, mass 0.009; collision mesh filename=meshes/left_index_proximal_link.STL; visual mesh filename=meshes/left_index_proximal_link.STL
- added link left_index_tip_link, mass 0.001; collision mesh filename=meshes/left_index_tip_link.STL; visual mesh filename=meshes/left_index_tip_link.STL
- added link left_middle_distal_link, mass 0.009; collision mesh filename=meshes/left_middle_distal_link.STL; visual mesh filename=meshes/left_middle_distal_link.STL
- added link left_middle_proximal_link, mass 0.009; collision mesh filename=meshes/left_middle_proximal_link.STL; visual mesh filename=meshes/left_middle_proximal_link.STL
- added link left_middle_tip_link, mass 0.001; collision mesh filename=meshes/left_middle_tip_link.STL; visual mesh filename=meshes/left_middle_tip_link.STL
- added link left_pinky_distal_link, mass 0.009; collision mesh filename=meshes/left_pinky_distal_link.STL; visual mesh filename=meshes/left_pinky_distal_link.STL
- added link left_pinky_proximal_link, mass 0.009; collision mesh filename=meshes/left_pinky_proximal_link.STL; visual mesh filename=meshes/left_pinky_proximal_link.STL
- added link left_pinky_tip_link, mass 0.001; collision mesh filename=meshes/left_pinky_tip_link.STL; visual mesh filename=meshes/left_pinky_tip_link.STL
- added link left_ring_distal_link, mass 0.009; collision mesh filename=meshes/left_ring_distal_link.STL; visual mesh filename=meshes/left_ring_distal_link.STL
- added link left_ring_proximal_link, mass 0.009; collision mesh filename=meshes/left_ring_proximal_link.STL; visual mesh filename=meshes/left_ring_proximal_link.STL
- added link left_ring_tip_link, mass 0.001; collision mesh filename=meshes/left_ring_tip_link.STL; visual mesh filename=meshes/left_ring_tip_link.STL
- added link left_thumb_distal_link, mass 0.01; collision mesh filename=meshes/left_thumb_distal_link.STL; visual mesh filename=meshes/left_thumb_distal_link.STL
- added link left_thumb_metacarpal_link, mass 0.01; collision mesh filename=meshes/left_thumb_metacarpal_link.STL; visual mesh filename=meshes/left_thumb_metacarpal_link.STL
- added link left_thumb_proximal_link, mass 0.05; collision mesh filename=meshes/left_thumb_proximal_link.STL; visual mesh filename=meshes/left_thumb_proximal_link.STL
- added link left_thumb_tip_link, mass 0.001; collision mesh filename=meshes/left_thumb_tip_link.STL; visual mesh filename=meshes/left_thumb_tip_link.STL
Joints:
- joint left_index_distal_joint: child left_index_distal_Link -> left_index_distal_link; parent left_index_proximal_Link -> left_index_proximal_link
- joint left_index_proximal_joint: child left_index_proximal_Link -> left_index_proximal_link
- joint left_index_tip_joint: axis 0 1 0 -> (none); child left_index_tip_Link -> left_index_tip_link; limit lower=1 upper=1 effort=1 velocity=1 -> (none); parent left_index_distal_Link -> left_index_distal_link; type revolute -> fixed
- joint left_middle_distal_joint: child left_middle_distal_Link -> left_middle_distal_link; parent left_middle_proximal_Link -> left_middle_proximal_link
- joint left_middle_proximal_joint: child left_middle_proximal_Link -> left_middle_proximal_link
- joint left_middle_tip_joint: axis 0 1 0 -> (none); child left_middle_tip_Link -> left_middle_tip_link; limit lower=1 upper=1 effort=1 velocity=1 -> (none); parent left_middle_distal_Link -> left_middle_distal_link; type revolute -> fixed
- joint left_pinky_distal_joint: child left_pinky_distal_Link -> left_pinky_distal_link; parent left_pinky_proximal_Link -> left_pinky_proximal_link
- joint left_pinky_proximal_joint: child left_pinky_proximal_Link -> left_pinky_proximal_link
- joint left_pinky_tip_joint: axis 0 1 0 -> (none); child left_pinky_tip_Link -> left_pinky_tip_link; limit lower=1 upper=1 effort=1 velocity=1 -> (none); parent left_pinky_distal_Link -> left_pinky_distal_link; type revolute -> fixed
- joint left_ring_distal_joint: child left_ring_distal_Link -> left_ring_distal_link; parent left_ring_proximal_Link -> left_ring_proximal_link
- joint left_ring_proximal_joint: child left_ring_proximal_Link -> left_ring_proximal_link
- joint left_ring_tip_joint: axis 0 1 0 -> (none); child left_ring_tip_Link -> left_ring_tip_link; limit lower=1 upper=1 effort=1 velocity=1 -> (none); parent left_ring_distal_Link -> left_ring_distal_link; type revolute -> fixed
- joint left_thumb_distal_joint: child left_thumb_distal_Link -> left_thumb_distal_link; parent left_thumb_proximal_Link -> left_thumb_proximal_link
- joint left_thumb_metacarpal_joint: child left_thumb_metacarpal_Link -> left_thumb_metacarpal_link
- joint left_thumb_proximal_joint: child left_thumb_proximal_Link -> left_thumb_proximal_link; parent left_thumb_metacarpal_Link -> left_thumb_metacarpal_link
- joint left_thumb_tip_joint: axis -1 0 0 -> (none); child left_thumb_tip_Link -> left_thumb_tip_link; limit lower=0 upper=0 effort=0 velocity=0 -> (none); parent left_thumb_distal_Link -> left_thumb_distal_link; type revolute -> fixed
- joint right_index_tip_joint: axis 0 1 0 -> (none); limit lower=0 upper=0 effort=0 velocity=0 -> (none); type revolute -> fixed
- joint right_middle_tip_joint: axis 0 1 0 -> (none); limit lower=0 upper=0 effort=0 velocity=0 -> (none); type revolute -> fixed
- joint right_pinky_tip_joint: axis 0 1 0 -> (none); limit lower=0 upper=0 effort=0 velocity=0 -> (none); type revolute -> fixed
- joint right_ring_tip_joint: axis 0 1 0 -> (none); limit lower=0 upper=0 effort=0 velocity=0 -> (none); type revolute -> fixed
- joint right_thumb_tip_joint: axis 1 0 0 -> (none); limit lower=0 upper=0 effort=0 velocity=0 -> (none); type revolute -> fixed

Commit message: chore: Ensure naming between left and right hand is consistent
Signed-off-by: Tanner, Gilbert <gilbertta@edu.aau.at>

File: robots/g1_with_brainco_hand/g1_29dof_mode_15_brainco_hand.urdf (robot description, URDF)
Before this commit: robot g1_29dof_mode_15_brainco_hand, 73 links, 72 joints
Links:
- removed link right_index_tip
- removed link right_middle_tip
- removed link right_pinky_tip
- removed link right_ring_tip
- removed link right_thumb_tip
- added link right_index_tip_link, mass 0.001; collision mesh filename=meshes/right_index_tip_link.STL; visual mesh filename=meshes/right_index_tip_link.STL
- added link right_middle_tip_link, mass 0.001; collision mesh filename=meshes/right_middle_tip_link.STL; visual mesh filename=meshes/right_middle_tip_link.STL
- added link right_pinky_tip_link, mass 0.001; collision mesh filename=meshes/right_pinky_tip_link.STL; visual mesh filename=meshes/right_pinky_tip_link.STL
- added link right_ring_tip_link, mass 0.001; collision mesh filename=meshes/right_ring_tip_link.STL; visual mesh filename=meshes/right_ring_tip_link.STL
- added link right_thumb_tip_link, mass 0.001; collision mesh filename=meshes/right_thumb_tip_link.STL; visual mesh filename=meshes/right_thumb_tip_link.STL
- link d435_link: geometry visual sphere radius=0.001
- link imu_in_pelvis: geometry visual sphere radius=0.001
- link imu_in_torso: geometry visual sphere radius=0.001
- link mid360_link: geometry visual sphere radius=0.001
Joints:
- joint right_index_tip_joint: child right_index_tip -> right_index_tip_link
- joint right_middle_tip_joint: child right_middle_tip -> right_middle_tip_link
- joint right_pinky_tip_joint: child right_pinky_tip -> right_pinky_tip_link
- joint right_ring_tip_joint: child right_ring_tip -> right_ring_tip_link
- joint right_thumb_tip_joint: child right_thumb_tip -> right_thumb_tip_link
