Commit message: update h2 r1 r1air urdf

File: robots/r1_air_description/R1_AIR.urdf (robot description, URDF)
Before this commit: robot R1_AIR, 34 links, 33 joints
Links:
- link left_elbow_link: mass 0.986213 -> 0.655100
- link left_shoulder_yaw_link: mass 0.738441 -> 0.725600
- link pelvis_link: mass 6.988703 -> 9.134
- link right_elbow_link: mass 0.986213 -> 0.655100
- link right_shoulder_yaw_link: mass 0.738441 -> 0.725600
