Commit message: update R1 head `<inertial>`

File: robots/r1_description/R1.urdf (robot description, URDF)
Before this commit: robot R1, 40 links, 39 joints
Links:
- link head_pitch_link: mass 0.39234316 -> 0.50391253
- link head_yaw_link: mass 0.92216186 -> 0.71432240
- link left_hip_roll_link: mass  0.207609 -> 0.207609
- link right_hip_roll_link: mass  0.207609 -> 0.207609
