Commit message: update R1

File: robots/r1_description/R1.urdf (robot description, URDF)
Before this commit: robot R1, 40 links, 39 joints
Links:
- added link camera_link, mass 0.00224; collision mesh filename=meshes/camera_link.STL; visual mesh filename=meshes/camera_link.STL
- link waist_yaw_link: mass 6.024198 -> 6.324198
Joints:
- added joint camera_joint: type fixed, parent head_yaw_link, child camera_link, origin xyz=0.066971 0 -0.021637 rpy=0 0.34907 0, axis 0 0 0
- joint head_yaw_joint: limit lower=-2.0071 upper=2.0071 effort=33 velocity=33.4 -> lower=-2.0071 upper=2.0071 effort=0.86 velocity=11
- joint left_shoulder_pitch_joint: limit lower=-3.1416 upper=2.0944 effort=60 velocity=18.8 -> lower=-3.1416 upper=2.0944 effort=60 velocity=18.7
- joint left_shoulder_roll_joint: limit lower=-0.22689 upper=2.4784 effort=60 velocity=18.8 -> lower=-0.22689 upper=2.4784 effort=60 velocity=18.7
- joint right_shoulder_pitch_joint: limit lower=-3.1416 upper=2.0944 effort=60 velocity=18.8 -> lower=-3.1416 upper=2.0944 effort=60 velocity=18.7
- joint right_shoulder_roll_joint: limit lower=-2.47849 upper=0.2268 effort=60 velocity=18.8 -> lower=-2.47849 upper=0.2268 effort=60 velocity=18.7
- joint waist_yaw_joint: limit lower=-2.618 upper=2.618 effort=60 velocity=18.8 -> lower=-2.618 upper=2.618 effort=60 velocity=18.7
