Commit message: update h2 urdf

File: robots/h2_description/H2.urdf (robot description, URDF)
Before this commit: robot H2, 32 links, 31 joints
Links:
- link left_ankle_pitch_link: mass 0.84496747 -> 0.89496747
- link left_elbow_link: mass 1.69431869 -> 1.70611556
- link left_hip_pitch_link: mass 2.79752530 -> 2.8737
- link left_hip_roll_link: mass 0.62714607 -> 0.78507858
- link left_hip_yaw_link: mass 7.08752046 -> 7.0875
- link left_knee_link: mass 3.55340244 -> 4.35340244
- link left_shoulder_pitch_link: mass 1.06055553 -> 1.1927
- link left_shoulder_roll_link: mass 1.34511054 -> 1.10982649
- link left_shoulder_yaw_link: mass 0.91571732 -> 0.35273875
- link left_wrist_pitch_link: mass 0.94695328 -> 0.61525753
- link left_wrist_roll_link: mass 0.96983674 -> 0.77425984
- link left_wrist_yaw_link: mass 0.60575230 -> 0.61608207
- link pelvis: mass 7.60468095 -> 8.5477
- link right_ankle_pitch_link: mass 0.84496747 -> 0.89496747
- link right_elbow_link: mass 1.69431869 -> 1.7061723
- link right_hip_pitch_link: mass 2.79752530 -> 2.8737
- link right_hip_roll_link: mass 0.62714607 -> 0.75122
- link right_hip_yaw_link: mass 7.08752046 -> 7.0875
- link right_knee_link: mass 3.55340244 -> 4.35340244
- link right_shoulder_pitch_link: mass 1.06055553 -> 1.1927
- link right_shoulder_roll_link: mass 1.34511054 -> 1.10982142
- link right_shoulder_yaw_link: mass 0.91571732 -> 0.35274186
- link right_wrist_pitch_link: mass 0.94695328 -> 0.61583659
- link right_wrist_roll_link: mass 0.96983674 -> 0.77426501
- link right_wrist_yaw_link: mass 0.60575230 -> 0.6160821
- link torso_link: mass 15.87026294 -> 18.532
- link waist_roll_link: mass 0.06585040 -> 0.13841947
- link waist_yaw_link: mass 0.27976220 -> 0.31293574
Joints:
- joint head_pitch_joint: origin xyz=-0.00011475 0.020709 0.42181 rpy=0 0 0 -> xyz=-0.0001147 -0.0189 0.4218 rpy=0 0 0
- joint head_yaw_joint: origin xyz=0 -0.0189 0.1325 rpy=0 0 0 -> xyz=0 0.0189 0.1335 rpy=0 0 0
- joint left_ankle_pitch_joint: origin xyz=0 -0.0368 0 rpy=0 0 0 -> xyz=-0.014516 -0.0373 0 rpy=0 0 0
- joint left_ankle_roll_joint: origin xyz=0.018383 0 -0.49662 rpy=0 0 0 -> xyz=0.032719 -0.023002 -0.49662 rpy=0 0 0
- joint left_elbow_joint: limit lower=-0.986111 upper=3.0717795 effort=54 velocity=34.3 -> lower=-0.986 upper=3.071 effort=60 velocity=18.7; origin xyz=0.015424 0.020635 -0.13364 rpy=0 0 0 -> xyz=0.016655 0.02211 -0.12792 rpy=0 0 0
- joint left_hip_pitch_joint: origin xyz=0 0.0819279 -0.043723 rpy=-0.5236 0 0 -> xyz=0 0.08038 -0.046407 rpy=-0.5236 0 0
- joint left_hip_roll_joint: origin xyz=0.018422 0.0635 -0.022095 rpy=0.5236 0 0 -> xyz=0.041774 0.0635 -0.019 rpy=0.5236 0 0
- joint left_hip_yaw_joint: origin xyz=-0.0047433 -0.0057328 -0.075875 rpy=0 0 0 -> xyz=-0.028187 -0.0095 -0.0737 rpy=0 0 0
- joint left_knee_joint: origin xyz=-0.010386 -0.0042181 -0.31742 rpy=0 0 0 -> xyz=-0.010308 0.022549 -0.31959 rpy=0 0 0
- joint left_shoulder_pitch_joint: limit lower=-2.6179939 upper=1.8325957 effort=120 velocity=28.375 -> lower=-2.618 upper=1.833 effort=130 velocity=21.9; origin xyz=0.0019779 0.11553 0.35792 rpy=0.26914 0 0 -> xyz=0.0030848 0.11 0.36008 rpy=0.26914 0 0
- joint left_shoulder_roll_joint: limit lower=-0.5166175 upper=2.6354472 effort=54 velocity=34.3 -> lower=-0.517 upper=2.494 effort=60 velocity=18.7; origin xyz=-0.00082158 0.060413 -0.040043 rpy=-0.26914 0 0 -> xyz=-0.0032074 0.059938 -0.039865 rpy=-0.26914 0 0
- joint left_shoulder_yaw_joint: limit lower=-2.6179939 upper=2.6179939 effort=54 velocity=34.3 -> lower=-2.618 upper=2.618 effort=60 velocity=18.7; origin xyz=-0.0025946 0.0038061 -0.09623 rpy=0 0 0 -> xyz=-0.0025601 0.0036752 -0.10421 rpy=0 0 0
- joint left_wrist_pitch_joint: limit lower=-0.4363323 upper=0.4363323 effort=25 velocity=50.125 -> lower=-0.576 upper=0.576 effort=10 velocity=37.7; origin xyz=0.080589 3.0398E-05 -0.0013317 rpy=0 0 0 -> xyz=0.037994 0.031144 0.00045104 rpy=0 0 0
- joint left_wrist_roll_joint: limit lower=-2.6179939 upper=2.6179939 effort=54 velocity=34.3 -> lower=-2.618 upper=2.618 effort=60 velocity=18.7; origin xyz=0.13119 -0.021207 -0.013343 rpy=0 0 0 -> xyz=0.13119 -0.021497 -0.013769 rpy=0 0 0
- joint left_wrist_yaw_joint: limit lower=-1.2217305 upper=1.2217305 effort=25 velocity=50.125 -> lower=-1.22 upper=1.22 effort=60 velocity=37.7; origin xyz=0.028225 0.00048901 0.00058318 rpy=0 0 0 -> xyz=0.069283 -0.031045 -0.0006247 rpy=0 0 0
- joint right_ankle_pitch_joint: origin xyz=0 0.0373 0 rpy=0 0 0 -> xyz=-0.014516 0.0373 0 rpy=0 0 0
- joint right_ankle_roll_joint: origin xyz=0.018383 0 -0.49662 rpy=0 0 0 -> xyz=0.032719 0.023002 -0.49662 rpy=0 0 0
- joint right_elbow_joint: limit lower=-0.986111 upper=3.0717795 effort=54 velocity=34.3 -> lower=-0.986 upper=3.071 effort=60 velocity=18.7; origin xyz=0.015346 -0.020599 -0.13363 rpy=0 0 0 -> xyz=0.016655 -0.02211 -0.12792 rpy=0 0 0
- joint right_hip_pitch_joint: origin xyz=0 -0.0803801 -0.046403 rpy=0.5236 0 0 -> xyz=0 -0.08038 -0.046407 rpy=0.5236 0 0
- joint right_hip_roll_joint: origin xyz=0.037774 -0.0635 -0.019 rpy=-0.5236 0 0 -> xyz=0.041774 -0.0635 -0.019 rpy=-0.5236 0 0
- joint right_hip_yaw_joint: origin xyz=-0.024111 0.0057328 -0.075875 rpy=0 0 0 -> xyz=-0.028187 0.0095 -0.0737 rpy=0 0 0
- joint right_knee_joint: origin xyz=-0.010386 0.0042181 -0.31742 rpy=0 0 0 -> xyz=-0.010308 -0.022549 -0.31959 rpy=0 0 0
- joint right_shoulder_pitch_joint: limit lower=-2.6179939 upper=1.8325957 effort=120 velocity=28.375 -> lower=-2.618 upper=1.833 effort=130 velocity=21.9; origin xyz=0.0019706 -0.11185 0.35789 rpy=-0.26914 0 0 -> xyz=0.0030848 -0.11 0.36008 rpy=-0.26914 0 0
- joint right_shoulder_roll_joint: limit lower=-2.6354472 upper=0.5166175 effort=54 velocity=34.3 -> lower=-2.494 upper=0.517 effort=60 velocity=18.7; origin xyz=-0.00082577 -0.060403 -0.040059 rpy=0.26914 0 0 -> xyz=-0.0032074 -0.059938 -0.039865 rpy=0.26914 0 0
- joint right_shoulder_yaw_joint: limit lower=-2.6179939 upper=2.6179939 effort=54 velocity=34.3 -> lower=-2.618 upper=2.618 effort=60 velocity=18.7; origin xyz=-0.0025949 -0.0037808 -0.096231 rpy=0 0 0 -> xyz=-0.0025601 -0.0036752 -0.10421 rpy=0 0 0
- joint right_wrist_pitch_joint: limit lower=-0.4363323 upper=0.4363323 effort=25 velocity=50.125 -> lower=-0.576 upper=0.576 effort=10 velocity=37.7; origin xyz=0.076351 -0.00015864 0.0011464 rpy=0 0 0 -> xyz=0.037994 -0.031144 0.00045104 rpy=0 0 0
- joint right_wrist_roll_joint: limit lower=-2.6179939 upper=2.6179939 effort=54 velocity=34.3 -> lower=-2.618 upper=2.618 effort=60 velocity=18.7; origin xyz=0.13177 0.021197 -0.013782 rpy=0 0 0 -> xyz=0.13119 0.021497 -0.013769 rpy=0 0 0
- joint right_wrist_yaw_joint: limit lower=-1.2217305 upper=1.2217305 effort=25 velocity=50.125 -> lower=-1.22 upper=1.22 effort=10 velocity=37.7; origin xyz=0.028195 5.8414E-05 -0.0012184 rpy=0 0 0 -> xyz=0.069283 0.031045 -0.0006247 rpy=0 0 0
- joint waist_roll_joint: origin xyz=0 -0.0015099 0.0325 rpy=0 0 0 -> xyz=0 0 0.0325 rpy=0 0 0
- joint waist_yaw_joint: origin xyz=0 0.0015099 0.090537 rpy=0 0 0 -> xyz=0 0 0.090537 rpy=0 0 0

Commit message: fix h2 max effort

File: robots/h2_description/H2.urdf (robot description, URDF)
Before this commit: robot H2, 32 links, 31 joints
Joints:
- joint left_wrist_yaw_joint: limit lower=-1.22 upper=1.22 effort=60 velocity=37.7 -> lower=-1.22 upper=1.22 effort=10 velocity=37.7

Commit message: update h2_description

File: robots/h2_description/H2.urdf (robot description, URDF)
Before this commit: robot H2, 32 links, 31 joints
Links:
- added link left_hand_link, mass 0.41885723; collision mesh filename=meshes/left_hand_link.stl; visual mesh filename=meshes/left_hand_link.stl
- added link right_hand_link, mass 0.41885723; collision mesh filename=meshes/right_hand_link.stl; visual mesh filename=meshes/right_hand_link.stl
- link left_wrist_yaw_link: mass 0.61608207 -> 0.19722487
- link right_wrist_yaw_link: mass 0.6160821 -> 0.19722487
Joints:
- added joint left_hand_joint: type fixed, parent left_wrist_yaw_link, child left_hand_link, origin xyz=0.05771524 0 -0.00014865 rpy=0 0 0
- added joint right_hand_joint: type fixed, parent right_wrist_yaw_link, child right_hand_link, origin xyz=0.05824125 0 -0.00017221 rpy=0 0 0

File: robots/h2_description/H2_dae.urdf (robot description, URDF)
Before this commit: robot H2, 32 links, 31 joints
Links:
- added link left_hand_link, mass 0.41885723; collision mesh filename=meshes/left_hand_link.stl; visual mesh filename=meshes/left_hand_link.dae
- added link right_hand_link, mass 0.41885723; collision mesh filename=meshes/right_hand_link.stl; visual mesh filename=meshes/right_hand_link.dae
- link left_wrist_yaw_link: mass 0.61608207 -> 0.19722487
- link right_wrist_yaw_link: mass 0.6160821 -> 0.19722487
Joints:
- added joint left_hand_joint: type fixed, parent left_wrist_yaw_link, child left_hand_link, origin xyz=0.05771524 0 -0.00014865 rpy=0 0 0
- added joint right_hand_joint: type fixed, parent right_wrist_yaw_link, child right_hand_link, origin xyz=0.05824125 0 -0.00017221 rpy=0 0 0
