Commit message: add a2 camera and lidar link

File: robots/a2_description/urdf/a2.urdf (robot description, URDF)
Before this commit: robot a2, 17 links, 16 joints
Links:
- added link camera_link
- added link front_lidar_link
- added link rear_lidar_link
Joints:
- added joint camera_joint: type fixed, parent base_link, child camera_link, origin xyz=0.3381 0.0336 0.0525 rpy=0 0 0
- added joint front_lidar_joint: type fixed, parent base_link, child front_lidar_link, origin xyz=0.33767 0.0 0.08134 rpy=1.5708 0 1.5708
- added joint rear_lidar_joint: type fixed, parent front_lidar_link, child rear_lidar_link, origin xyz=0.0 0.005997 -0.617643765 rpy=0 3.14159 0
