Commit message: update R1 A5

File: robots/r1_a5_description/r1_a5.urdf (robot description, URDF)
Before this commit: robot A5, 14 links, 13 joints
Links:
- added link camera_link, mass 0.00224; collision mesh filename=meshes/camera_link.STL; visual mesh filename=meshes/camera_link.STL
- link waist_yaw_link: mass 6.024198 -> 6.324198
Joints:
- added joint camera_joint: type fixed, parent head_yaw_link, child camera_link, origin xyz=0.066971 0 -0.021637 rpy=0 0.349066 0, axis 0 0 0
