Commit message: update R1 A7

File: robots/r1_a7_description/r1_a7.urdf (robot description, URDF)
Before this commit: robot A7, 18 links, 17 joints
Links:
- added link camera_link, mass 0.024; collision mesh filename=meshes/camera_link.STL; visual mesh filename=meshes/camera_link.STL
- link left_wrist_yaw_link: mass 0.63414044 -> 0.08314044
- link right_wrist_yaw_link: mass 0.63414044 -> 0.08314044
- link waist_yaw_link: mass 6.024198 -> 6.384198
Joints:
- added joint camera_joint: type fixed, parent head_yaw_link, child camera_link, origin xyz=0.066971 0 -0.021637 rpy=0 0.34907 0, axis 0 0 0
