Commit message: update h2x

File: robots/h2x_description/h2x.urdf (robot description, URDF)
Before this commit: robot H2-X, 50 links, 49 joints
Joints:
- joint left_ankle_lower_motor_joint: limit lower=-1.1 upper=1.1 effort=53.7 velocity=29.6333 -> (none); type revolute -> fixed
- joint left_ankle_upper_motor_joint: limit lower=-1.1 upper=1.1 effort=53.7 velocity=29.6333 -> (none); type revolute -> fixed
- joint left_waist_motor_joint: limit lower=-1.3 upper=0.7 effort=111.0 velocity=22.7 -> (none); type revolute -> fixed
- joint right_ankle_lower_motor_joint: limit lower=-1.1 upper=1.1 effort=53.7 velocity=29.6333 -> (none); type revolute -> fixed
- joint right_ankle_upper_motor_joint: limit lower=-1.1 upper=1.1 effort=53.7 velocity=29.6333 -> (none); type revolute -> fixed
- joint right_waist_motor_joint: limit lower=-0.7 upper=1.3 effort=111.0 velocity=22.7 -> (none); type revolute -> fixed
