Commit message: update h2d

File: robots/h2d_description/h2d.urdf (robot description, URDF)
Before this commit: robot H2D, 28 links, 27 joints
Links:
- link pelvis_link: mass 97.063 -> 86.0
Joints:
- joint head_pitch_joint: axis 0 -1 0 -> 0 1 0; limit lower=-0.5236 upper=0.83775 effort=50 velocity=10 -> lower=-0.83775 upper=0.5236 effort=50 velocity=10
- joint left_dex1_finger_joint_1: axis 0 -1 0 -> 0 1 0; limit lower=-0.02 upper=0.0245 effort=20 velocity=0.2 -> lower=-0.0245 upper=0.02 effort=20 velocity=0.2
- joint left_elbow_joint: axis 0.00089601 -1 -0.00013173 -> 0 1 0; limit lower=-0.986 upper=3.071 effort=60 velocity=18.7 -> lower=-3.071 upper=0.986 effort=60 velocity=18.7
- joint left_shoulder_roll_joint: axis -1 0 0 -> 1 0 0; limit lower=-0.517 upper=2.494 effort=60 velocity=18.7 -> lower=-2.494 upper=0.517 effort=60 velocity=18.7
- joint left_shoulder_yaw_joint: axis 0 -6.4058E-05 1 -> 0 0 1
- joint left_wheel_roll_joint: axis 0 -1 0 -> 0 1 0
- joint left_wrist_pitch_joint: axis 0.00085677 -0.99993 -0.011791 -> 0 1 0
- joint left_wrist_roll_joint: axis -1 3.0614E-05 0 -> 1 0 0
- joint left_wrist_yaw_joint: axis -0.0042346 0.00012806 -0.99999 -> 0 0 1
- joint pelvis_joint: axis 0 0 0 -> (none)
- joint right_dex1_finger_joint_1: axis 0 -1 0 -> 0 1 0; limit lower=-0.02 upper=0.0245 effort=20 velocity=0.2 -> lower=-0.0245 upper=0.02 effort=20 velocity=0.2
- joint right_elbow_joint: axis 0.00089601 1 -0.00013173 -> 0 1 0
- joint right_shoulder_pitch_joint: axis 0 -1 0 -> 0 1 0; limit lower=-2.618 upper=1.833 effort=130 velocity=21.9 -> lower=-1.833 upper=2.618 effort=130 velocity=21.9
- joint right_shoulder_roll_joint: axis -1 0 0 -> 1 0 0; limit lower=-2.494 upper=0.517 effort=60 velocity=18.7 -> lower=-0.517 upper=2.494 effort=60 velocity=18.7
- joint right_shoulder_yaw_joint: axis 0 -6.4058E-05 1 -> 0 0 1
- joint right_wrist_pitch_joint: axis 0.00085677 -0.99993 -0.011791 -> 0 1 0
- joint right_wrist_roll_joint: axis -1 -3.0614E-05 0 -> 1 0 0
- joint right_wrist_yaw_joint: axis -0.0042346 -0.00012806 -0.99999 -> 0 0 1
- joint waist_pitch_joint: axis 0 -1 0 -> 0 1 0; limit lower=-2 upper=0 effort=200 velocity=30 -> lower=0 upper=2 effort=200 velocity=30
