Commit message: update g1_d

File: robots/g1_d_description/g1_d.urdf (robot description, URDF)
Before this commit: robot G1_D, 41 links, 40 joints
Links:
- added link Body_Depth_Camera_Link, mass 0.0034103483590604; collision mesh filename=meshes/Body_Depth_Camera_Link.STL; visual mesh filename=meshes/Body_Depth_Camera_Link.STL
- added link Left_depth_Camera_Link, mass 0.01577; collision mesh filename=meshes/Left_depth_Camera_Link.STL; visual mesh filename=meshes/Left_depth_Camera_Link.STL
- added link Lidar_Link, mass 0.24404; collision mesh filename=meshes/Lidar_Link.STL; visual mesh filename=meshes/Lidar_Link.STL
- added link RIght_depth_Camera_Link, mass 0.01577; collision mesh filename=meshes/RIght_depth_Camera_Link.STL; visual mesh filename=meshes/RIght_depth_Camera_Link.STL
Joints:
- added joint Body_Depth_Camera_Joint: type fixed, parent Yaw_Link, child Body_Depth_Camera_Link, origin xyz=0.058 0.0325 0.5205 rpy=0 0.83103 0, axis 0 0 0, limit lower=0 upper=0 effort=0 velocity=0
- added joint Left_depth_Camera_Joint: type fixed, parent AGV_link, child Left_depth_Camera_Link, origin xyz=0.249925151 0.091113702 -0.004567121 rpy=0 0 0, axis 0 0 0
- added joint Lidar_Joint: type fixed, parent AGV_link, child Lidar_Link, origin xyz=0.1871 -0.016137 0.10085 rpy=0 0 0, axis 0 1 0, limit lower=0 upper=0 effort=0 velocity=0
- added joint RIght_depth_Camera_Joint: type fixed, parent AGV_link, child RIght_depth_Camera_Link, origin xyz=0.246495981 -0.090876247 -0.002656756 rpy=0 0 0, axis 0 0 0
