Commit message: update G1_D_Dex1

File: robots/g1_d_description/g1_d_with_dex1_1.urdf (robot description, URDF)
Before this commit: robot G1_D_Dex1, 35 links, 34 joints
Links:
- added link Caster_FL_Link, mass 0.0574593243579511; collision mesh filename=meshes/Caster_FL_Link.STL; visual mesh filename=meshes/Caster_FL_Link.STL
- added link Caster_FL_Wheel_Link, mass 0.0925647599142116; collision mesh filename=meshes/Caster_FL_Wheel_Link.STL; visual mesh filename=meshes/Caster_FL_Wheel_Link.STL
- added link Caster_FR_Link, mass 0.0574593243577952; collision mesh filename=meshes/Caster_FR_Link.STL; visual mesh filename=meshes/Caster_FR_Link.STL
- added link Caster_FR_Wheel_Link, mass 0.0925647599142605; collision mesh filename=meshes/Caster_FR_Wheel_Link.STL; visual mesh filename=meshes/Caster_FR_Wheel_Link.STL
- added link Caster_RL_Link, mass 0.057459324357813; collision mesh filename=meshes/Caster_RL_Link.STL; visual mesh filename=meshes/Caster_RL_Link.STL
- added link Caster_RL_Wheel_Link, mass 0.0925647599142039; collision mesh filename=meshes/Caster_RL_Wheel_Link.STL; visual mesh filename=meshes/Caster_RL_Wheel_Link.STL
- added link Caster_RR_Link, mass 0.0574593243579309; collision mesh filename=meshes/Caster_RR_Link.STL; visual mesh filename=meshes/Caster_RR_Link.STL
- added link Caster_RR_Wheel_Link, mass 0.0925647599142061; collision mesh filename=meshes/Caster_RR_Wheel_Link.STL; visual mesh filename=meshes/Caster_RR_Wheel_Link.STL
- added link left_dex1_camera_link, mass 0.021494; collision mesh filename=meshes/Camera.STL; visual mesh filename=meshes/Camera.STL
- added link right_dex1_camera_link, mass 0.021494; collision mesh filename=meshes/Camera.STL; visual mesh filename=meshes/Camera.STL
- link left_dex1_base_link: mass 0.19138 -> 0.3649
- link left_dex1_finger_link_1: mass 0.086783 -> 0.092189; geometry collision mesh filename=meshes/Dex1_finger_link_1.STL; visual mesh filename=meshes/Dex1_finger_link_1.STL
- link left_dex1_finger_link_2: mass 0.086783 -> 0.092189; geometry collision mesh filename=meshes/Dex1_finger_link_2.STL; visual mesh filename=meshes/Dex1_finger_link_2.STL
- link right_dex1_base_link: mass 0.19138 -> 0.3649
- link right_dex1_finger_link_1: mass 0.086783 -> 0.092189; geometry collision mesh filename=meshes/Dex1_finger_link_1.STL; visual mesh filename=meshes/Dex1_finger_link_1.STL
- link right_dex1_finger_link_2: mass 0.086783 -> 0.092189; geometry collision mesh filename=meshes/Dex1_finger_link_2.STL; visual mesh filename=meshes/Dex1_finger_link_2.STL
Joints:
- added joint Caster_FL_Joint: type continuous, parent AGV_link, child Caster_FL_Link, origin xyz=0.167225030065905 0.171 -0.0148569592560352 rpy=0 0 0, axis 0.0151106556171685 -3.50561964968218E-05 -0.999885826911194
- added joint Caster_FL_Wheel_Joint: type continuous, parent Caster_FL_Link, child Caster_FL_Wheel_Link, origin xyz=-0.025518 5.9202E-05 -0.065143 rpy=0 0 0, axis 0.00232 1 0
- added joint Caster_FR_Joint: type continuous, parent AGV_link, child Caster_FR_Link, origin xyz=0.16643 -0.17177 -0.014857 rpy=0 0 0, axis 0.015111 -3.5056E-05 -0.99989
- added joint Caster_FR_Wheel_Joint: type continuous, parent Caster_FR_Link, child Caster_FR_Wheel_Link, origin xyz=-0.0255184881556991 5.92020066988441E-05 -0.0651430407439647 rpy=0 0 0, axis -0.00231995904376139 -0.999997308891397 0
- added joint Caster_RL_Joint: type continuous, parent AGV_link, child Caster_RL_Link, origin xyz=-0.16598 0.17177 -0.019893 rpy=0 0 0, axis 0.015111 -3.5056E-05 -0.99989
- added joint Caster_RL_Wheel_Joint: type continuous, parent Caster_RL_Link, child Caster_RL_Wheel_Link, origin xyz=-0.025518 5.9202E-05 -0.065143 rpy=0 0 0, axis 0.00232 1 0
- added joint Caster_RR_Joint: type continuous, parent AGV_link, child Caster_RR_Link, origin xyz=-0.16677 -0.171 -0.019893 rpy=0 0 0, axis 0.015111 -3.5056E-05 -0.99989
- added joint Caster_RR_Wheel_Joint: type continuous, parent Caster_RR_Link, child Caster_RR_Wheel_Link, origin xyz=-0.025518 5.9202E-05 -0.065143 rpy=0 0 0, axis -0.00232 -1 0
- added joint left_dex1_camera_joint: type fixed, parent left_dex1_base_link, child left_dex1_camera_link, origin xyz=0.068743 0 0.047476 rpy=1.5708 0.5236 0
- added joint right_dex1_camera_joint: type fixed, parent right_dex1_base_link, child right_dex1_camera_link, origin xyz=0.068743 0 0.047476 rpy=1.5708 0.5236 0
- joint left_dex1_finger_joint_1: limit lower=-0.02 upper=0.0245 effort=20 velocity=0.2 -> lower=0 upper=0.041 effort=20 velocity=0.2; origin xyz=0 0 0 rpy=0 0 0 -> xyz=0.0633 0.024916 0.010658 rpy=0 0 0
- joint left_dex1_finger_joint_2: limit lower=-0.02 upper=0.0245 effort=20 velocity=0.2 -> lower=0 upper=0.041 effort=20 velocity=0.2; origin xyz=0 0 0 rpy=0 0 0 -> xyz=0.0633 -0.024916 -0.010658 rpy=0 0 0
- joint right_dex1_finger_joint_1: limit lower=-0.02 upper=0.0245 effort=20 velocity=0.2 -> lower=0 upper=0.041 effort=20 velocity=0.2; origin xyz=0 0 0 rpy=0 0 0 -> xyz=0.0633 0.024916 0.010658 rpy=0 0 0
- joint right_dex1_finger_joint_2: limit lower=-0.02 upper=0.0245 effort=20 velocity=0.2 -> lower=0 upper=0.041 effort=20 velocity=0.2; origin xyz=0 0 0 rpy=0 0 0 -> xyz=0.0633 -0.024916 -0.010658 rpy=0 0 0

Commit message: update G1_D_Dex1

File: robots/g1_d_description/g1_d_with_dex1_1.urdf (robot description, URDF)
Before this commit: robot G1_D_Dex1, 45 links, 44 joints
Joints:
- joint Left_depth_Camera_Joint: origin xyz=0.249925151 0.091113702 -0.004567121 rpy=0 0 0 -> xyz=0.246495981 0.090876247 -0.002656756 rpy=0 0 0
