Commit message: update dex1_1

File: robots/dexterous_hand_description/dex1_1/dex1_1.urdf (robot description, URDF)
Before this commit: robot dex1_1, 7 links, 6 joints
Links:
- removed link Link1_1
- removed link Link1_2
- removed link Link1_3
- removed link Link2_1
- removed link Link2_2
- removed link Link2_3
- removed link base_link
- added link Camera, mass 0.021494; collision mesh filename=meshes/Camera.STL; visual mesh filename=meshes/Camera.STL
- added link Dex1_base_link, mass 0.3649; collision mesh filename=meshes/Dex1_base_link.STL; visual mesh filename=meshes/Dex1_base_link.STL
- added link Dex1_finger_link_1, mass 0.092189; collision mesh filename=meshes/Dex1_finger_link_1.STL; visual mesh filename=meshes/Dex1_finger_link_1.STL
- added link Dex1_finger_link_2, mass 0.092189; collision mesh filename=meshes/Dex1_finger_link_2.STL; visual mesh filename=meshes/Dex1_finger_link_2.STL
Joints:
- removed joint Joint1_1
- removed joint Joint1_2
- removed joint Joint1_3
- removed joint Joint2_1
- removed joint Joint2_2
- removed joint Joint2_3
- added joint Camera: type fixed, parent Dex1_base_link, child Camera, origin xyz=0.068743 0 0.047476 rpy=1.5708 0.5236 0, axis 0 0 0
- added joint Dex1_finger_joint_1: type prismatic, parent Dex1_base_link, child Dex1_finger_link_1, origin xyz=0.0633 0.024916 0.010658 rpy=0 0 0, axis 0 -1 0, limit lower=0 upper=0.041 effort=0 velocity=0
- added joint Dex1_finger_joint_2: type prismatic, parent Dex1_base_link, child Dex1_finger_link_2, origin xyz=0.0633 -0.024916 -0.010658 rpy=0 0 0, axis 0 1 0, limit lower=0 upper=0.041 effort=0 velocity=0
